File: 8channels/probe-rs-hive.kicad_pcb (KiCad board)
At the start: 4 copper layers, 46 x 52.8 mm, 16 parts, among them J1 Conn_01x18_Female, J2 Conn_01x18_Male, P1 PCIEX1_02X18, P2 PCIEX1_02X18, U1 SN74CB3Q3251PWR, U2 SN74CB3Q3251PWR, U3 SN74CB3Q3251PWR, U4 SN74CB3Q3251PWR

Commit message: Fix DRC
Routing:
- net /VCC: track 36.1 -> 134.9 mm, vias 0 -> 6
- net /RST: track 130.3 -> 135.0 mm
- net /S2: track 77.0 -> 76.1 mm
- net /OE: track 50.9 -> 50.0 mm, vias 4 -> 5
- net /GND: vias 0 -> 16
- added copper zone on B.Cu, net /GND
Other:
- rule via_min_drill: 0.3 -> 0.2
