File: 8lanes/8lanes.kicad_pcb (KiCad board)
At the start: 4 copper layers, 72.5 x 237.5 mm, 56 parts, among them J101 Conn_01x20_Female, J102 Conn_01x20_Female, J103 Conn_ARM_JTAG_SWD_20, J104 Conn_ARM_JTAG_SWD_20, J105 Conn_01x20_Female, J106 Conn_01x20_Female, J107 Conn_ARM_JTAG_SWD_20, J108 Conn_ARM_JTAG_SWD_20, J109 Conn_01x20_Female, J110 Conn_01x20_Female, J111 Conn_ARM_JTAG_SWD_20, J112 Conn_ARM_JTAG_SWD_20, J113 Conn_01x20_Female, J114 Conn_01x20_Female, J115 Conn_ARM_JTAG_SWD_20, J116 Conn_ARM_JTAG_SWD_20, J117 Raspberry_Pi_2_3, J118 Conn_ST_STDC14, J119 Conn_ST_STDC14, J120 Conn_ST_STDC14, J121 Conn_ST_STDC14, J122 Conn_ST_STDC14, J123 Conn_ST_STDC14, J124 Conn_ST_STDC14, J125 Conn_ST_STDC14, U101 SN74CB3Q3251PWR, U102 SN74CB3Q3251PWR, U103 SN74CB3Q3251PWR, U104 SN74CB3Q3251PWR, U105 SN74CB3Q3251PWR, U106 SN74CB3Q3251PWR, U107 SN74CB3Q3251PWR, U108 SN74CB3Q3251PWR, U109 SN74CB3Q3251PWR, U110 SN74CB3Q3251PWR, U111 SN74CB3Q3251PWR, U112 SN74CB3Q3251PWR, U113 SN74CB3Q3251PWR, U114 SN74CB3Q3251PWR

Commit message: Silk fix
Other:
- board text added: "probe-rs Hive Design by Noah Huesser (@yatekii) Routing by Emil Fresk (@korken89)"
- board text removed: "Probe-rs Hive Design by Noah Huesser (@yatekii) Routing by Emil Fresk (@korken89)"
