File: 8lanes/8lanes.kicad_pcb (KiCad board)
At the start: 4 copper layers, 72.5 x 237.5 mm, 56 parts, among them J101 Conn_01x20_Female, J102 Conn_01x20_Female, J103 Conn_ARM_JTAG_SWD_20, J104 Conn_ARM_JTAG_SWD_20, J105 Conn_01x20_Female, J106 Conn_01x20_Female, J107 Conn_ARM_JTAG_SWD_20, J108 Conn_ARM_JTAG_SWD_20, J109 Conn_01x20_Female, J110 Conn_01x20_Female, J111 Conn_ARM_JTAG_SWD_20, J112 Conn_ARM_JTAG_SWD_20, J113 Conn_01x20_Female, J114 Conn_01x20_Female, J115 Conn_ARM_JTAG_SWD_20, J116 Conn_ARM_JTAG_SWD_20, J117 Raspberry_Pi_2_3, J118 Conn_ST_STDC14, J119 Conn_ST_STDC14, J120 Conn_ST_STDC14, J121 Conn_ST_STDC14, J122 Conn_ST_STDC14, J123 Conn_ST_STDC14, J124 Conn_ST_STDC14, J125 Conn_ST_STDC14, U101 SN74CB3Q3251PWR, U102 SN74CB3Q3251PWR, U103 SN74CB3Q3251PWR, U104 SN74CB3Q3251PWR, U105 SN74CB3Q3251PWR, U106 SN74CB3Q3251PWR, U107 SN74CB3Q3251PWR, U108 SN74CB3Q3251PWR, U109 SN74CB3Q3251PWR, U110 SN74CB3Q3251PWR, U111 SN74CB3Q3251PWR, U112 SN74CB3Q3251PWR, U113 SN74CB3Q3251PWR, U114 SN74CB3Q3251PWR

Commit message: More distance between lanes
Parts:
- moved C115 17.5 mm to (70.5, 217.5)
- moved J114 17.5 mm to (55.0, 212.5)
- moved U108 17.5 mm to (67.5, 217.5)
- moved C108 15.0 mm to (70.5, 185.0)
- moved J110 15.0 mm to (55.0, 180.0)
- moved U106 15.0 mm to (67.5, 185.0)
- moved C106 12.5 mm to (70.5, 152.5)
- moved J106 12.5 mm to (55.0, 147.5)
- moved U104 12.5 mm to (67.5, 152.5)
- moved C105 10.0 mm to (70.5, 120.0)
- moved J102 10.0 mm to (55.0, 115.0)
- moved U102 10.0 mm to (67.5, 120.0)
- moved C104 7.50 mm to (70.5, 87.5)
- moved J113 7.50 mm to (55.0, 82.5)
- moved U107 7.50 mm to (67.5, 87.5)
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Routing:
- net /TMS|SWDIO: track 251.6 -> 271.0 mm
- net +5V: track 329.1 -> 347.6 mm
- net /MCU_S0: track 302.1 -> 319.6 mm
- net /ROW_S2: track 262.5 -> 280.0 mm
- net /ROW_S1: track 264.4 -> 281.9 mm
- net /ROW_S0: track 265.5 -> 283.0 mm
- net /OE_LANE8: track 220.9 -> 238.4 mm
- net /MCU_S2: track 313.5 -> 331.0 mm
- net /MCU_S1: track 330.7 -> 348.2 mm
- net /TDI|EXT: track 282.5 -> 299.7 mm
- net /RST: track 273.4 -> 288.5 mm
- net /OE_LANE7: track 190.2 -> 205.2 mm
- net /TCK|SWDCLK: track 289.1 -> 304.0 mm
- net /TDO|SWO: track 269.5 -> 282.9 mm
- net /OE_LANE6: track 159.8 -> 172.3 mm
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Other:
- board size 72.5 x 237.5 mm -> 72.5 x 255 mm
- board text added: "probe-rs Hive By Noah Huesser (@yatekii) & Emil Fresk (@korken89)"
- board text removed: "probe-rs Hive Design by Noah Huesser (@yatekii) Routing by Emil Fresk (@korken89)"
