File: shields/target_stack_shield/bus_switches.sch (KiCad schematic (older format))
At the start: 8 parts, among them U1 SN74CB3T16211DGGR, U2 SN74CB3T16211DGGR, U3 SN74CB3T16211DGGR, U4 SN74CB3T16211DGGR

Commit message: Further work on layout
Connections:
- net BUS_RST: now also U1.41 (2B1), U1.54 (1B1), U2.41 (2B1), U2.54 (1B1), U3.15 (2A1), U3.2 (1A1), U4.15 (2A1), U4.2 (1A1); no longer U1.36 (2B5), U1.50 (1B5), U2.36 (2B5), U2.50 (1B5), U3.21 (2A5), U3.6 (1A5), U4.21 (2A5), U4.6 (1A5)
- net BUS_TCK|SWDCLK: now also U1.37 (2B4), U1.51 (1B4), U2.37 (2B4), U2.51 (1B4), U3.20 (2A4), U3.5 (1A4), U4.20 (2A4), U4.5 (1A4); no longer U1.40 (2B2), U1.53 (1B2), U2.40 (2B2), U2.53 (1B2), U3.16 (2A2), U3.3 (1A2), U4.16 (2A2), U4.3 (1A2)
- net BUS_TDI|NC: now also U1.40 (2B2), U1.53 (1B2), U2.40 (2B2), U2.53 (1B2), U3.16 (2A2), U3.3 (1A2), U4.16 (2A2), U4.3 (1A2); no longer U1.37 (2B4), U1.51 (1B4), U2.37 (2B4), U2.51 (1B4), U3.20 (2A4), U3.5 (1A4), U4.20 (2A4), U4.5 (1A4)
- net BUS_TMS|SWDIO: now also U1.36 (2B5), U1.50 (1B5), U2.36 (2B5), U2.50 (1B5), U3.21 (2A5), U3.6 (1A5), U4.21 (2A5), U4.6 (1A5); no longer U1.41 (2B1), U1.54 (1B1), U2.41 (2B1), U2.54 (1B1), U3.15 (2A1), U3.2 (1A1), U4.15 (2A1), U4.2 (1A1)
- net RST_0: now also U2.15 (2A1); no longer U2.21 (2A5)
- net RST_1: now also U2.2 (1A1); no longer U2.6 (1A5)
- net RST_2: now also U1.15 (2A1); no longer U1.21 (2A5)
- net RST_3: now also U1.2 (1A1); no longer U1.6 (1A5)
- net TARGET_SW_CH0: now also U3.56 (1~OE); no longer U3.55 (2~OE)
- net TARGET_SW_CH1: now also U3.55 (2~OE); no longer U3.56 (1~OE)
- net TARGET_SW_CH2: now also U4.56 (1~OE); no longer U4.55 (2~OE)
- net TARGET_SW_CH3: now also U4.55 (2~OE); no longer U4.56 (1~OE)
- net TCK|SWDCLK_0: now also U2.20 (2A4); no longer U2.16 (2A2)
- net TCK|SWDCLK_1: now also U2.5 (1A4); no longer U2.3 (1A2)
- net TCK|SWDCLK_2: now also U1.20 (2A4); no longer U1.16 (2A2)
- net TCK|SWDCLK_3: now also U1.5 (1A4); no longer U1.3 (1A2)
- net TDI|NC_0: now also U2.16 (2A2); no longer U2.20 (2A4)
- net TDI|NC_1: now also U2.3 (1A2); no longer U2.5 (1A4)
- net TDI|NC_2: now also U1.16 (2A2); no longer U1.20 (2A4)
- net TDI|NC_3: now also U1.3 (1A2); no longer U1.5 (1A4)
- net TGT_GPIO0.0: now also U3.48 (1B6); no longer U3.35 (2B6)
- net TGT_GPIO0.1: now also U3.47 (1B7); no longer U3.34 (2B7)
- net TGT_GPIO0.2: now also U3.46 (1B8); no longer U3.33 (2B8)
- net TGT_GPIO0.3: now also U3.45 (1B9); no longer U3.32 (2B9)
- net TGT_GPIO1.0: now also U3.35 (2B6); no longer U3.48 (1B6)
- net TGT_GPIO1.1: now also U3.34 (2B7); no longer U3.47 (1B7)
- net TGT_GPIO1.2: now also U3.33 (2B8); no longer U3.46 (1B8)
- net TGT_GPIO1.3: now also U3.32 (2B9); no longer U3.45 (1B9)
- net TGT_GPIO2.0: now also U4.48 (1B6); no longer U4.35 (2B6)
- net TGT_GPIO2.1: now also U4.47 (1B7); no longer U4.34 (2B7)
- net TGT_GPIO2.2: now also U4.46 (1B8); no longer U4.33 (2B8)
- net TGT_GPIO2.3: now also U4.45 (1B9); no longer U4.32 (2B9)
- net TGT_GPIO3.0: now also U4.35 (2B6); no longer U4.48 (1B6)
- net TGT_GPIO3.1: now also U4.34 (2B7); no longer U4.47 (1B7)
- net TGT_GPIO3.2: now also U4.33 (2B8); no longer U4.46 (1B8)
- net TGT_GPIO3.3: now also U4.32 (2B9); no longer U4.45 (1B9)
- net TGT_RST_0: now also U3.54 (1B1); no longer U3.36 (2B5)
- net TGT_RST_1: now also U3.41 (2B1); no longer U3.50 (1B5)
- net TGT_RST_2: now also U4.54 (1B1); no longer U4.36 (2B5)
- net TGT_RST_3: now also U4.41 (2B1); no longer U4.50 (1B5)
- net TGT_TCK|SWDCLK_0: now also U3.51 (1B4); no longer U3.40 (2B2)
- net TGT_TCK|SWDCLK_1: now also U3.37 (2B4); no longer U3.53 (1B2)
- net TGT_TCK|SWDCLK_2: now also U4.51 (1B4); no longer U4.40 (2B2)
- net TGT_TCK|SWDCLK_3: now also U4.37 (2B4); no longer U4.53 (1B2)
- net TGT_TDI|NC_0: now also U3.53 (1B2); no longer U3.37 (2B4)
- net TGT_TDI|NC_1: now also U3.40 (2B2); no longer U3.51 (1B4)
- net TGT_TDI|NC_2: now also U4.53 (1B2); no longer U4.37 (2B4)
- net TGT_TDI|NC_3: now also U4.40 (2B2); no longer U4.51 (1B4)
- net TGT_TDO|SWO_0: now also U3.52 (1B3); no longer U3.39 (2B3)
- net TGT_TDO|SWO_1: now also U3.39 (2B3); no longer U3.52 (1B3)
- net TGT_TDO|SWO_2: now also U4.52 (1B3); no longer U4.39 (2B3)
- net TGT_TDO|SWO_3: now also U4.39 (2B3); no longer U4.52 (1B3)
- net TGT_TMS|SWDIO_0: now also U3.50 (1B5); no longer U3.41 (2B1)
- net TGT_TMS|SWDIO_1: now also U3.36 (2B5); no longer U3.54 (1B1)
- net TGT_TMS|SWDIO_2: now also U4.50 (1B5); no longer U4.41 (2B1)
- net TGT_TMS|SWDIO_3: now also U4.36 (2B5); no longer U4.54 (1B1)
- net TGT_UART_RxD0: now also U3.43 (1B11); no longer U3.30 (2B11)
- net TGT_UART_RxD1: now also U3.30 (2B11); no longer U3.43 (1B11)
- net TGT_UART_RxD2: now also U4.43 (1B11); no longer U4.30 (2B11)
- net TGT_UART_RxD3: now also U4.30 (2B11); no longer U4.43 (1B11)
- net TGT_UART_TxD0: now also U3.44 (1B10); no longer U3.31 (2B10)
- net TGT_UART_TxD1: now also U3.31 (2B10); no longer U3.44 (1B10)
- net TGT_UART_TxD2: now also U4.44 (1B10); no longer U4.31 (2B10)
- net TGT_UART_TxD3: now also U4.31 (2B10); no longer U4.44 (1B10)
- net TMS|SWDIO_0: now also U2.21 (2A5); no longer U2.15 (2A1)
- net TMS|SWDIO_1: now also U2.6 (1A5); no longer U2.2 (1A1)
- net TMS|SWDIO_2: now also U1.21 (2A5); no longer U1.15 (2A1)
- net TMS|SWDIO_3: now also U1.6 (1A5); no longer U1.2 (1A1)

Commit message: finished target stack shield layout
Connections:
- net BUS_GPIO1: now also U3.6 (1A5), U4.6 (1A5); no longer U3.9 (1A7), U4.9 (1A7)
- net BUS_GPIO2: now also U3.5 (1A4), U4.5 (1A4); no longer U3.10 (1A8), U4.10 (1A8)
- net BUS_GPIO3: now also U3.4 (1A3), U4.4 (1A3); no longer U3.11 (1A9), U4.11 (1A9)
- net BUS_RST: now also U3.13 (1A11), U4.13 (1A11); no longer U3.2 (1A1), U4.2 (1A1)
- net BUS_TCK|SWDCLK: now also U3.10 (1A8), U4.10 (1A8); no longer U3.5 (1A4), U4.5 (1A4)
- net BUS_TDI|NC: now also U3.12 (1A10), U4.12 (1A10); no longer U3.3 (1A2), U4.3 (1A2)
- net BUS_TDO|SWO: now also U3.11 (1A9), U4.11 (1A9); no longer U3.4 (1A3), U4.4 (1A3)
- net BUS_TMS|SWDIO: now also U3.9 (1A7), U4.9 (1A7); no longer U3.6 (1A5), U4.6 (1A5)
- net BUS_UART_RxD: now also U3.2 (1A1), U4.2 (1A1); no longer U3.13 (1A11), U4.13 (1A11)
- net BUS_UART_TxD: now also U3.3 (1A2), U4.3 (1A2); no longer U3.12 (1A10), U4.12 (1A10)
- net TGT_GPIO0.1: now also U3.50 (1B5); no longer U3.47 (1B7)
- net TGT_GPIO0.2: now also U3.51 (1B4); no longer U3.46 (1B8)
- net TGT_GPIO0.3: now also U3.52 (1B3); no longer U3.45 (1B9)
- net TGT_GPIO2.1: now also U4.50 (1B5); no longer U4.47 (1B7)
- net TGT_GPIO2.2: now also U4.51 (1B4); no longer U4.46 (1B8)
- net TGT_GPIO2.3: now also U4.52 (1B3); no longer U4.45 (1B9)
- net TGT_RST_0: now also U3.43 (1B11); no longer U3.54 (1B1)
- net TGT_RST_2: now also U4.43 (1B11); no longer U4.54 (1B1)
- net TGT_TCK|SWDCLK_0: now also U3.46 (1B8); no longer U3.51 (1B4)
- net TGT_TCK|SWDCLK_2: now also U4.46 (1B8); no longer U4.51 (1B4)
- net TGT_TDI|NC_0: now also U3.44 (1B10); no longer U3.53 (1B2)
- net TGT_TDI|NC_2: now also U4.44 (1B10); no longer U4.53 (1B2)
- net TGT_TDO|SWO_0: now also U3.45 (1B9); no longer U3.52 (1B3)
- net TGT_TDO|SWO_2: now also U4.45 (1B9); no longer U4.52 (1B3)
- net TGT_TMS|SWDIO_0: now also U3.47 (1B7); no longer U3.50 (1B5)
- net TGT_TMS|SWDIO_2: now also U4.47 (1B7); no longer U4.50 (1B5)
- net TGT_UART_RxD0: now also U3.54 (1B1); no longer U3.43 (1B11)
- net TGT_UART_RxD2: now also U4.54 (1B1); no longer U4.43 (1B11)
- net TGT_UART_TxD0: now also U3.53 (1B2); no longer U3.44 (1B10)
- net TGT_UART_TxD2: now also U4.53 (1B2); no longer U4.44 (1B10)
Changed lines of the file:
@@
 	0    1    -1   0
 $EndComp
-Text Label 7700 7250 0    50   ~ 0
+Text Label 7700 8250 0    50   ~ 0
 BUS_RST
-Text Label 7700 7650 0    50   ~ 0
+Text Label 7700 7850 0    50   ~ 0
 BUS_TMS|SWDIO
-Text Label 7700 7550 0    50   ~ 0
+Text Label 7700 7950 0    50   ~ 0
 BUS_TCK|SWDCLK
-Text Label 7700 7450 0    50   ~ 0
+Text Label 7700 8050 0    50   ~ 0
 BUS_TDO|SWO
-Text Label 7700 7350 0    50   ~ 0
+Text Label 7700 8150 0    50   ~ 0
 BUS_TDI|NC
 Text Label 7700 7750 0    50   ~ 0
 BUS_GPIO0
-Text Label 7700 7850 0    50   ~ 0
+Text Label 7700 7650 0    50   ~ 0
 BUS_GPIO1
-Text Label 7700 7950 0    50   ~ 0
+Text Label 7700 7550 0    50   ~ 0
 BUS_GPIO2
-Text Label 7700 8050 0    50   ~ 0
+Text Label 7700 7450 0    50   ~ 0
 BUS_GPIO3
-Text Label 7700 8150 0    50   ~ 0
+Text Label 7700 7350 0    50   ~ 0
 BUS_UART_TxD
-Text Label 7700 8250 0    50   ~ 0
+Text Label 7700 7250 0    50   ~ 0
 BUS_UART_RxD
 $Comp
@@
 	0    1    -1   0
 $EndComp
-Text Label 7700 2400 0    50   ~ 0
+Text Label 7700 3400 0    50   ~ 0
 BUS_RST
-Text Label 7700 2800 0    50   ~ 0
+Text Label 7700 3000 0    50   ~ 0
 BUS_TMS|SWDIO
-Text Label 7700 2700 0    50   ~ 0
+Text Label 7700 3100 0    50   ~ 0
 BUS_TCK|SWDCLK
-Text Label 7700 2600 0    50   ~ 0
+Text Label 7700 3200 0    50   ~ 0
 BUS_TDO|SWO
-Text Label 7700 2500 0    50   ~ 0
+Text Label 7700 3300 0    50   ~ 0
 BUS_TDI|NC
 Text Label 7700 2900 0    50   ~ 0
 BUS_GPIO0
-Text Label 7700 3000 0    50   ~ 0
+Text Label 7700 2800 0    50   ~ 0
 BUS_GPIO1
-Text Label 7700 3100 0    50   ~ 0
+Text Label 7700 2700 0    50   ~ 0
 BUS_GPIO2
-Text Label 7700 3200 0    50   ~ 0
+Text Label 7700 2600 0    50   ~ 0
 BUS_GPIO3
-Text Label 7700 3300 0    50   ~ 0
+Text Label 7700 2500 0    50   ~ 0
 BUS_UART_TxD
-Text Label 7700 3400 0    50   ~ 0
+Text Label 7700 2400 0    50   ~ 0
 BUS_UART_RxD
 $Comp
@@
 Text Label 3150 2100 0    50   ~ 0
 BUS_SW_CH3
-Text HLabel 9750 2200 2    50   BiDi ~ 0
+Text HLabel 9750 2400 2    50   BiDi ~ 0
 TGT_TMS|SWDIO_0
-Text HLabel 9750 2100 2    50   Output ~ 0
+Text HLabel 9750 2500 2    50   Output ~ 0
 TGT_TCK|SWDCLK_0
-Text HLabel 9750 1900 2    50   Output ~ 0
+Text HLabel 9750 2700 2    50   Output ~ 0
 TGT_TDI|NC_0
-Text HLabel 9750 2000 2    50   Input ~ 0
+Text HLabel 9750 2600 2    50   Input ~ 0
 TGT_TDO|SWO_0
-Text HLabel 9750 1800 2    50   Output ~ 0
+Text HLabel 9750 2800 2    50   Output ~ 0
 TGT_RST_0
 Text HLabel 9750 2300 2    50   BiDi ~ 0
 TGT_GPIO0.0
-Text HLabel 9750 2400 2    50   BiDi ~ 0
+Text HLabel 9750 2200 2    50   BiDi ~ 0
 TGT_GPIO0.1
-Text HLabel 9750 2500 2    50   BiDi ~ 0
+Text HLabel 9750 2100 2    50   BiDi ~ 0
 TGT_GPIO0.2
-Text HLabel 9750 2600 2    50   BiDi ~ 0
+Text HLabel 9750 2000 2    50   BiDi ~ 0
 TGT_GPIO0.3
-Text HLabel 9750 2700 2    50   BiDi ~ 0
+Text HLabel 9750 1900 2    50   BiDi ~ 0
 TGT_UART_TxD0
-Text HLabel 9750 2800 2    50   BiDi ~ 0
+Text HLabel 9750 1800 2    50   BiDi ~ 0
 TGT_UART_RxD0
 $Comp
@@
 	0    -1   1    0
 $EndComp
-Text HLabel 9750 7650 2    50   BiDi ~ 0
+Text HLabel 9750 6650 2    50   BiDi ~ 0
 TGT_UART_RxD2
-Text HLabel 9750 7550 2    50   BiDi ~ 0
+Text HLabel 9750 6750 2    50   BiDi ~ 0
 TGT_UART_TxD2
-Text HLabel 9750 7450 2    50   BiDi ~ 0
+Text HLabel 9750 6850 2    50   BiDi ~ 0
 TGT_GPIO2.3
-Text HLabel 9750 7350 2    50   BiDi ~ 0
+Text HLabel 9750 6950 2    50   BiDi ~ 0
 TGT_GPIO2.2
-Text HLabel 9750 7250 2    50   BiDi ~ 0
+Text HLabel 9750 7050 2    50   BiDi ~ 0
 TGT_GPIO2.1
 Text HLabel 9750 7150 2    50   BiDi ~ 0
 TGT_GPIO2.0
-Text HLabel 9750 6650 2    50   Output ~ 0
+Text HLabel 9750 7650 2    50   Output ~ 0
 TGT_RST_2
-Text HLabel 9750 6750 2    50   Output ~ 0
+Text HLabel 9750 7550 2    50   Output ~ 0
 TGT_TDI|NC_2
-Text HLabel 9750 6850 2    50   Input ~ 0
+Text HLabel 9750 7450 2    50   Input ~ 0
 TGT_TDO|SWO_2
-Text HLabel 9750 6950 2    50   Output ~ 0
+Text HLabel 9750 7350 2    50   Output ~ 0
 TGT_TCK|SWDCLK_2
-Text HLabel 9750 7050 2    50   BiDi ~ 0
+Text HLabel 9750 7250 2    50   BiDi ~ 0
 TGT_TMS|SWDIO_2
 $Comp
@@
 	7700 9550 8350 9550
 Wire Wire Line
+	7700 8250 8350 8250
+Wire Wire Line
+	7700 8150 8350 8150
+Wire Wire Line
+	7700 8050 8350 8050
+Wire Wire Line
+	7700 7950 8350 7950
+Wire Wire Line
+	7700 7850 8350 7850
+Wire Wire Line
+	7700 7750 8350 7750
+Wire Wire Line
+	7700 7650 8350 7650
+Wire Wire Line
+	7700 7550 8350 7550
+Wire Wire Line
+	7700 7450 8350 7450
+Wire Wire Line
+	7700 7350 8350 7350
+Wire Wire Line
 	7700 7250 8350 7250
-Wire Wire Line
-	7700 7350 8350 7350
-Wire Wire Line
-	7700 7450 8350 7450
-Wire Wire Line
-	7700 7550 8350 7550
-Wire Wire Line
-	7700 7650 8350 7650
-Wire Wire Line
-	7700 7750 8350 7750
-Wire Wire Line
-	7700 7850 8350 7850
-Wire Wire Line
-	7700 7950 8350 7950
-Wire Wire Line
-	7700 8050 8350 8050
-Wire Wire Line
-	7700 8150 8350 8150
-Wire Wire Line
-	7700 8250 8350 8250
 Wire Bus Line
 	6700 2300 6700 2900
@@
 	8350 3700 7700 3700
 Wire Wire Line
+	8350 2400 7700 2400
+Wire Wire Line
+	8350 2500 7700 2500
+Wire Wire Line
+	8350 2600 7700 2600
+Wire Wire Line
+	8350 2700 7700 2700
+Wire Wire Line
+	8350 2800 7700 2800
+Wire Wire Line
+	8350 2900 7700 2900
+Wire Wire Line
+	8350 3000 7700 3000
+Wire Wire Line
+	8350 3100 7700 3100
+Wire Wire Line
+	8350 3200 7700 3200
+Wire Wire Line
+	8350 3300 7700 3300
+Wire Wire Line
 	8350 3400 7700 3400
-Wire Wire Line
-	8350 3300 7700 3300
-Wire Wire Line
-	8350 3200 7700 3200
-Wire Wire Line
-	8350 3100 7700 3100
-Wire Wire Line
-	8350 3000 7700 3000
-Wire Wire Line
-	8350 2900 7700 2900
-Wire Wire Line
-	8350 2800 7700 2800
-Wire Wire Line
-	8350 2700 7700 2700
-Wire Wire Line
-	8350 2600 7700 2600
-Wire Wire Line
-	8350 2500 7700 2500
-Wire Wire Line
-	8350 2400 7700 2400
 Wire Bus Line
 	7700 3700 7500 3700

Commit message: added partlist and prices
Parts:
- U1, U2, U3, U4: Digikey Price (CHF) (none) -> 2.64; Manufacturer_Part_Number (none) -> SN74CB3T16211DGGR; Mouser Price (CHF) (none) -> 2.67
Changed lines of the file:
@@
 F 7 "Texas Instruments" H 4400 8350 50  0001 L BNN "SUPPLIER"
 F 8 "1567376" H 4400 8350 50  0001 L BNN "OC_FARNELL"
+F 9 "2.64" H 4400 8350 50  0001 C CNN "Digikey Price (CHF)"
+F 10 "SN74CB3T16211DGGR" H 4400 8350 50  0001 C CNN "Manufacturer_Part_Number"
+F 11 "2.67" H 4400 8350 50  0001 C CNN "Mouser Price (CHF)"
 	1    4400 8350
 	1    0    0    -1
@@
 F 7 "Texas Instruments" H 4400 3500 50  0001 L BNN "SUPPLIER"
 F 8 "1567376" H 4400 3500 50  0001 L BNN "OC_FARNELL"
+F 9 "2.64" H 4400 3500 50  0001 C CNN "Digikey Price (CHF)"
+F 10 "SN74CB3T16211DGGR" H 4400 3500 50  0001 C CNN "Manufacturer_Part_Number"
+F 11 "2.67" H 4400 3500 50  0001 C CNN "Mouser Price (CHF)"
 	1    4400 3500
 	1    0    0    -1
@@
 F 7 "Texas Instruments" H 9050 3500 50  0001 L BNN "SUPPLIER"
 F 8 "1567376" H 9050 3500 50  0001 L BNN "OC_FARNELL"
+F 9 "2.64" H 9050 3500 50  0001 C CNN "Digikey Price (CHF)"
+F 10 "SN74CB3T16211DGGR" H 9050 3500 50  0001 C CNN "Manufacturer_Part_Number"
+F 11 "2.67" H 9050 3500 50  0001 C CNN "Mouser Price (CHF)"
 	1    9050 3500
 	1    0    0    -1
@@
 F 7 "Texas Instruments" H 9050 8350 50  0001 L BNN "SUPPLIER"
 F 8 "1567376" H 9050 8350 50  0001 L BNN "OC_FARNELL"
+F 9 "2.64" H 9050 8350 50  0001 C CNN "Digikey Price (CHF)"
+F 10 "SN74CB3T16211DGGR" H 9050 8350 50  0001 C CNN "Manufacturer_Part_Number"
+F 11 "2.67" H 9050 8350 50  0001 C CNN "Mouser Price (CHF)"
 	1    9050 8350
 	1    0    0    -1
