File: shields/target_stack_shield/target_stack_shield.sch (KiCad schematic (older format))
At the start: 12 parts, among them IC1 NCP1117DT33T5G, J1 GPIO shield connector 40pin, J2 probe shield connector 26pin, J3 m2_keyA_67pin

Commit message: added M2.5 Daughterboard backup mounting solution
Parts:
- added H5: MountingHoleDaughterboard, MountingHole:MountingHole_2.7mm_M2.5, symbol Mechanical:MountingHole
Changed lines of the file:
@@
 Connection ~ 2350 3750
 Connection ~ 2350 3650
+$Comp
+L Mechanical:MountingHole H5
+U 1 1 6184E469
+P 1200 2150
+F 0 "H5" H 1300 2196 50  0000 L CNN
+F 1 "MountingHoleDaughterboard" H 1300 2105 50  0000 L CNN
+F 2 "MountingHole:MountingHole_2.7mm_M2.5" H 1200 2150 50  0001 C CNN
+F 3 "~" H 1200 2150 50  0001 C CNN
+	1    1200 2150
+	1    0    0    -1
+$EndComp
 $EndSCHEMATC

Commit message: updated LED resistor values, updated partlists, minor change to daughterboard template
Parts:
- R1: value 195 -> 560
Changed lines of the file:
@@
 P 6000 1600
 F 0 "R1" H 6059 1646 50  0000 L CNN
-F 1 "195" H 6059 1555 50  0000 L CNN
+F 1 "560" H 6059 1555 50  0000 L CNN
 F 2 "Resistor_SMD:R_0603_1608Metric_Pad1.05x0.95mm_HandSolder" H 6000 1600 50  0001 C CNN
 F 3 "~" H 6000 1600 50  0001 C CNN
