File: daughterboard/STM32_00/STM32_00.sch (KiCad schematic (older format))
At the start: 2 parts, among them J1 m2_keyA_67pin_daughterboard

Commit message: minor adjustments to daughterboard template, added STM32 daughterboard schematics
Parts:
- J1: symbol daughterboard_template-rescue:m2_keyA_67pin_daughterboard-hive -> hive:m2_keyA_67pin_daughterboard
Changed lines of the file:
@@
 encoding utf-8
 Sheet 1 5
-Title "Daughterboard template"
-Date "2021-10-11"
+Title "Daughterboard STM32 00"
+Date "2021-11-05"
 Rev "0"
 Comp "probe-rs"
@@
 You can implement 4 targets per daugtherboard.\nPlease use the corresponding hierarchical schematics for that.\n
 $Comp
-L daughterboard_template-rescue:m2_keyA_67pin_daughterboard-hive J1
+L hive:m2_keyA_67pin_daughterboard J1
 U 1 1 6181B4AF
 P 6000 3300
