File: daughterboard/STM32_00/target1.sch (KiCad schematic (older format))
At the start: 12 parts, among them U1 STM32F401CCUx

Commit message: added testpoints to daughterboards, updated readme
Parts:
- added TP1: JTMS-SWDIO, symbol Connector:TestPoint
- added TP10: GPIO2, symbol Connector:TestPoint
- added TP11: GPIO3, symbol Connector:TestPoint
- added TP2: JTCK-SWCLK, symbol Connector:TestPoint
- added TP3: JTDO-SWO, symbol Connector:TestPoint
- added TP4: JTDI, symbol Connector:TestPoint
- added TP5: NRST, symbol Connector:TestPoint
- added TP6: USART1_TX, symbol Connector:TestPoint
- added TP7: USART1_RX, symbol Connector:TestPoint
- added TP8: GPIO0, symbol Connector:TestPoint
- added TP9: GPIO1, symbol Connector:TestPoint
Connections:
- net GPIO1.0: now also TP8.1
- net GPIO1.1: now also TP9.1
- net GPIO1.2: now also TP10.1
- net GPIO1.3: now also TP11.1
- net RST_1: now also TP5.1
- net TCK|SWDCLK_1: now also TP2.1
- net TDI|NC_1: now also TP4.1
- net TDO|SWO_1: now also TP3.1
- net TMS|SWDIO_1: now also TP1.1
- net UART_RxD1: now also TP6.1
- net UART_TxD1: now also TP7.1
Changed lines of the file:
@@
 JTCK-SWCLK
 Wire Wire Line
-	1600 2700 2150 2700
-Text Label 2150 2700 2    50   ~ 0
+	1600 2700 2300 2700
+Text Label 2300 2700 2    50   ~ 0
 USART1_RX
 Wire Wire Line
-	1600 2600 2150 2600
-Text Label 2150 2600 2    50   ~ 0
+	1600 2600 2300 2600
+Text Label 2300 2600 2    50   ~ 0
 USART1_TX
 Wire Wire Line
-	1600 2100 2150 2100
-Text Label 2150 2100 2    50   ~ 0
+	1600 2100 2300 2100
+Text Label 2300 2100 2    50   ~ 0
 NRST
 Wire Wire Line
-	1600 1900 2150 1900
-Text Label 2150 2000 2    50   ~ 0
+	1600 1900 2300 1900
+Text Label 2300 2000 2    50   ~ 0
 JTDI
 Wire Wire Line
-	2150 2000 1600 2000
-Text Label 2150 1900 2    50   ~ 0
+	2300 2000 1600 2000
+Text Label 2300 1900 2    50   ~ 0
 JTDO-SWO
 Wire Wire Line
-	1600 2800 2150 2800
-Text Label 2150 2800 2    50   ~ 0
+	1600 2800 2300 2800
+Text Label 2300 2800 2    50   ~ 0
 GPIO0
 Wire Wire Line
-	1600 2900 2150 2900
-Text Label 2150 2900 2    50   ~ 0
+	1600 2900 2300 2900
+Text Label 2300 2900 2    50   ~ 0
 GPIO1
 Wire Wire Line
-	1600 3000 2150 3000
-Text Label 2150 3000 2    50   ~ 0
+	1600 3000 2300 3000
+Text Label 2300 3000 2    50   ~ 0
 GPIO2
 Wire Wire Line
-	1600 3100 2150 3100
-Text Label 2150 3100 2    50   ~ 0
+	1600 3100 2300 3100
+Text Label 2300 3100 2    50   ~ 0
 GPIO3
 Text Label 2300 1700 2    50   ~ 0
@@
 Wire Wire Line
 	7350 4550 7950 4550
+$Comp
+L Connector:TestPoint TP?
+U 1 1 619418F1
+P 2300 1700
+AR Path="/616688D6/619418F1" Ref="TP?"  Part="1"
+AR Path="/61667F91/619418F1" Ref="TP1"  Part="1"
+F 0 "TP1" V 2300 1900 50  0000 L CNN
+F 1 "JTMS-SWDIO" V 2300 2200 50  0000 L CNN
+F 2 "" H 2500 1700 50  0001 C CNN
+F 3 "~" H 2500 1700 50  0001 C CNN
+	1    2300 1700
+	0    1    1    0
+$EndComp
+$Comp
+L Connector:TestPoint TP?
+U 1 1 619418F7
+P 2300 1800
+AR Path="/616688D6/619418F7" Ref="TP?"  Part="1"
+AR Path="/61667F91/619418F7" Ref="TP2"  Part="1"
+F 0 "TP2" V 2300 2000 50  0000 L CNN
+F 1 "JTCK-SWCLK" V 2300 2300 50  0000 L CNN
+F 2 "" H 2500 1800 50  0001 C CNN
+F 3 "~" H 2500 1800 50  0001 C CNN
+	1    2300 1800
+	0    1    1    0
+$EndComp
+$Comp
+L Connector:TestPoint TP?
+U 1 1 619418FD
+P 2300 1900
+AR Path="/616688D6/619418FD" Ref="TP?"  Part="1"
+AR Path="/61667F91/619418FD" Ref="TP3"  Part="1"
+F 0 "TP3" V 2300 2100 50  0000 L CNN
+F 1 "JTDO-SWO" V 2300 2400 50  0000 L CNN
+F 2 "" H 2500 1900 50  0001 C CNN
+F 3 "~" H 2500 1900 50  0001 C CNN
+	1    2300 1900
+	0    1    1    0
+$EndComp
+$Comp
+L Connector:TestPoint TP?
+U 1 1 61941903
+P 2300 2000
+AR Path="/616688D6/61941903" Ref="TP?"  Part="1"
+AR Path="/61667F91/61941903" Ref="TP4"  Part="1"
+F 0 "TP4" V 2300 2200 50  0000 L CNN
+F 1 "JTDI" V 2300 2500 50  0000 L CNN
+F 2 "" H 2500 2000 50  0001 C CNN
+F 3 "~" H 2500 2000 50  0001 C CNN
+	1    2300 2000
+	0    1    1    0
+$EndComp
+$Comp
+L Connector:TestPoint TP?
+U 1 1 61941909
+P 2300 2100
+AR Path="/616688D6/61941909" Ref="TP?"  Part="1"
+AR Path="/61667F91/61941909" Ref="TP5"  Part="1"
+F 0 "TP5" V 2300 2300 50  0000 L CNN
+F 1 "NRST" V 2300 2600 50  0000 L CNN
+F 2 "" H 2500 2100 50  0001 C CNN
+F 3 "~" H 2500 2100 50  0001 C CNN
+	1    2300 2100
+	0    1    1    0
+$EndComp
+$Comp
+L Connector:TestPoint TP?
+U 1 1 6194190F
+P 2300 2600
+AR Path="/616688D6/6194190F" Ref="TP?"  Part="1"
+AR Path="/61667F91/6194190F" Ref="TP6"  Part="1"
+F 0 "TP6" V 2300 2800 50  0000 L CNN
+F 1 "USART1_TX" V 2300 3100 50  0000 L CNN
+F 2 "" H 2500 2600 50  0001 C CNN
+F 3 "~" H 2500 2600 50  0001 C CNN
+	1    2300 2600
+	0    1    1    0
+$EndComp
+$Comp
+L Connector:TestPoint TP?
+U 1 1 61941915
+P 2300 2700
+AR Path="/616688D6/61941915" Ref="TP?"  Part="1"
+AR Path="/61667F91/61941915" Ref="TP7"  Part="1"
+F 0 "TP7" V 2300 2900 50  0000 L CNN
+F 1 "USART1_RX" V 2300 3200 50  0000 L CNN
+F 2 "" H 2500 2700 50  0001 C CNN
+F 3 "~" H 2500 2700 50  0001 C CNN
+	1    2300 2700
+	0    1    1    0
+$EndComp
+$Comp
+L Connector:TestPoint TP?
+U 1 1 6194191B
+P 2300 2800
+AR Path="/616688D6/6194191B" Ref="TP?"  Part="1"
+AR Path="/61667F91/6194191B" Ref="TP8"  Part="1"
+F 0 "TP8" V 2300 3000 50  0000 L CNN
+F 1 "GPIO0" V 2300 3300 50  0000 L CNN
+F 2 "" H 2500 2800 50  0001 C CNN
+F 3 "~" H 2500 2800 50  0001 C CNN
+	1    2300 2800
+	0    1    1    0
+$EndComp
+$Comp
+L Connector:TestPoint TP?
+U 1 1 61941921
+P 2300 2900
+AR Path="/616688D6/61941921" Ref="TP?"  Part="1"
+AR Path="/61667F91/61941921" Ref="TP9"  Part="1"
+F 0 "TP9" V 2300 3100 50  0000 L CNN
+F 1 "GPIO1" V 2300 3400 50  0000 L CNN
+F 2 "" H 2500 2900 50  0001 C CNN
+F 3 "~" H 2500 2900 50  0001 C CNN
+	1    2300 2900
+	0    1    1    0
+$EndComp
+$Comp
+L Connector:TestPoint TP?
+U 1 1 61941927
+P 2300 3000
+AR Path="/616688D6/61941927" Ref="TP?"  Part="1"
+AR Path="/61667F91/61941927" Ref="TP10"  Part="1"
+F 0 "TP10" V 2300 3200 50  0000 L CNN
+F 1 "GPIO2" V 2300 3500 50  0000 L CNN
+F 2 "" H 2500 3000 50  0001 C CNN
+F 3 "~" H 2500 3000 50  0001 C CNN
+	1    2300 3000
+	0    1    1    0
+$EndComp
+$Comp
+L Connector:TestPoint TP?
+U 1 1 6194192D
+P 2300 3100
+AR Path="/616688D6/6194192D" Ref="TP?"  Part="1"
+AR Path="/61667F91/6194192D" Ref="TP11"  Part="1"
+F 0 "TP11" V 2300 3300 50  0000 L CNN
+F 1 "GPIO3" V 2300 3600 50  0000 L CNN
+F 2 "" H 2500 3100 50  0001 C CNN
+F 3 "~" H 2500 3100 50  0001 C CNN
+	1    2300 3100
+	0    1    1    0
+$EndComp
 $EndSCHEMATC

Commit message: finished layout of STM32 daughterboard
Parts:
- removed C8: 100n, symbol Device:C_Small
- removed TP10: GPIO2, symbol Connector:TestPoint
- removed TP11: GPIO3, symbol Connector:TestPoint
- removed TP5: NRST, symbol Connector:TestPoint
- removed TP8: GPIO0, symbol Connector:TestPoint
- removed TP9: GPIO1, symbol Connector:TestPoint
- C1, C2, C3, C4, C5, C6, C7: footprint (none) -> Capacitor_SMD:C_0603_1608Metric_Pad1.05x0.95mm_HandSolder
- JP1, JP2: footprint (none) -> Jumper:SolderJumper-2_P1.3mm_Open_TrianglePad1.0x1.5mm
- R1: footprint (none) -> Resistor_SMD:R_0603_1608Metric_Pad1.05x0.95mm_HandSolder
- TP1, TP2, TP3, TP4, TP6, TP7: footprint (none) -> TestPoint:TestPoint_Pad_1.0x1.0mm
Changed lines of the file:
@@
 F 0 "C4" H 7942 2046 50  0000 L CNN
 F 1 "100n" H 7942 1955 50  0000 L CNN
-F 2 "" H 7850 2000 50  0001 C CNN
+F 2 "Capacitor_SMD:C_0603_1608Metric_Pad1.05x0.95mm_HandSolder" H 7850 2000 50  0001 C CNN
 F 3 "~" H 7850 2000 50  0001 C CNN
 	1    7850 2000
@@
 F 0 "C5" H 8442 2046 50  0000 L CNN
 F 1 "100n" H 8442 1955 50  0000 L CNN
-F 2 "" H 8350 2000 50  0001 C CNN
+F 2 "Capacitor_SMD:C_0603_1608Metric_Pad1.05x0.95mm_HandSolder" H 8350 2000 50  0001 C CNN
 F 3 "~" H 8350 2000 50  0001 C CNN
 	1    8350 2000
@@
 F 0 "C6" H 8892 2046 50  0000 L CNN
 F 1 "100n" H 8892 1955 50  0000 L CNN
-F 2 "" H 8800 2000 50  0001 C CNN
+F 2 "Capacitor_SMD:C_0603_1608Metric_Pad1.05x0.95mm_HandSolder" H 8800 2000 50  0001 C CNN
 F 3 "~" H 8800 2000 50  0001 C CNN
 	1    8800 2000
-	1    0    0    -1
-$EndComp
-$Comp
-L Device:C_Small C?
-U 1 1 619D53B7
-P 9700 2000
-AR Path="/616688D6/619D53B7" Ref="C?"  Part="1"
-AR Path="/61668157/619D53B7" Ref="C?"  Part="1"
-AR Path="/61667F91/619D53B7" Ref="C8"  Part="1"
-F 0 "C8" H 9792 2046 50  0000 L CNN
-F 1 "100n" H 9792 1955 50  0000 L CNN
-F 2 "" H 9700 2000 50  0001 C CNN
-F 3 "~" H 9700 2000 50  0001 C CNN
-	1    9700 2000
 	1    0    0    -1
 $EndComp
@@
 F 0 "C3" H 7442 2046 50  0000 L CNN
 F 1 "4.7u" H 7442 1955 50  0000 L CNN
-F 2 "" H 7350 2000 50  0001 C CNN
+F 2 "Capacitor_SMD:C_0603_1608Metric_Pad1.05x0.95mm_HandSolder" H 7350 2000 50  0001 C CNN
 F 3 "~" H 7350 2000 50  0001 C CNN
 	1    7350 2000
@@
 $EndComp
 Wire Wire Line
-	9700 1900 9700 1750
-Wire Wire Line
 	7350 1900 7350 1750
 Connection ~ 7350 1750
@@
 Wire Wire Line
 	8350 1750 8800 1750
-Wire Wire Line
-	9250 1750 9700 1750
 $Comp
 L power:GND #PWR?
 U 1 1 619D53CF
-P 9700 2300
+P 9250 2300
 AR Path="/616688D6/619D53CF" Ref="#PWR?"  Part="1"
 AR Path="/61668157/619D53CF" Ref="#PWR?"  Part="1"
 AR Path="/61667F91/619D53CF" Ref="#PWR012"  Part="1"
-F 0 "#PWR012" H 9700 2050 50  0001 C CNN
-F 1 "GND" H 9705 2127 50  0000 C CNN
-F 2 "" H 9700 2300 50  0001 C CNN
-F 3 "" H 9700 2300 50  0001 C CNN
-	1    9700 2300
-	1    0    0    -1
-$EndComp
-Wire Wire Line
-	9700 2300 9700 2200
-Wire Wire Line
-	9700 2200 9250 2200
+F 0 "#PWR012" H 9250 2050 50  0001 C CNN
+F 1 "GND" H 9255 2127 50  0000 C CNN
+F 2 "" H 9250 2300 50  0001 C CNN
+F 3 "" H 9250 2300 50  0001 C CNN
+	1    9250 2300
+	1    0    0    -1
+$EndComp
+Wire Wire Line
+	9250 2300 9250 2200
 Wire Wire Line
 	7350 2200 7350 2100
@@
 Wire Wire Line
 	8800 2200 8350 2200
-Wire Wire Line
-	9700 2100 9700 2200
-Connection ~ 9700 2200
 $Comp
 L power:+3V3 #PWR?
 U 1 1 619D53E2
-P 9700 1600
+P 9250 1600
 AR Path="/616688D6/619D53E2" Ref="#PWR?"  Part="1"
 AR Path="/61668157/619D53E2" Ref="#PWR?"  Part="1"
 AR Path="/61667F91/619D53E2" Ref="#PWR011"  Part="1"
-F 0 "#PWR011" H 9700 1450 50  0001 C CNN
-F 1 "+3V3" H 9715 1773 50  0000 C CNN
-F 2 "" H 9700 1600 50  0001 C CNN
-F 3 "" H 9700 1600 50  0001 C CNN
-	1    9700 1600
-	1    0    0    -1
-$EndComp
-Wire Wire Line
-	9700 1600 9700 1750
-Connection ~ 9700 1750
+F 0 "#PWR011" H 9250 1450 50  0001 C CNN
+F 1 "+3V3" H 9265 1773 50  0000 C CNN
+F 2 "" H 9250 1600 50  0001 C CNN
+F 3 "" H 9250 1600 50  0001 C CNN
+	1    9250 1600
+	1    0    0    -1
+$EndComp
+Wire Wire Line
+	9250 1600 9250 1750
 $Comp
 L Device:C_Small C?
@@
 F 0 "C7" H 9342 2046 50  0000 L CNN
 F 1 "100n" H 9342 1955 50  0000 L CNN
-F 2 "" H 9250 2000 50  0001 C CNN
+F 2 "Capacitor_SMD:C_0603_1608Metric_Pad1.05x0.95mm_HandSolder" H 9250 2000 50  0001 C CNN
 F 3 "~" H 9250 2000 50  0001 C CNN
 	1    9250 2000
@@
 Wire Wire Line
 	9250 2100 9250 2200
-Wire Wire Line
-	9250 2200 8800 2200
 Connection ~ 9250 1750
-Connection ~ 9250 2200
 Wire Wire Line
 	6700 1750 7350 1750
@@
 F 0 "C2" V 5300 2800 50  0000 C CNN
 F 1 "4.7u" V 5300 2400 50  0000 C CNN
-F 2 "" H 5250 2550 50  0001 C CNN
+F 2 "Capacitor_SMD:C_0603_1608Metric_Pad1.05x0.95mm_HandSolder" H 5250 2550 50  0001 C CNN
 F 3 "~" H 5250 2550 50  0001 C CNN
 	1    5250 2550
@@
 F 0 "R1" V 5500 2100 50  0000 C CNN
 F 1 "100k" V 5500 2550 50  0000 C CNN
-F 2 "" H 5550 2350 50  0001 C CNN
+F 2 "Resistor_SMD:R_0603_1608Metric_Pad1.05x0.95mm_HandSolder" H 5550 2350 50  0001 C CNN
 F 3 "~" H 5550 2350 50  0001 C CNN
 	1    5550 2350
@@
 F 0 "JP2" H 4900 4155 50  0000 C CNN
 F 1 "NJRST1" H 4900 4064 50  0000 C CNN
-F 2 "" H 4900 3950 50  0001 C CNN
+F 2 "Jumper:SolderJumper-2_P1.3mm_Open_TrianglePad1.0x1.5mm" H 4900 3950 50  0001 C CNN
 F 3 "~" H 4900 3950 50  0001 C CNN
 	1    4900 3950
@@
 F 0 "C1" H 1042 4196 50  0000 L CNN
 F 1 "100n" H 1042 4105 50  0000 L CNN
-F 2 "" H 950 4150 50  0001 C CNN
+F 2 "Capacitor_SMD:C_0603_1608Metric_Pad1.05x0.95mm_HandSolder" H 950 4150 50  0001 C CNN
 F 3 "~" H 950 4150 50  0001 C CNN
 	1    950  4150
@@
 F 0 "JP1" V 1496 4062 50  0000 R CNN
 F 1 "NRST1" V 1405 4062 50  0000 R CNN
-F 2 "" H 1450 4150 50  0001 C CNN
+F 2 "Jumper:SolderJumper-2_P1.3mm_Open_TrianglePad1.0x1.5mm" H 1450 4150 50  0001 C CNN
 F 3 "~" H 1450 4150 50  0001 C CNN
 	1    1450 4150
@@
 F 0 "TP1" V 2300 1900 50  0000 L CNN
 F 1 "JTMS-SWDIO" V 2300 2200 50  0000 L CNN
-F 2 "" H 2500 1700 50  0001 C CNN
+F 2 "TestPoint:TestPoint_Pad_1.0x1.0mm" H 2500 1700 50  0001 C CNN
 F 3 "~" H 2500 1700 50  0001 C CNN
 	1    2300 1700
@@
 F 0 "TP2" V 2300 2000 50  0000 L CNN
 F 1 "JTCK-SWCLK" V 2300 2300 50  0000 L CNN
-F 2 "" H 2500 1800 50  0001 C CNN
+F 2 "TestPoint:TestPoint_Pad_1.0x1.0mm" H 2500 1800 50  0001 C CNN
 F 3 "~" H 2500 1800 50  0001 C CNN
 	1    2300 1800
@@
 F 0 "TP3" V 2300 2100 50  0000 L CNN
 F 1 "JTDO-SWO" V 2300 2400 50  0000 L CNN
-F 2 "" H 2500 1900 50  0001 C CNN
+F 2 "TestPoint:TestPoint_Pad_1.0x1.0mm" H 2500 1900 50  0001 C CNN
 F 3 "~" H 2500 1900 50  0001 C CNN
 	1    2300 1900
@@
 F 0 "TP4" V 2300 2200 50  0000 L CNN
 F 1 "JTDI" V 2300 2500 50  0000 L CNN
-F 2 "" H 2500 2000 50  0001 C CNN
+F 2 "TestPoint:TestPoint_Pad_1.0x1.0mm" H 2500 2000 50  0001 C CNN
 F 3 "~" H 2500 2000 50  0001 C CNN
 	1    2300 2000
-	0    1    1    0
-$EndComp
-$Comp
-L Connector:TestPoint TP?
-U 1 1 61941909
-P 2300 2100
-AR Path="/616688D6/61941909" Ref="TP?"  Part="1"
-AR Path="/61667F91/61941909" Ref="TP5"  Part="1"
-F 0 "TP5" V 2300 2300 50  0000 L CNN
-F 1 "NRST" V 2300 2600 50  0000 L CNN
-F 2 "" H 2500 2100 50  0001 C CNN
-F 3 "~" H 2500 2100 50  0001 C CNN
-	1    2300 2100
 	0    1    1    0
 $EndComp
@@
 F 0 "TP6" V 2300 2800 50  0000 L CNN
 F 1 "USART1_TX" V 2300 3100 50  0000 L CNN
-F 2 "" H 2500 2600 50  0001 C CNN
+F 2 "TestPoint:TestPoint_Pad_1.0x1.0mm" H 2500 2600 50  0001 C CNN
 F 3 "~" H 2500 2600 50  0001 C CNN
 	1    2300 2600
@@
 F 0 "TP7" V 2300 2900 50  0000 L CNN
 F 1 "USART1_RX" V 2300 3200 50  0000 L CNN
-F 2 "" H 2500 2700 50  0001 C CNN
+F 2 "TestPoint:TestPoint_Pad_1.0x1.0mm" H 2500 2700 50  0001 C CNN
 F 3 "~" H 2500 2700 50  0001 C CNN
 	1    2300 2700
 	0    1    1    0
 $EndComp
-$Comp
-L Connector:TestPoint TP?
-U 1 1 6194191B
-P 2300 2800
-AR Path="/616688D6/6194191B" Ref="TP?"  Part="1"
-AR Path="/61667F91/6194191B" Ref="TP8"  Part="1"
-F 0 "TP8" V 2300 3000 50  0000 L CNN
-F 1 "GPIO0" V 2300 3300 50  0000 L CNN
-F 2 "" H 2500 2800 50  0001 C CNN
-F 3 "~" H 2500 2800 50  0001 C CNN
-	1    2300 2800
-	0    1    1    0
-$EndComp
-$Comp
-L Connector:TestPoint TP?
-U 1 1 61941921
-P 2300 2900
-AR Path="/616688D6/61941921" Ref="TP?"  Part="1"
-AR Path="/61667F91/61941921" Ref="TP9"  Part="1"
-F 0 "TP9" V 2300 3100 50  0000 L CNN
-F 1 "GPIO1" V 2300 3400 50  0000 L CNN
-F 2 "" H 2500 2900 50  0001 C CNN
-F 3 "~" H 2500 2900 50  0001 C CNN
-	1    2300 2900
-	0    1    1    0
-$EndComp
-$Comp
-L Connector:TestPoint TP?
-U 1 1 61941927
-P 2300 3000
-AR Path="/616688D6/61941927" Ref="TP?"  Part="1"
-AR Path="/61667F91/61941927" Ref="TP10"  Part="1"
-F 0 "TP10" V 2300 3200 50  0000 L CNN
-F 1 "GPIO2" V 2300 3500 50  0000 L CNN
-F 2 "" H 2500 3000 50  0001 C CNN
-F 3 "~" H 2500 3000 50  0001 C CNN
-	1    2300 3000
-	0    1    1    0
-$EndComp
-$Comp
-L Connector:TestPoint TP?
-U 1 1 6194192D
-P 2300 3100
-AR Path="/616688D6/6194192D" Ref="TP?"  Part="1"
-AR Path="/61667F91/6194192D" Ref="TP11"  Part="1"
-F 0 "TP11" V 2300 3300 50  0000 L CNN
-F 1 "GPIO3" V 2300 3600 50  0000 L CNN
-F 2 "" H 2500 3100 50  0001 C CNN
-F 3 "~" H 2500 3100 50  0001 C CNN
-	1    2300 3100
-	0    1    1    0
-$EndComp
+Connection ~ 9250 2200
+Wire Wire Line
+	8800 2200 9250 2200
 $EndSCHEMATC
