File: daughterboard/STM32_00/target2.sch (KiCad schematic (older format))
At the start: 10 parts, among them U2 STM32L151C8TxA

Commit message: added testpoints to daughterboards, updated readme
Parts:
- added TP22: JTMS-SWDIO, symbol Connector:TestPoint
- added TP23: JTCK-SWCLK, symbol Connector:TestPoint
- added TP24: JTDO-SWO, symbol Connector:TestPoint
- added TP25: JTDI, symbol Connector:TestPoint
- added TP26: NRST, symbol Connector:TestPoint
- added TP27: USART1_TX, symbol Connector:TestPoint
- added TP28: USART1_RX, symbol Connector:TestPoint
- added TP29: GPIO0, symbol Connector:TestPoint
- added TP30: GPIO1, symbol Connector:TestPoint
- added TP31: GPIO2, symbol Connector:TestPoint
- added TP32: GPIO3, symbol Connector:TestPoint
Connections:
- net GPIO2.0: now also TP29.1
- net GPIO2.1: now also TP30.1
- net GPIO2.2: now also TP31.1
- net GPIO2.3: now also TP32.1
- net RST_2: now also TP26.1
- net TCK|SWDCLK_2: now also TP23.1
- net TDI|NC_2: now also TP25.1
- net TDO|SWO_2: now also TP24.1
- net TMS|SWDIO_2: now also TP22.1
- net UART_RxD2: now also TP27.1
- net UART_TxD2: now also TP28.1
Changed lines of the file:
@@
 JTCK-SWCLK
 Wire Wire Line
-	1650 2700 2200 2700
-Text Label 2200 2700 2    50   ~ 0
+	1650 2700 2350 2700
+Text Label 2350 2700 2    50   ~ 0
 USART1_RX
 Wire Wire Line
-	1650 2600 2200 2600
-Text Label 2200 2600 2    50   ~ 0
+	1650 2600 2350 2600
+Text Label 2350 2600 2    50   ~ 0
 USART1_TX
 Wire Wire Line
-	1650 2100 2200 2100
-Text Label 2200 2100 2    50   ~ 0
+	1650 2100 2350 2100
+Text Label 2350 2100 2    50   ~ 0
 NRST
 Wire Wire Line
-	1650 1900 2200 1900
-Text Label 2200 2000 2    50   ~ 0
+	1650 1900 2350 1900
+Text Label 2350 2000 2    50   ~ 0
 JTDI
 Wire Wire Line
-	2200 2000 1650 2000
-Text Label 2200 1900 2    50   ~ 0
+	2350 2000 1650 2000
+Text Label 2350 1900 2    50   ~ 0
 JTDO-SWO
 Wire Wire Line
-	1650 2800 2200 2800
-Text Label 2200 2800 2    50   ~ 0
+	1650 2800 2350 2800
+Text Label 2350 2800 2    50   ~ 0
 GPIO0
 Wire Wire Line
-	1650 2900 2200 2900
-Text Label 2200 2900 2    50   ~ 0
+	1650 2900 2350 2900
+Text Label 2350 2900 2    50   ~ 0
 GPIO1
 Wire Wire Line
-	1650 3000 2200 3000
-Text Label 2200 3000 2    50   ~ 0
+	1650 3000 2350 3000
+Text Label 2350 3000 2    50   ~ 0
 GPIO2
 Wire Wire Line
-	1650 3100 2200 3100
-Text Label 2200 3100 2    50   ~ 0
+	1650 3100 2350 3100
+Text Label 2350 3100 2    50   ~ 0
 GPIO3
 Text Label 7800 4850 2    50   ~ 0
@@
 Wire Wire Line
 	7400 4650 7250 4650
+$Comp
+L Connector:TestPoint TP22
+U 1 1 61913CA5
+P 2350 1700
+F 0 "TP22" V 2350 1900 50  0000 L CNN
+F 1 "JTMS-SWDIO" V 2350 2200 50  0000 L CNN
+F 2 "" H 2550 1700 50  0001 C CNN
+F 3 "~" H 2550 1700 50  0001 C CNN
+	1    2350 1700
+	0    1    1    0
+$EndComp
+$Comp
+L Connector:TestPoint TP23
+U 1 1 619159C5
+P 2350 1800
+F 0 "TP23" V 2350 2000 50  0000 L CNN
+F 1 "JTCK-SWCLK" V 2350 2300 50  0000 L CNN
+F 2 "" H 2550 1800 50  0001 C CNN
+F 3 "~" H 2550 1800 50  0001 C CNN
+	1    2350 1800
+	0    1    1    0
+$EndComp
+$Comp
+L Connector:TestPoint TP24
+U 1 1 61915BF9
+P 2350 1900
+F 0 "TP24" V 2350 2100 50  0000 L CNN
+F 1 "JTDO-SWO" V 2350 2400 50  0000 L CNN
+F 2 "" H 2550 1900 50  0001 C CNN
+F 3 "~" H 2550 1900 50  0001 C CNN
+	1    2350 1900
+	0    1    1    0
+$EndComp
+$Comp
+L Connector:TestPoint TP25
+U 1 1 61915F15
+P 2350 2000
+F 0 "TP25" V 2350 2200 50  0000 L CNN
+F 1 "JTDI" V 2350 2500 50  0000 L CNN
+F 2 "" H 2550 2000 50  0001 C CNN
+F 3 "~" H 2550 2000 50  0001 C CNN
+	1    2350 2000
+	0    1    1    0
+$EndComp
+$Comp
+L Connector:TestPoint TP26
+U 1 1 61916127
+P 2350 2100
+F 0 "TP26" V 2350 2300 50  0000 L CNN
+F 1 "NRST" V 2350 2600 50  0000 L CNN
+F 2 "" H 2550 2100 50  0001 C CNN
+F 3 "~" H 2550 2100 50  0001 C CNN
+	1    2350 2100
+	0    1    1    0
+$EndComp
+$Comp
+L Connector:TestPoint TP27
+U 1 1 61916482
+P 2350 2600
+F 0 "TP27" V 2350 2800 50  0000 L CNN
+F 1 "USART1_TX" V 2350 3100 50  0000 L CNN
+F 2 "" H 2550 2600 50  0001 C CNN
+F 3 "~" H 2550 2600 50  0001 C CNN
+	1    2350 2600
+	0    1    1    0
+$EndComp
+$Comp
+L Connector:TestPoint TP28
+U 1 1 61916984
+P 2350 2700
+F 0 "TP28" V 2350 2900 50  0000 L CNN
+F 1 "USART1_RX" V 2350 3200 50  0000 L CNN
+F 2 "" H 2550 2700 50  0001 C CNN
+F 3 "~" H 2550 2700 50  0001 C CNN
+	1    2350 2700
+	0    1    1    0
+$EndComp
+$Comp
+L Connector:TestPoint TP29
+U 1 1 61916C76
+P 2350 2800
+F 0 "TP29" V 2350 3000 50  0000 L CNN
+F 1 "GPIO0" V 2350 3300 50  0000 L CNN
+F 2 "" H 2550 2800 50  0001 C CNN
+F 3 "~" H 2550 2800 50  0001 C CNN
+	1    2350 2800
+	0    1    1    0
+$EndComp
+$Comp
+L Connector:TestPoint TP30
+U 1 1 6191730D
+P 2350 2900
+F 0 "TP30" V 2350 3100 50  0000 L CNN
+F 1 "GPIO1" V 2350 3400 50  0000 L CNN
+F 2 "" H 2550 2900 50  0001 C CNN
+F 3 "~" H 2550 2900 50  0001 C CNN
+	1    2350 2900
+	0    1    1    0
+$EndComp
+$Comp
+L Connector:TestPoint TP31
+U 1 1 61917564
+P 2350 3000
+F 0 "TP31" V 2350 3200 50  0000 L CNN
+F 1 "GPIO2" V 2350 3500 50  0000 L CNN
+F 2 "" H 2550 3000 50  0001 C CNN
+F 3 "~" H 2550 3000 50  0001 C CNN
+	1    2350 3000
+	0    1    1    0
+$EndComp
+$Comp
+L Connector:TestPoint TP32
+U 1 1 619179D0
+P 2350 3100
+F 0 "TP32" V 2350 3300 50  0000 L CNN
+F 1 "GPIO3" V 2350 3600 50  0000 L CNN
+F 2 "" H 2550 3100 50  0001 C CNN
+F 3 "~" H 2550 3100 50  0001 C CNN
+	1    2350 3100
+	0    1    1    0
+$EndComp
 $EndSCHEMATC

Commit message: finished layout of STM32 daughterboard
Parts:
- removed C17: 100n, symbol Device:C_Small
- removed TP26: NRST, symbol Connector:TestPoint
- removed TP29: GPIO0, symbol Connector:TestPoint
- removed TP30: GPIO1, symbol Connector:TestPoint
- removed TP31: GPIO2, symbol Connector:TestPoint
- removed TP32: GPIO3, symbol Connector:TestPoint
- C12, C13, C14, C15, C16: footprint (none) -> Capacitor_SMD:C_0603_1608Metric_Pad1.05x0.95mm_HandSolder
- JP4, JP5: footprint (none) -> Jumper:SolderJumper-2_P1.3mm_Open_TrianglePad1.0x1.5mm
- R4: footprint (none) -> Resistor_SMD:R_0603_1608Metric_Pad1.05x0.95mm_HandSolder
- TP22, TP23, TP24, TP25, TP27, TP28: footprint (none) -> TestPoint:TestPoint_Pad_1.0x1.0mm
Changed lines of the file:
@@
 F 0 "C14" H 8092 2046 50  0000 L CNN
 F 1 "100n" H 8092 1955 50  0000 L CNN
-F 2 "" H 8000 2000 50  0001 C CNN
+F 2 "Capacitor_SMD:C_0603_1608Metric_Pad1.05x0.95mm_HandSolder" H 8000 2000 50  0001 C CNN
 F 3 "~" H 8000 2000 50  0001 C CNN
 	1    8000 2000
@@
 F 0 "C15" H 8592 2046 50  0000 L CNN
 F 1 "100n" H 8592 1955 50  0000 L CNN
-F 2 "" H 8500 2000 50  0001 C CNN
+F 2 "Capacitor_SMD:C_0603_1608Metric_Pad1.05x0.95mm_HandSolder" H 8500 2000 50  0001 C CNN
 F 3 "~" H 8500 2000 50  0001 C CNN
 	1    8500 2000
@@
 F 0 "C16" H 9042 2046 50  0000 L CNN
 F 1 "100n" H 9042 1955 50  0000 L CNN
-F 2 "" H 8950 2000 50  0001 C CNN
+F 2 "Capacitor_SMD:C_0603_1608Metric_Pad1.05x0.95mm_HandSolder" H 8950 2000 50  0001 C CNN
 F 3 "~" H 8950 2000 50  0001 C CNN
 	1    8950 2000
-	1    0    0    -1
-$EndComp
-$Comp
-L Device:C_Small C17
-U 1 1 618B3EC4
-P 9400 2000
-F 0 "C17" H 9492 2046 50  0000 L CNN
-F 1 "100n" H 9492 1955 50  0000 L CNN
-F 2 "" H 9400 2000 50  0001 C CNN
-F 3 "~" H 9400 2000 50  0001 C CNN
-	1    9400 2000
 	1    0    0    -1
 $EndComp
@@
 F 0 "C13" H 7592 2046 50  0000 L CNN
 F 1 "10u" H 7592 1955 50  0000 L CNN
-F 2 "" H 7500 2000 50  0001 C CNN
+F 2 "Capacitor_SMD:C_0603_1608Metric_Pad1.05x0.95mm_HandSolder" H 7500 2000 50  0001 C CNN
 F 3 "~" H 7500 2000 50  0001 C CNN
 	1    7500 2000
@@
 NoConn ~ 6050 2650
 Wire Wire Line
-	9400 1900 9400 1750
-Wire Wire Line
 	6550 1750 6550 2050
 Wire Wire Line
@@
 	8500 1750 8950 1750
 Connection ~ 8950 1750
-Wire Wire Line
-	8950 1750 9400 1750
 $Comp
 L power:GND #PWR0132
 U 1 1 618BB360
-P 9400 2300
-F 0 "#PWR0132" H 9400 2050 50  0001 C CNN
-F 1 "GND" H 9405 2127 50  0000 C CNN
-F 2 "" H 9400 2300 50  0001 C CNN
-F 3 "" H 9400 2300 50  0001 C CNN
-	1    9400 2300
-	1    0    0    -1
-$EndComp
-Wire Wire Line
-	9400 2300 9400 2200
-Wire Wire Line
-	9400 2200 8950 2200
+P 8950 2300
+F 0 "#PWR0132" H 8950 2050 50  0001 C CNN
+F 1 "GND" H 8955 2127 50  0000 C CNN
+F 2 "" H 8950 2300 50  0001 C CNN
+F 3 "" H 8950 2300 50  0001 C CNN
+	1    8950 2300
+	1    0    0    -1
+$EndComp
+Wire Wire Line
+	8950 2300 8950 2200
 Wire Wire Line
 	7500 2200 7500 2100
@@
 Wire Wire Line
 	8950 2200 8500 2200
-Wire Wire Line
-	9400 2100 9400 2200
-Connection ~ 9400 2200
 $Comp
 L power:+3V3 #PWR0133
 U 1 1 618BD70C
-P 9400 1600
-F 0 "#PWR0133" H 9400 1450 50  0001 C CNN
-F 1 "+3V3" H 9415 1773 50  0000 C CNN
-F 2 "" H 9400 1600 50  0001 C CNN
-F 3 "" H 9400 1600 50  0001 C CNN
-	1    9400 1600
-	1    0    0    -1
-$EndComp
-Wire Wire Line
-	9400 1600 9400 1750
-Connection ~ 9400 1750
+P 8950 1600
+F 0 "#PWR0133" H 8950 1450 50  0001 C CNN
+F 1 "+3V3" H 8965 1773 50  0000 C CNN
+F 2 "" H 8950 1600 50  0001 C CNN
+F 3 "" H 8950 1600 50  0001 C CNN
+	1    8950 1600
+	1    0    0    -1
+$EndComp
+Wire Wire Line
+	8950 1600 8950 1750
 $Comp
 L power:GND #PWR0134
@@
 F 0 "R4" V 5896 2450 50  0000 C CNN
 F 1 "100k" V 5805 2450 50  0000 C CNN
-F 2 "" H 5700 2450 50  0001 C CNN
+F 2 "Resistor_SMD:R_0603_1608Metric_Pad1.05x0.95mm_HandSolder" H 5700 2450 50  0001 C CNN
 F 3 "~" H 5700 2450 50  0001 C CNN
 	1    5700 2450
@@
 F 0 "JP5" H 5050 4155 50  0000 C CNN
 F 1 "NJRST2" H 5050 4064 50  0000 C CNN
-F 2 "" H 5050 3950 50  0001 C CNN
+F 2 "Jumper:SolderJumper-2_P1.3mm_Open_TrianglePad1.0x1.5mm" H 5050 3950 50  0001 C CNN
 F 3 "~" H 5050 3950 50  0001 C CNN
 	1    5050 3950
@@
 F 0 "C12" H 1092 4746 50  0000 L CNN
 F 1 "100n" H 1092 4655 50  0000 L CNN
-F 2 "" H 1000 4700 50  0001 C CNN
+F 2 "Capacitor_SMD:C_0603_1608Metric_Pad1.05x0.95mm_HandSolder" H 1000 4700 50  0001 C CNN
 F 3 "~" H 1000 4700 50  0001 C CNN
 	1    1000 4700
@@
 F 0 "JP4" V 1546 4612 50  0000 R CNN
 F 1 "NRST2" V 1455 4612 50  0000 R CNN
-F 2 "" H 1500 4700 50  0001 C CNN
+F 2 "Jumper:SolderJumper-2_P1.3mm_Open_TrianglePad1.0x1.5mm" H 1500 4700 50  0001 C CNN
 F 3 "~" H 1500 4700 50  0001 C CNN
 	1    1500 4700
@@
 F 0 "TP22" V 2350 1900 50  0000 L CNN
 F 1 "JTMS-SWDIO" V 2350 2200 50  0000 L CNN
-F 2 "" H 2550 1700 50  0001 C CNN
+F 2 "TestPoint:TestPoint_Pad_1.0x1.0mm" H 2550 1700 50  0001 C CNN
 F 3 "~" H 2550 1700 50  0001 C CNN
 	1    2350 1700
@@
 F 0 "TP23" V 2350 2000 50  0000 L CNN
 F 1 "JTCK-SWCLK" V 2350 2300 50  0000 L CNN
-F 2 "" H 2550 1800 50  0001 C CNN
+F 2 "TestPoint:TestPoint_Pad_1.0x1.0mm" H 2550 1800 50  0001 C CNN
 F 3 "~" H 2550 1800 50  0001 C CNN
 	1    2350 1800
@@
 F 0 "TP24" V 2350 2100 50  0000 L CNN
 F 1 "JTDO-SWO" V 2350 2400 50  0000 L CNN
-F 2 "" H 2550 1900 50  0001 C CNN
+F 2 "TestPoint:TestPoint_Pad_1.0x1.0mm" H 2550 1900 50  0001 C CNN
 F 3 "~" H 2550 1900 50  0001 C CNN
 	1    2350 1900
@@
 F 0 "TP25" V 2350 2200 50  0000 L CNN
 F 1 "JTDI" V 2350 2500 50  0000 L CNN
-F 2 "" H 2550 2000 50  0001 C CNN
+F 2 "TestPoint:TestPoint_Pad_1.0x1.0mm" H 2550 2000 50  0001 C CNN
 F 3 "~" H 2550 2000 50  0001 C CNN
 	1    2350 2000
-	0    1    1    0
-$EndComp
-$Comp
-L Connector:TestPoint TP26
-U 1 1 61916127
-P 2350 2100
-F 0 "TP26" V 2350 2300 50  0000 L CNN
-F 1 "NRST" V 2350 2600 50  0000 L CNN
-F 2 "" H 2550 2100 50  0001 C CNN
-F 3 "~" H 2550 2100 50  0001 C CNN
-	1    2350 2100
 	0    1    1    0
 $EndComp
@@
 F 0 "TP27" V 2350 2800 50  0000 L CNN
 F 1 "USART1_TX" V 2350 3100 50  0000 L CNN
-F 2 "" H 2550 2600 50  0001 C CNN
+F 2 "TestPoint:TestPoint_Pad_1.0x1.0mm" H 2550 2600 50  0001 C CNN
 F 3 "~" H 2550 2600 50  0001 C CNN
 	1    2350 2600
@@
 F 0 "TP28" V 2350 2900 50  0000 L CNN
 F 1 "USART1_RX" V 2350 3200 50  0000 L CNN
-F 2 "" H 2550 2700 50  0001 C CNN
+F 2 "TestPoint:TestPoint_Pad_1.0x1.0mm" H 2550 2700 50  0001 C CNN
 F 3 "~" H 2550 2700 50  0001 C CNN
 	1    2350 2700
 	0    1    1    0
 $EndComp
-$Comp
-L Connector:TestPoint TP29
-U 1 1 61916C76
-P 2350 2800
-F 0 "TP29" V 2350 3000 50  0000 L CNN
-F 1 "GPIO0" V 2350 3300 50  0000 L CNN
-F 2 "" H 2550 2800 50  0001 C CNN
-F 3 "~" H 2550 2800 50  0001 C CNN
-	1    2350 2800
-	0    1    1    0
-$EndComp
-$Comp
-L Connector:TestPoint TP30
-U 1 1 6191730D
-P 2350 2900
-F 0 "TP30" V 2350 3100 50  0000 L CNN
-F 1 "GPIO1" V 2350 3400 50  0000 L CNN
-F 2 "" H 2550 2900 50  0001 C CNN
-F 3 "~" H 2550 2900 50  0001 C CNN
-	1    2350 2900
-	0    1    1    0
-$EndComp
-$Comp
-L Connector:TestPoint TP31
-U 1 1 61917564
-P 2350 3000
-F 0 "TP31" V 2350 3200 50  0000 L CNN
-F 1 "GPIO2" V 2350 3500 50  0000 L CNN
-F 2 "" H 2550 3000 50  0001 C CNN
-F 3 "~" H 2550 3000 50  0001 C CNN
-	1    2350 3000
-	0    1    1    0
-$EndComp
-$Comp
-L Connector:TestPoint TP32
-U 1 1 619179D0
-P 2350 3100
-F 0 "TP32" V 2350 3300 50  0000 L CNN
-F 1 "GPIO3" V 2350 3600 50  0000 L CNN
-F 2 "" H 2550 3100 50  0001 C CNN
-F 3 "~" H 2550 3100 50  0001 C CNN
-	1    2350 3100
-	0    1    1    0
-$EndComp
