File: daughterboard/LPC_00/target0.sch (KiCad schematic (older format))
At the start: 9 parts

Commit message: finished LPC Daughterboard schematics
Parts:
- gave numbers to parts that had none: 9
Changed lines of the file:
@@
 RESETN
 $Comp
-L Device:R_Small R?
+L Device:R_Small R4
 U 1 1 619E8148
 P 900 4450
-F 0 "R?" H 959 4496 50  0000 L CNN
+F 0 "R4" H 959 4496 50  0000 L CNN
 F 1 "100k" H 959 4405 50  0000 L CNN
 F 2 "" H 900 4450 50  0001 C CNN
@@
 $EndComp
 $Comp
-L power:+3V3 #PWR?
+L power:+3V3 #PWR08
 U 1 1 619E814E
 P 900 4700
-F 0 "#PWR?" H 900 4550 50  0001 C CNN
+F 0 "#PWR08" H 900 4550 50  0001 C CNN
 F 1 "+3V3" H 915 4873 50  0000 C CNN
 F 2 "" H 900 4700 50  0001 C CNN
@@
 P 1550 4450
 AR Path="/616688D6/619E8156" Ref="JP?"  Part="1"
-AR Path="/61668514/619E8156" Ref="JP?"  Part="1"
-F 0 "JP?" V 1504 4518 50  0000 L CNN
+AR Path="/61668514/619E8156" Ref="JP2"  Part="1"
+F 0 "JP2" V 1504 4518 50  0000 L CNN
 F 1 "NRST" V 1595 4518 50  0000 L CNN
 F 2 "" H 1550 4450 50  0001 C CNN
@@
 	900  4050 900  4350
 $Comp
-L power:GND #PWR?
+L power:GND #PWR09
 U 1 1 619E8160
 P 1550 4700
-F 0 "#PWR?" H 1550 4450 50  0001 C CNN
+F 0 "#PWR09" H 1550 4450 50  0001 C CNN
 F 1 "GND" H 1555 4527 50  0000 C CNN
 F 2 "" H 1550 4700 50  0001 C CNN
@@
 SWCLK
 $Comp
-L Device:R_Small R?
+L Device:R_Small R5
 U 1 1 619E816A
 P 2150 4400
-F 0 "R?" H 2209 4446 50  0000 L CNN
+F 0 "R5" H 2209 4446 50  0000 L CNN
 F 1 "10k" H 2209 4355 50  0000 L CNN
 F 2 "" H 2150 4400 50  0001 C CNN
@@
 $EndComp
 $Comp
-L Device:R_Small R?
+L Device:R_Small R6
 U 1 1 619E8176
 P 2600 4400
-F 0 "R?" H 2659 4446 50  0000 L CNN
+F 0 "R6" H 2659 4446 50  0000 L CNN
 F 1 "10k" H 2659 4355 50  0000 L CNN
 F 2 "" H 2600 4400 50  0001 C CNN
@@
 	2150 3450 2150 4300
 $Comp
-L power:+3V3 #PWR?
+L power:+3V3 #PWR010
 U 1 1 619E817F
 P 2150 4650
-F 0 "#PWR?" H 2150 4500 50  0001 C CNN
+F 0 "#PWR010" H 2150 4500 50  0001 C CNN
 F 1 "+3V3" H 2165 4823 50  0000 C CNN
 F 2 "" H 2150 4650 50  0001 C CNN
@@
 P 2600 4650
 AR Path="/616688D6/619E818B" Ref="#PWR?"  Part="1"
-AR Path="/61668514/619E818B" Ref="#PWR?"  Part="1"
-F 0 "#PWR?" H 2600 4400 50  0001 C CNN
+AR Path="/61668514/619E818B" Ref="#PWR011"  Part="1"
+F 0 "#PWR011" H 2600 4400 50  0001 C CNN
 F 1 "GND" H 2605 4477 50  0000 C CNN
 F 2 "" H 2600 4650 50  0001 C CNN
@@
 P 7000 4400
 AR Path="/616688D6/619E957B" Ref="#PWR?"  Part="1"
-AR Path="/61668514/619E957B" Ref="#PWR?"  Part="1"
-F 0 "#PWR?" H 7000 4150 50  0001 C CNN
+AR Path="/61668514/619E957B" Ref="#PWR013"  Part="1"
+F 0 "#PWR013" H 7000 4150 50  0001 C CNN
 F 1 "GND" H 7005 4227 50  0000 C CNN
 F 2 "" H 7000 4400 50  0001 C CNN
@@
 Connection ~ 7000 4300
 $Comp
-L Device:C_Small C?
+L Device:C_Small C5
 U 1 1 619EA817
 P 7900 1550
-F 0 "C?" H 7992 1596 50  0000 L CNN
+F 0 "C5" H 7992 1596 50  0000 L CNN
 F 1 "100n" H 7992 1505 50  0000 L CNN
 F 2 "" H 7900 1550 50  0001 C CNN
@@
 $EndComp
 $Comp
-L Device:C_Small C?
+L Device:C_Small C6
 U 1 1 619ECAC7
 P 8300 1550
-F 0 "C?" H 8392 1596 50  0000 L CNN
+F 0 "C6" H 8392 1596 50  0000 L CNN
 F 1 "100n" H 8392 1505 50  0000 L CNN
 F 2 "" H 8300 1550 50  0001 C CNN
@@
 $EndComp
 $Comp
-L Device:C_Small C?
+L Device:C_Small C4
 U 1 1 619EEE66
 P 7400 1550
-F 0 "C?" H 7492 1596 50  0000 L CNN
+F 0 "C4" H 7492 1596 50  0000 L CNN
 F 1 "4.7u" H 7492 1505 50  0000 L CNN
 F 2 "" H 7400 1550 50  0001 C CNN
@@
 P 8300 1850
 AR Path="/616688D6/619F0EBB" Ref="#PWR?"  Part="1"
-AR Path="/61668514/619F0EBB" Ref="#PWR?"  Part="1"
-F 0 "#PWR?" H 8300 1600 50  0001 C CNN
+AR Path="/61668514/619F0EBB" Ref="#PWR014"  Part="1"
+F 0 "#PWR014" H 8300 1600 50  0001 C CNN
 F 1 "GND" H 8305 1677 50  0000 C CNN
 F 2 "" H 8300 1850 50  0001 C CNN
@@
 SWCLK-TCLK
 $Comp
-L hive_daughterboard:LPC845M301JHI33Y U?
+L hive_daughterboard:LPC845M301JHI33Y U0
 U 1 1 619D8987
 P 6850 2700
-F 0 "U?" H 6850 2000 50  0000 C CNN
+F 0 "U0" H 6850 2000 50  0000 C CNN
 F 1 "LPC845M301JHI33Y" H 6850 2100 50  0000 C CNN
 F 2 "QFN50P500X500X85-33N-D" H 9150 3500 50  0001 L CNN
@@
 P 4250 2800
 AR Path="/616688D6/619FD73A" Ref="JP?"  Part="1"
-AR Path="/61668514/619FD73A" Ref="JP?"  Part="1"
-F 0 "JP?" H 4500 2750 50  0000 C CNN
+AR Path="/61668514/619FD73A" Ref="JP3"  Part="1"
+F 0 "JP3" H 4500 2750 50  0000 C CNN
 F 1 "NJRST" H 4000 2750 50  0000 C CNN
 F 2 "" H 4250 2800 50  0001 C CNN
@@
 P 3900 2800
 AR Path="/616688D6/61A00138" Ref="#PWR?"  Part="1"
-AR Path="/61668514/61A00138" Ref="#PWR?"  Part="1"
-F 0 "#PWR?" H 3900 2550 50  0001 C CNN
+AR Path="/61668514/61A00138" Ref="#PWR012"  Part="1"
+F 0 "#PWR012" H 3900 2550 50  0001 C CNN
 F 1 "GND" V 3905 2672 50  0000 R CNN
 F 2 "" H 3900 2800 50  0001 C CNN
