File: daughterboard/LPC_00/target0.sch (KiCad schematic (older format))
At the start: 9 parts, among them U0 LPC845M301JHI33Y

Commit message: ERC on daughterboards
Connections:
- net SWCLK is gone; now on net TCK|SWDCLK_0: R6.1
- net SWDIO is gone; now on net TMS|SWDIO_0: R5.1
Changed lines of the file:
@@
 	1550 4700 1550 4600
 Text Label 2150 3450 3    50   ~ 0
-SWDIO
+SWDIO-TMS
 Text Label 2600 3450 3    50   ~ 0
-SWCLK
+SWCLK-TCLK
 $Comp
 L Device:R_Small R5

Commit message: added testpoints to daughterboards, updated readme
Parts:
- added TP11: SWDIO-TMS, symbol Connector:TestPoint
- added TP12: SWCLK-TCLK, symbol Connector:TestPoint
- added TP13: TDO, symbol Connector:TestPoint
- added TP14: TDI, symbol Connector:TestPoint
- added TP15: RESETN, symbol Connector:TestPoint
- added TP16: USART_TX, symbol Connector:TestPoint
- added TP17: USART_RX, symbol Connector:TestPoint
- added TP18: GPIO0, symbol Connector:TestPoint
- added TP19: GPIO1, symbol Connector:TestPoint
- added TP20: GPIO2, symbol Connector:TestPoint
- added TP21: GPIO3, symbol Connector:TestPoint
Connections:
- net GPIO0.0: now also TP18.1
- net GPIO0.1: now also TP19.1
- net GPIO0.2: now also TP20.1
- net GPIO0.3: now also TP21.1
- net RST_0: now also TP15.1
- net TCK|SWDCLK_0: now also TP12.1
- net TDI|NC_0: now also TP14.1
- net TDO|SWO_0: now also TP13.1
- net TMS|SWDIO_0: now also TP11.1
- net UART_RxD0: now also TP16.1
- net UART_TxD0: now also TP17.1
Changed lines of the file:
@@
 NoConn ~ 8550 3300
 NoConn ~ 8550 3800
+$Comp
+L Connector:TestPoint TP?
+U 1 1 6191611D
+P 2250 1650
+AR Path="/616688D6/6191611D" Ref="TP?"  Part="1"
+AR Path="/61668514/6191611D" Ref="TP11"  Part="1"
+F 0 "TP11" V 2250 1850 50  0000 L CNN
+F 1 "SWDIO-TMS" V 2250 2200 50  0000 L CNN
+F 2 "" H 2450 1650 50  0001 C CNN
+F 3 "~" H 2450 1650 50  0001 C CNN
+	1    2250 1650
+	0    1    1    0
+$EndComp
+$Comp
+L Connector:TestPoint TP?
+U 1 1 61916123
+P 2250 1750
+AR Path="/616688D6/61916123" Ref="TP?"  Part="1"
+AR Path="/61668514/61916123" Ref="TP12"  Part="1"
+F 0 "TP12" V 2250 1950 50  0000 L CNN
+F 1 "SWCLK-TCLK" V 2250 2300 50  0000 L CNN
+F 2 "" H 2450 1750 50  0001 C CNN
+F 3 "~" H 2450 1750 50  0001 C CNN
+	1    2250 1750
+	0    1    1    0
+$EndComp
+$Comp
+L Connector:TestPoint TP?
+U 1 1 61916129
+P 2250 1850
+AR Path="/616688D6/61916129" Ref="TP?"  Part="1"
+AR Path="/61668514/61916129" Ref="TP13"  Part="1"
+F 0 "TP13" V 2250 2050 50  0000 L CNN
+F 1 "TDO" V 2250 2400 50  0000 L CNN
+F 2 "" H 2450 1850 50  0001 C CNN
+F 3 "~" H 2450 1850 50  0001 C CNN
+	1    2250 1850
+	0    1    1    0
+$EndComp
+$Comp
+L Connector:TestPoint TP?
+U 1 1 6191612F
+P 2250 2050
+AR Path="/616688D6/6191612F" Ref="TP?"  Part="1"
+AR Path="/61668514/6191612F" Ref="TP15"  Part="1"
+F 0 "TP15" V 2250 2250 50  0000 L CNN
+F 1 "RESETN" V 2250 2600 50  0000 L CNN
+F 2 "" H 2450 2050 50  0001 C CNN
+F 3 "~" H 2450 2050 50  0001 C CNN
+	1    2250 2050
+	0    1    1    0
+$EndComp
+$Comp
+L Connector:TestPoint TP?
+U 1 1 61916135
+P 2250 2550
+AR Path="/616688D6/61916135" Ref="TP?"  Part="1"
+AR Path="/61668514/61916135" Ref="TP16"  Part="1"
+F 0 "TP16" V 2250 2750 50  0000 L CNN
+F 1 "USART_TX" V 2250 3100 50  0000 L CNN
+F 2 "" H 2450 2550 50  0001 C CNN
+F 3 "~" H 2450 2550 50  0001 C CNN
+	1    2250 2550
+	0    1    1    0
+$EndComp
+$Comp
+L Connector:TestPoint TP?
+U 1 1 6191613B
+P 2250 2650
+AR Path="/616688D6/6191613B" Ref="TP?"  Part="1"
+AR Path="/61668514/6191613B" Ref="TP17"  Part="1"
+F 0 "TP17" V 2250 2850 50  0000 L CNN
+F 1 "USART_RX" V 2250 3200 50  0000 L CNN
+F 2 "" H 2450 2650 50  0001 C CNN
+F 3 "~" H 2450 2650 50  0001 C CNN
+	1    2250 2650
+	0    1    1    0
+$EndComp
+$Comp
+L Connector:TestPoint TP?
+U 1 1 61916141
+P 2250 2750
+AR Path="/616688D6/61916141" Ref="TP?"  Part="1"
+AR Path="/61668514/61916141" Ref="TP18"  Part="1"
+F 0 "TP18" V 2250 2950 50  0000 L CNN
+F 1 "GPIO0" V 2250 3300 50  0000 L CNN
+F 2 "" H 2450 2750 50  0001 C CNN
+F 3 "~" H 2450 2750 50  0001 C CNN
+	1    2250 2750
+	0    1    1    0
+$EndComp
+$Comp
+L Connector:TestPoint TP?
+U 1 1 61916147
+P 2250 2850
+AR Path="/616688D6/61916147" Ref="TP?"  Part="1"
+AR Path="/61668514/61916147" Ref="TP19"  Part="1"
+F 0 "TP19" V 2250 3050 50  0000 L CNN
+F 1 "GPIO1" V 2250 3400 50  0000 L CNN
+F 2 "" H 2450 2850 50  0001 C CNN
+F 3 "~" H 2450 2850 50  0001 C CNN
+	1    2250 2850
+	0    1    1    0
+$EndComp
+$Comp
+L Connector:TestPoint TP?
+U 1 1 6191614D
+P 2250 2950
+AR Path="/616688D6/6191614D" Ref="TP?"  Part="1"
+AR Path="/61668514/6191614D" Ref="TP20"  Part="1"
+F 0 "TP20" V 2250 3150 50  0000 L CNN
+F 1 "GPIO2" V 2250 3500 50  0000 L CNN
+F 2 "" H 2450 2950 50  0001 C CNN
+F 3 "~" H 2450 2950 50  0001 C CNN
+	1    2250 2950
+	0    1    1    0
+$EndComp
+$Comp
+L Connector:TestPoint TP?
+U 1 1 61916153
+P 2250 3050
+AR Path="/616688D6/61916153" Ref="TP?"  Part="1"
+AR Path="/61668514/61916153" Ref="TP21"  Part="1"
+F 0 "TP21" V 2250 3250 50  0000 L CNN
+F 1 "GPIO3" V 2250 3600 50  0000 L CNN
+F 2 "" H 2450 3050 50  0001 C CNN
+F 3 "~" H 2450 3050 50  0001 C CNN
+	1    2250 3050
+	0    1    1    0
+$EndComp
+$Comp
+L Connector:TestPoint TP?
+U 1 1 61916C5A
+P 2250 1950
+AR Path="/616688D6/61916C5A" Ref="TP?"  Part="1"
+AR Path="/61668514/61916C5A" Ref="TP14"  Part="1"
+F 0 "TP14" V 2250 2150 50  0000 L CNN
+F 1 "TDI" V 2250 2500 50  0000 L CNN
+F 2 "" H 2450 1950 50  0001 C CNN
+F 3 "~" H 2450 1950 50  0001 C CNN
+	1    2250 1950
+	0    1    1    0
+$EndComp
 $EndSCHEMATC

Commit message: sarted with LPC daughterboard layout
Parts:
- removed TP15: RESETN, symbol Connector:TestPoint
- removed TP18: GPIO0, symbol Connector:TestPoint
- removed TP19: GPIO1, symbol Connector:TestPoint
- removed TP20: GPIO2, symbol Connector:TestPoint
- removed TP21: GPIO3, symbol Connector:TestPoint
- C4, C5, C6: footprint (none) -> Capacitor_SMD:C_0603_1608Metric_Pad1.05x0.95mm_HandSolder
- JP2, JP3: footprint (none) -> Jumper:SolderJumper-2_P1.3mm_Open_TrianglePad1.0x1.5mm
- R4, R5, R6: footprint (none) -> Resistor_SMD:R_0603_1608Metric_Pad1.05x0.95mm_HandSolder
- TP11, TP12, TP13, TP14, TP16, TP17: footprint (none) -> TestPoint:TestPoint_Pad_1.0x1.0mm
- U0: footprint QFN50P500X500X85-33N-D -> hive_daughterboard:LPC845M301JHI33Y
Connections:
- net +3V3: now also C4.1, C5.1, C6.1, U0.19 (VDD), U0.21 (VREFP)
- net GPIO0.0: now also U0.11 (PIO0_27); no longer U0.14 (PIO0_24)
- net GPIO0.1: now also U0.12 (PIO0_26); no longer U0.13 (PIO0_25)
- net GPIO0.2: now also U0.13 (PIO0_25); no longer U0.12 (PIO0_26)
- net GPIO0.3: now also U0.14 (PIO0_24); no longer U0.11 (PIO0_27)
Changed lines of the file:
@@
 F 0 "R4" H 959 4496 50  0000 L CNN
 F 1 "100k" H 959 4405 50  0000 L CNN
-F 2 "" H 900 4450 50  0001 C CNN
+F 2 "Resistor_SMD:R_0603_1608Metric_Pad1.05x0.95mm_HandSolder" H 900 4450 50  0001 C CNN
 F 3 "~" H 900 4450 50  0001 C CNN
 	1    900  4450
@@
 F 0 "JP2" V 1504 4518 50  0000 L CNN
 F 1 "NRST" V 1595 4518 50  0000 L CNN
-F 2 "" H 1550 4450 50  0001 C CNN
+F 2 "Jumper:SolderJumper-2_P1.3mm_Open_TrianglePad1.0x1.5mm" H 1550 4450 50  0001 C CNN
 F 3 "~" H 1550 4450 50  0001 C CNN
 	1    1550 4450
@@
 F 0 "R5" H 2209 4446 50  0000 L CNN
 F 1 "10k" H 2209 4355 50  0000 L CNN
-F 2 "" H 2150 4400 50  0001 C CNN
+F 2 "Resistor_SMD:R_0603_1608Metric_Pad1.05x0.95mm_HandSolder" H 2150 4400 50  0001 C CNN
 F 3 "~" H 2150 4400 50  0001 C CNN
 	1    2150 4400
@@
 F 0 "R6" H 2659 4446 50  0000 L CNN
 F 1 "10k" H 2659 4355 50  0000 L CNN
-F 2 "" H 2600 4400 50  0001 C CNN
+F 2 "Resistor_SMD:R_0603_1608Metric_Pad1.05x0.95mm_HandSolder" H 2600 4400 50  0001 C CNN
 F 3 "~" H 2600 4400 50  0001 C CNN
 	1    2600 4400
@@
 F 0 "C5" H 7992 1596 50  0000 L CNN
 F 1 "100n" H 7992 1505 50  0000 L CNN
-F 2 "" H 7900 1550 50  0001 C CNN
+F 2 "Capacitor_SMD:C_0603_1608Metric_Pad1.05x0.95mm_HandSolder" H 7900 1550 50  0001 C CNN
 F 3 "~" H 7900 1550 50  0001 C CNN
 	1    7900 1550
@@
 F 0 "C6" H 8392 1596 50  0000 L CNN
 F 1 "100n" H 8392 1505 50  0000 L CNN
-F 2 "" H 8300 1550 50  0001 C CNN
+F 2 "Capacitor_SMD:C_0603_1608Metric_Pad1.05x0.95mm_HandSolder" H 8300 1550 50  0001 C CNN
 F 3 "~" H 8300 1550 50  0001 C CNN
 	1    8300 1550
@@
 F 0 "C4" H 7492 1596 50  0000 L CNN
 F 1 "4.7u" H 7492 1505 50  0000 L CNN
-F 2 "" H 7400 1550 50  0001 C CNN
+F 2 "Capacitor_SMD:C_0603_1608Metric_Pad1.05x0.95mm_HandSolder" H 7400 1550 50  0001 C CNN
 F 3 "~" H 7400 1550 50  0001 C CNN
 	1    7400 1550
@@
 F 0 "U0" H 6850 2000 50  0000 C CNN
 F 1 "LPC845M301JHI33Y" H 6850 2100 50  0000 C CNN
-F 2 "QFN50P500X500X85-33N-D" H 9150 3500 50  0001 L CNN
+F 2 "hive_daughterboard:LPC845M301JHI33Y" H 9150 3500 50  0001 L CNN
 F 3 "http://www.nxp.com/docs/en/data-sheet/LPC84x.pdf" H 9150 3400 50  0001 L CNN
 F 4 "NXP - LPC845M301JHI33Y - MCU, 32BIT, 30MHZ, HVQFN-33" H 9150 3300 50  0001 L CNN "Description"
@@
 F 0 "JP3" H 4500 2750 50  0000 C CNN
 F 1 "NJRST" H 4000 2750 50  0000 C CNN
-F 2 "" H 4250 2800 50  0001 C CNN
+F 2 "Jumper:SolderJumper-2_P1.3mm_Open_TrianglePad1.0x1.5mm" H 4250 2800 50  0001 C CNN
 F 3 "~" H 4250 2800 50  0001 C CNN
 	1    4250 2800
@@
 USART_TX
 Wire Wire Line
+	8550 3600 9100 3600
+Text Label 9100 3600 2    50   ~ 0
+GPIO1
+Wire Wire Line
+	8550 3700 9100 3700
+Text Label 9100 3700 2    50   ~ 0
+GPIO0
+Wire Wire Line
+	8550 3400 9100 3400
+Text Label 9100 3400 2    50   ~ 0
+GPIO3
+Wire Wire Line
 	8550 3500 9100 3500
 Text Label 9100 3500 2    50   ~ 0
-GPIO1
-Wire Wire Line
-	8550 3400 9100 3400
-Text Label 9100 3400 2    50   ~ 0
-GPIO0
-Wire Wire Line
-	8550 3700 9100 3700
-Text Label 9100 3700 2    50   ~ 0
-GPIO3
-Wire Wire Line
-	8550 3600 9100 3600
-Text Label 9100 3600 2    50   ~ 0
 GPIO2
 NoConn ~ 5150 3000
@@
 F 0 "TP11" V 2250 1850 50  0000 L CNN
 F 1 "SWDIO-TMS" V 2250 2200 50  0000 L CNN
-F 2 "" H 2450 1650 50  0001 C CNN
+F 2 "TestPoint:TestPoint_Pad_1.0x1.0mm" H 2450 1650 50  0001 C CNN
 F 3 "~" H 2450 1650 50  0001 C CNN
 	1    2250 1650
@@
 F 0 "TP12" V 2250 1950 50  0000 L CNN
 F 1 "SWCLK-TCLK" V 2250 2300 50  0000 L CNN
-F 2 "" H 2450 1750 50  0001 C CNN
+F 2 "TestPoint:TestPoint_Pad_1.0x1.0mm" H 2450 1750 50  0001 C CNN
 F 3 "~" H 2450 1750 50  0001 C CNN
 	1    2250 1750
@@
 F 0 "TP13" V 2250 2050 50  0000 L CNN
 F 1 "TDO" V 2250 2400 50  0000 L CNN
-F 2 "" H 2450 1850 50  0001 C CNN
+F 2 "TestPoint:TestPoint_Pad_1.0x1.0mm" H 2450 1850 50  0001 C CNN
 F 3 "~" H 2450 1850 50  0001 C CNN
 	1    2250 1850
-	0    1    1    0
-$EndComp
-$Comp
-L Connector:TestPoint TP?
-U 1 1 6191612F
-P 2250 2050
-AR Path="/616688D6/6191612F" Ref="TP?"  Part="1"
-AR Path="/61668514/6191612F" Ref="TP15"  Part="1"
-F 0 "TP15" V 2250 2250 50  0000 L CNN
-F 1 "RESETN" V 2250 2600 50  0000 L CNN
-F 2 "" H 2450 2050 50  0001 C CNN
-F 3 "~" H 2450 2050 50  0001 C CNN
-	1    2250 2050
 	0    1    1    0
 $EndComp
@@
 F 0 "TP16" V 2250 2750 50  0000 L CNN
 F 1 "USART_TX" V 2250 3100 50  0000 L CNN
-F 2 "" H 2450 2550 50  0001 C CNN
+F 2 "TestPoint:TestPoint_Pad_1.0x1.0mm" H 2450 2550 50  0001 C CNN
 F 3 "~" H 2450 2550 50  0001 C CNN
 	1    2250 2550
@@
 F 0 "TP17" V 2250 2850 50  0000 L CNN
 F 1 "USART_RX" V 2250 3200 50  0000 L CNN
-F 2 "" H 2450 2650 50  0001 C CNN
+F 2 "TestPoint:TestPoint_Pad_1.0x1.0mm" H 2450 2650 50  0001 C CNN
 F 3 "~" H 2450 2650 50  0001 C CNN
 	1    2250 2650
-	0    1    1    0
-$EndComp
-$Comp
-L Connector:TestPoint TP?
-U 1 1 61916141
-P 2250 2750
-AR Path="/616688D6/61916141" Ref="TP?"  Part="1"
-AR Path="/61668514/61916141" Ref="TP18"  Part="1"
-F 0 "TP18" V 2250 2950 50  0000 L CNN
-F 1 "GPIO0" V 2250 3300 50  0000 L CNN
-F 2 "" H 2450 2750 50  0001 C CNN
-F 3 "~" H 2450 2750 50  0001 C CNN
-	1    2250 2750
-	0    1    1    0
-$EndComp
-$Comp
-L Connector:TestPoint TP?
-U 1 1 61916147
-P 2250 2850
-AR Path="/616688D6/61916147" Ref="TP?"  Part="1"
-AR Path="/61668514/61916147" Ref="TP19"  Part="1"
-F 0 "TP19" V 2250 3050 50  0000 L CNN
-F 1 "GPIO1" V 2250 3400 50  0000 L CNN
-F 2 "" H 2450 2850 50  0001 C CNN
-F 3 "~" H 2450 2850 50  0001 C CNN
-	1    2250 2850
-	0    1    1    0
-$EndComp
-$Comp
-L Connector:TestPoint TP?
-U 1 1 6191614D
-P 2250 2950
-AR Path="/616688D6/6191614D" Ref="TP?"  Part="1"
-AR Path="/61668514/6191614D" Ref="TP20"  Part="1"
-F 0 "TP20" V 2250 3150 50  0000 L CNN
-F 1 "GPIO2" V 2250 3500 50  0000 L CNN
-F 2 "" H 2450 2950 50  0001 C CNN
-F 3 "~" H 2450 2950 50  0001 C CNN
-	1    2250 2950
-	0    1    1    0
-$EndComp
-$Comp
-L Connector:TestPoint TP?
-U 1 1 61916153
-P 2250 3050
-AR Path="/616688D6/61916153" Ref="TP?"  Part="1"
-AR Path="/61668514/61916153" Ref="TP21"  Part="1"
-F 0 "TP21" V 2250 3250 50  0000 L CNN
-F 1 "GPIO3" V 2250 3600 50  0000 L CNN
-F 2 "" H 2450 3050 50  0001 C CNN
-F 3 "~" H 2450 3050 50  0001 C CNN
-	1    2250 3050
 	0    1    1    0
 $EndComp
@@
 F 0 "TP14" V 2250 2150 50  0000 L CNN
 F 1 "TDI" V 2250 2500 50  0000 L CNN
-F 2 "" H 2450 1950 50  0001 C CNN
+F 2 "TestPoint:TestPoint_Pad_1.0x1.0mm" H 2450 1950 50  0001 C CNN
 F 3 "~" H 2450 1950 50  0001 C CNN
 	1    2250 1950
 	0    1    1    0
 $EndComp
+$Comp
+L power:+3V3 #PWR0117
+U 1 1 61987FA7
+P 8300 1250
+F 0 "#PWR0117" H 8300 1100 50  0001 C CNN
+F 1 "+3V3" H 8315 1423 50  0000 C CNN
+F 2 "" H 8300 1250 50  0001 C CNN
+F 3 "" H 8300 1250 50  0001 C CNN
+	1    8300 1250
+	1    0    0    -1
+$EndComp
+Wire Wire Line
+	8300 1250 8300 1350
+Connection ~ 8300 1350
 $EndSCHEMATC
