File: daughterboard/LPC_00/target3.sch (KiCad schematic (older format))
At the start: 0 parts

Commit message: finished LPC Daughterboard schematics
Parts:
- added C16: 4.7u, symbol Device:C_Small
- added C17, C18: 100n, symbol Device:C_Small
- added JP5: NRST, symbol Jumper:SolderJumper_2_Open
- added R11, R12: 100k, symbol Device:R_Small
- added U3: LPC1313FBD48_01,15, hive_daughterboard:LPC1313FBD48_0115, symbol hive_daughterboard:LPC1313FBD48_01,15
Connections:
- net +3V3: now also R11.2
- net GPIO3.0: now also U3.11 (PIO2_7)
- net GPIO3.1: now also U3.12 (PIO2_8)
- net GPIO3.2: now also U3.24 (PIO2_9)
- net GPIO3.3: now also U3.25 (PIO2_10)
- net RST_3: now also JP5.1 (A), R11.1, U3.3 (~RESET~/PIO0_0)
- net TCK|SWDCLK_3: now also U3.29 (SWCLK/PIO0_10/SCK0/CT16B0_MAT2)
- net TDI|NC_3: now also R12.1
- net TDO|SWO_3: now also U3.28 (_PIO0_9/MOSI0/CT16B0_MAT1/SWO)
- net TMS|SWDIO_3: now also U3.39 (SWDIO/PIO1_3/AD4/CT32B1_MAT2)
- net UART_RxD3: now also U3.47 (PIO1_7/TXD/CT32B0_MAT1)
- net UART_TxD3: now also U3.46 (PIO1_6/RXD/CT32B0_MAT0)
- new net: C16.1, C17.1, C18.1, U3.44 (VDD), U3.8 (VDD)
- new net GND: C16.2, C17.2, C18.2, JP5.2 (B), R12.2, U3.41 (VSS), U3.5 (VSS), U3.6 (XTALIN)
- no-connect marks 0 -> 33
Other:
- note removed: "Power"
