File: daughterboard/LPC_00/target3.sch (KiCad schematic (older format))
At the start: 7 parts, among them U3 LPC1313FBD48_01,15

Commit message: ERC on daughterboards
Connections:
- net +3V3: now also C16.1, C17.1, C18.1, U3.44 (VDD), U3.8 (VDD)
Changed lines of the file:
@@
 NoConn ~ 7500 4000
 NoConn ~ 7500 4100
+$Comp
+L power:+3V3 #PWR0116
+U 1 1 6190C567
+P 7850 1300
+F 0 "#PWR0116" H 7850 1150 50  0001 C CNN
+F 1 "+3V3" H 7865 1473 50  0000 C CNN
+F 2 "" H 7850 1300 50  0001 C CNN
+F 3 "" H 7850 1300 50  0001 C CNN
+	1    7850 1300
+	1    0    0    -1
+$EndComp
+Wire Wire Line
+	7850 1300 7850 1450
+Connection ~ 7850 1450
 $EndSCHEMATC

Commit message: added testpoints to daughterboards, updated readme
Parts:
- added TP32: SWDIO, symbol Connector:TestPoint
- added TP33: SWCLK, symbol Connector:TestPoint
- added TP34: SWO, symbol Connector:TestPoint
- added TP35: RESETN, symbol Connector:TestPoint
- added TP36: USART_TX, symbol Connector:TestPoint
- added TP37: USART_RX, symbol Connector:TestPoint
- added TP38: GPIO0, symbol Connector:TestPoint
- added TP39: GPIO1, symbol Connector:TestPoint
- added TP40: GPIO2, symbol Connector:TestPoint
- added TP41: GPIO3, symbol Connector:TestPoint
Connections:
- net GPIO3.0: now also TP38.1
- net GPIO3.1: now also TP39.1
- net GPIO3.2: now also TP40.1
- net GPIO3.3: now also TP41.1
- net RST_3: now also TP35.1
- net TCK|SWDCLK_3: now also TP33.1
- net TDO|SWO_3: now also TP34.1
- net TMS|SWDIO_3: now also TP32.1
- net UART_RxD3: now also TP36.1
- net UART_TxD3: now also TP37.1
Changed lines of the file:
@@
 	7850 1300 7850 1450
 Connection ~ 7850 1450
+$Comp
+L Connector:TestPoint TP?
+U 1 1 619199B0
+P 2200 1700
+AR Path="/616688D6/619199B0" Ref="TP?"  Part="1"
+AR Path="/61668157/619199B0" Ref="TP32"  Part="1"
+F 0 "TP32" V 2200 1900 50  0000 L CNN
+F 1 "SWDIO" V 2200 2250 50  0000 L CNN
+F 2 "" H 2400 1700 50  0001 C CNN
+F 3 "~" H 2400 1700 50  0001 C CNN
+	1    2200 1700
+	0    1    1    0
+$EndComp
+$Comp
+L Connector:TestPoint TP?
+U 1 1 619199B6
+P 2200 1800
+AR Path="/616688D6/619199B6" Ref="TP?"  Part="1"
+AR Path="/61668157/619199B6" Ref="TP33"  Part="1"
+F 0 "TP33" V 2200 2000 50  0000 L CNN
+F 1 "SWCLK" V 2200 2350 50  0000 L CNN
+F 2 "" H 2400 1800 50  0001 C CNN
+F 3 "~" H 2400 1800 50  0001 C CNN
+	1    2200 1800
+	0    1    1    0
+$EndComp
+$Comp
+L Connector:TestPoint TP?
+U 1 1 619199BC
+P 2200 1900
+AR Path="/616688D6/619199BC" Ref="TP?"  Part="1"
+AR Path="/61668157/619199BC" Ref="TP34"  Part="1"
+F 0 "TP34" V 2200 2100 50  0000 L CNN
+F 1 "SWO" V 2200 2450 50  0000 L CNN
+F 2 "" H 2400 1900 50  0001 C CNN
+F 3 "~" H 2400 1900 50  0001 C CNN
+	1    2200 1900
+	0    1    1    0
+$EndComp
+$Comp
+L Connector:TestPoint TP?
+U 1 1 619199C2
+P 2200 2100
+AR Path="/616688D6/619199C2" Ref="TP?"  Part="1"
+AR Path="/61668157/619199C2" Ref="TP35"  Part="1"
+F 0 "TP35" V 2200 2300 50  0000 L CNN
+F 1 "RESETN" V 2200 2650 50  0000 L CNN
+F 2 "" H 2400 2100 50  0001 C CNN
+F 3 "~" H 2400 2100 50  0001 C CNN
+	1    2200 2100
+	0    1    1    0
+$EndComp
+$Comp
+L Connector:TestPoint TP?
+U 1 1 619199C8
+P 2200 2600
+AR Path="/616688D6/619199C8" Ref="TP?"  Part="1"
+AR Path="/61668157/619199C8" Ref="TP36"  Part="1"
+F 0 "TP36" V 2200 2800 50  0000 L CNN
+F 1 "USART_TX" V 2200 3150 50  0000 L CNN
+F 2 "" H 2400 2600 50  0001 C CNN
+F 3 "~" H 2400 2600 50  0001 C CNN
+	1    2200 2600
+	0    1    1    0
+$EndComp
+$Comp
+L Connector:TestPoint TP?
+U 1 1 619199CE
+P 2200 2700
+AR Path="/616688D6/619199CE" Ref="TP?"  Part="1"
+AR Path="/61668157/619199CE" Ref="TP37"  Part="1"
+F 0 "TP37" V 2200 2900 50  0000 L CNN
+F 1 "USART_RX" V 2200 3250 50  0000 L CNN
+F 2 "" H 2400 2700 50  0001 C CNN
+F 3 "~" H 2400 2700 50  0001 C CNN
+	1    2200 2700
+	0    1    1    0
+$EndComp
+$Comp
+L Connector:TestPoint TP?
+U 1 1 619199D4
+P 2200 2800
+AR Path="/616688D6/619199D4" Ref="TP?"  Part="1"
+AR Path="/61668157/619199D4" Ref="TP38"  Part="1"
+F 0 "TP38" V 2200 3000 50  0000 L CNN
+F 1 "GPIO0" V 2200 3350 50  0000 L CNN
+F 2 "" H 2400 2800 50  0001 C CNN
+F 3 "~" H 2400 2800 50  0001 C CNN
+	1    2200 2800
+	0    1    1    0
+$EndComp
+$Comp
+L Connector:TestPoint TP?
+U 1 1 619199DA
+P 2200 2900
+AR Path="/616688D6/619199DA" Ref="TP?"  Part="1"
+AR Path="/61668157/619199DA" Ref="TP39"  Part="1"
+F 0 "TP39" V 2200 3100 50  0000 L CNN
+F 1 "GPIO1" V 2200 3450 50  0000 L CNN
+F 2 "" H 2400 2900 50  0001 C CNN
+F 3 "~" H 2400 2900 50  0001 C CNN
+	1    2200 2900
+	0    1    1    0
+$EndComp
+$Comp
+L Connector:TestPoint TP?
+U 1 1 619199E0
+P 2200 3000
+AR Path="/616688D6/619199E0" Ref="TP?"  Part="1"
+AR Path="/61668157/619199E0" Ref="TP40"  Part="1"
+F 0 "TP40" V 2200 3200 50  0000 L CNN
+F 1 "GPIO2" V 2200 3550 50  0000 L CNN
+F 2 "" H 2400 3000 50  0001 C CNN
+F 3 "~" H 2400 3000 50  0001 C CNN
+	1    2200 3000
+	0    1    1    0
+$EndComp
+$Comp
+L Connector:TestPoint TP?
+U 1 1 619199E6
+P 2200 3100
+AR Path="/616688D6/619199E6" Ref="TP?"  Part="1"
+AR Path="/61668157/619199E6" Ref="TP41"  Part="1"
+F 0 "TP41" V 2200 3300 50  0000 L CNN
+F 1 "GPIO3" V 2200 3650 50  0000 L CNN
+F 2 "" H 2400 3100 50  0001 C CNN
+F 3 "~" H 2400 3100 50  0001 C CNN
+	1    2200 3100
+	0    1    1    0
+$EndComp
 $EndSCHEMATC

Commit message: sarted with LPC daughterboard layout
Parts:
- removed TP35: RESETN, symbol Connector:TestPoint
- removed TP38: GPIO0, symbol Connector:TestPoint
- removed TP39: GPIO1, symbol Connector:TestPoint
- removed TP40: GPIO2, symbol Connector:TestPoint
- removed TP41: GPIO3, symbol Connector:TestPoint
- C16, C17, C18: footprint (none) -> Capacitor_SMD:C_0603_1608Metric_Pad1.05x0.95mm_HandSolder
- JP5: footprint (none) -> Jumper:SolderJumper-2_P1.3mm_Open_TrianglePad1.0x1.5mm
- R11, R12: footprint (none) -> Resistor_SMD:R_0603_1608Metric_Pad1.05x0.95mm_HandSolder
- TP32, TP33, TP34, TP36, TP37: footprint (none) -> TestPoint:TestPoint_Pad_1.0x1.0mm
Changed lines of the file:
@@
 F 0 "R11" H 909 4346 50  0000 L CNN
 F 1 "100k" H 909 4255 50  0000 L CNN
-F 2 "" H 850 4300 50  0001 C CNN
+F 2 "Resistor_SMD:R_0603_1608Metric_Pad1.05x0.95mm_HandSolder" H 850 4300 50  0001 C CNN
 F 3 "~" H 850 4300 50  0001 C CNN
 	1    850  4300
@@
 F 0 "JP5" V 1454 4368 50  0000 L CNN
 F 1 "NRST" V 1545 4368 50  0000 L CNN
-F 2 "" H 1500 4300 50  0001 C CNN
+F 2 "Jumper:SolderJumper-2_P1.3mm_Open_TrianglePad1.0x1.5mm" H 1500 4300 50  0001 C CNN
 F 3 "~" H 1500 4300 50  0001 C CNN
 	1    1500 4300
@@
 F 0 "R12" H 2309 4346 50  0000 L CNN
 F 1 "100k" H 2309 4255 50  0000 L CNN
-F 2 "" H 2250 4300 50  0001 C CNN
+F 2 "Resistor_SMD:R_0603_1608Metric_Pad1.05x0.95mm_HandSolder" H 2250 4300 50  0001 C CNN
 F 3 "~" H 2250 4300 50  0001 C CNN
 	1    2250 4300
@@
 F 0 "C17" H 7542 1696 50  0000 L CNN
 F 1 "100n" H 7542 1605 50  0000 L CNN
-F 2 "" H 7450 1650 50  0001 C CNN
+F 2 "Capacitor_SMD:C_0603_1608Metric_Pad1.05x0.95mm_HandSolder" H 7450 1650 50  0001 C CNN
 F 3 "~" H 7450 1650 50  0001 C CNN
 	1    7450 1650
@@
 F 0 "C18" H 7942 1696 50  0000 L CNN
 F 1 "100n" H 7942 1605 50  0000 L CNN
-F 2 "" H 7850 1650 50  0001 C CNN
+F 2 "Capacitor_SMD:C_0603_1608Metric_Pad1.05x0.95mm_HandSolder" H 7850 1650 50  0001 C CNN
 F 3 "~" H 7850 1650 50  0001 C CNN
 	1    7850 1650
@@
 F 0 "C16" H 7042 1696 50  0000 L CNN
 F 1 "4.7u" H 7042 1605 50  0000 L CNN
-F 2 "" H 6950 1650 50  0001 C CNN
+F 2 "Capacitor_SMD:C_0603_1608Metric_Pad1.05x0.95mm_HandSolder" H 6950 1650 50  0001 C CNN
 F 3 "~" H 6950 1650 50  0001 C CNN
 	1    6950 1650
@@
 F 0 "TP32" V 2200 1900 50  0000 L CNN
 F 1 "SWDIO" V 2200 2250 50  0000 L CNN
-F 2 "" H 2400 1700 50  0001 C CNN
+F 2 "TestPoint:TestPoint_Pad_1.0x1.0mm" H 2400 1700 50  0001 C CNN
 F 3 "~" H 2400 1700 50  0001 C CNN
 	1    2200 1700
@@
 F 0 "TP33" V 2200 2000 50  0000 L CNN
 F 1 "SWCLK" V 2200 2350 50  0000 L CNN
-F 2 "" H 2400 1800 50  0001 C CNN
+F 2 "TestPoint:TestPoint_Pad_1.0x1.0mm" H 2400 1800 50  0001 C CNN
 F 3 "~" H 2400 1800 50  0001 C CNN
 	1    2200 1800
@@
 F 0 "TP34" V 2200 2100 50  0000 L CNN
 F 1 "SWO" V 2200 2450 50  0000 L CNN
-F 2 "" H 2400 1900 50  0001 C CNN
+F 2 "TestPoint:TestPoint_Pad_1.0x1.0mm" H 2400 1900 50  0001 C CNN
 F 3 "~" H 2400 1900 50  0001 C CNN
 	1    2200 1900
-	0    1    1    0
-$EndComp
-$Comp
-L Connector:TestPoint TP?
-U 1 1 619199C2
-P 2200 2100
-AR Path="/616688D6/619199C2" Ref="TP?"  Part="1"
-AR Path="/61668157/619199C2" Ref="TP35"  Part="1"
-F 0 "TP35" V 2200 2300 50  0000 L CNN
-F 1 "RESETN" V 2200 2650 50  0000 L CNN
-F 2 "" H 2400 2100 50  0001 C CNN
-F 3 "~" H 2400 2100 50  0001 C CNN
-	1    2200 2100
 	0    1    1    0
 $EndComp
@@
 F 0 "TP36" V 2200 2800 50  0000 L CNN
 F 1 "USART_TX" V 2200 3150 50  0000 L CNN
-F 2 "" H 2400 2600 50  0001 C CNN
+F 2 "TestPoint:TestPoint_Pad_1.0x1.0mm" H 2400 2600 50  0001 C CNN
 F 3 "~" H 2400 2600 50  0001 C CNN
 	1    2200 2600
@@
 F 0 "TP37" V 2200 2900 50  0000 L CNN
 F 1 "USART_RX" V 2200 3250 50  0000 L CNN
-F 2 "" H 2400 2700 50  0001 C CNN
+F 2 "TestPoint:TestPoint_Pad_1.0x1.0mm" H 2400 2700 50  0001 C CNN
 F 3 "~" H 2400 2700 50  0001 C CNN
 	1    2200 2700
 	0    1    1    0
 $EndComp
-$Comp
-L Connector:TestPoint TP?
-U 1 1 619199D4
-P 2200 2800
-AR Path="/616688D6/619199D4" Ref="TP?"  Part="1"
-AR Path="/61668157/619199D4" Ref="TP38"  Part="1"
-F 0 "TP38" V 2200 3000 50  0000 L CNN
-F 1 "GPIO0" V 2200 3350 50  0000 L CNN
-F 2 "" H 2400 2800 50  0001 C CNN
-F 3 "~" H 2400 2800 50  0001 C CNN
-	1    2200 2800
-	0    1    1    0
-$EndComp
-$Comp
-L Connector:TestPoint TP?
-U 1 1 619199DA
-P 2200 2900
-AR Path="/616688D6/619199DA" Ref="TP?"  Part="1"
-AR Path="/61668157/619199DA" Ref="TP39"  Part="1"
-F 0 "TP39" V 2200 3100 50  0000 L CNN
-F 1 "GPIO1" V 2200 3450 50  0000 L CNN
-F 2 "" H 2400 2900 50  0001 C CNN
-F 3 "~" H 2400 2900 50  0001 C CNN
-	1    2200 2900
-	0    1    1    0
-$EndComp
-$Comp
-L Connector:TestPoint TP?
-U 1 1 619199E0
-P 2200 3000
-AR Path="/616688D6/619199E0" Ref="TP?"  Part="1"
-AR Path="/61668157/619199E0" Ref="TP40"  Part="1"
-F 0 "TP40" V 2200 3200 50  0000 L CNN
-F 1 "GPIO2" V 2200 3550 50  0000 L CNN
-F 2 "" H 2400 3000 50  0001 C CNN
-F 3 "~" H 2400 3000 50  0001 C CNN
-	1    2200 3000
-	0    1    1    0
-$EndComp
-$Comp
-L Connector:TestPoint TP?
-U 1 1 619199E6
-P 2200 3100
-AR Path="/616688D6/619199E6" Ref="TP?"  Part="1"
-AR Path="/61668157/619199E6" Ref="TP41"  Part="1"
-F 0 "TP41" V 2200 3300 50  0000 L CNN
-F 1 "GPIO3" V 2200 3650 50  0000 L CNN
-F 2 "" H 2400 3100 50  0001 C CNN
-F 3 "~" H 2400 3100 50  0001 C CNN
-	1    2200 3100
-	0    1    1    0
-$EndComp

Commit message: finsihed LPC daughterboard layout
Connections:
- net GPIO3.0: now also U3.14 (PIO0_3); no longer U3.11 (PIO2_7)
- net GPIO3.1: now also U3.15 (PIO0_4/SCL); no longer U3.12 (PIO2_8)
- net GPIO3.2: now also U3.16 (PIO0_5/SDA); no longer U3.24 (PIO2_9)
- net GPIO3.3: now also U3.17 (PIO1_9/CT16B1_MAT0); no longer U3.25 (PIO2_10)
Changed lines of the file:
@@
 UART_RX
 Wire Wire Line
-	7500 3100 8050 3100
-Text Label 8050 3100 2    50   ~ 0
+	4850 2700 4300 2700
+Text Label 4300 2700 0    50   ~ 0
 GPIO1
 Wire Wire Line
-	7500 3000 8050 3000
-Text Label 8050 3000 2    50   ~ 0
+	4850 2600 4300 2600
+Text Label 4300 2600 0    50   ~ 0
 GPIO0
 Wire Wire Line
-	7500 3300 8050 3300
-Text Label 8050 3300 2    50   ~ 0
+	4850 4500 4300 4500
+Text Label 4300 4500 0    50   ~ 0
 GPIO3
 Wire Wire Line
-	7500 3200 8050 3200
-Text Label 8050 3200 2    50   ~ 0
+	4850 2800 4300 2800
+Text Label 4300 2800 0    50   ~ 0
 GPIO2
 $Comp
@@
 NoConn ~ 4850 2400
 NoConn ~ 4850 2500
-NoConn ~ 4850 2600
-NoConn ~ 4850 2700
-NoConn ~ 4850 2800
 NoConn ~ 4850 2900
 NoConn ~ 4850 3000
@@
 NoConn ~ 4850 4100
 NoConn ~ 4850 4400
-NoConn ~ 4850 4500
 NoConn ~ 4850 4600
 NoConn ~ 4850 4700
@@
 	0    1    1    0
 $EndComp
+NoConn ~ 7500 3000
+NoConn ~ 7500 3100
+NoConn ~ 7500 3200
+NoConn ~ 7500 3300
 $EndSCHEMATC
