File: daughterboard/LPC_00/LPC_00.sch (KiCad schematic (older format))
At the start: 2 parts, among them J1 m2_keyA_67pin_daughterboard

Commit message: sarted with LPC daughterboard layout
Changed lines of the file:
@@
 	0    -1   -1   0
 $EndComp
+$Comp
+L power:PWR_FLAG #FLG0102
+U 1 1 6193E700
+P 7500 1500
+F 0 "#FLG0102" H 7500 1575 50  0001 C CNN
+F 1 "PWR_FLAG" H 7500 1673 50  0000 C CNN
+F 2 "" H 7500 1500 50  0001 C CNN
+F 3 "~" H 7500 1500 50  0001 C CNN
+	1    7500 1500
+	1    0    0    -1
+$EndComp
+Wire Wire Line
+	7500 1500 7500 1600
+Connection ~ 7500 1600
 $EndSCHEMATC
