File: daughterboard/ATSAMD_00/target0.sch (KiCad schematic (older format))
At the start: 10 parts

Commit message: ERC on daughterboards
Parts:
- gave numbers to parts that had none: 10
Changed lines of the file:
@@
 Add your target here and connect it to the provided Debug and GPIO/UART connections.\n\nDebug and GPIO/UART connections are 5V tolerant. Min signal level is 3.3V
 $Comp
-L MCU_Microchip_SAMD:ATSAMD10C13A-SS U?
+L MCU_Microchip_SAMD:ATSAMD10C13A-SS U0
 U 1 1 61929D97
 P 6150 2600
-F 0 "U?" H 5450 3450 50  0000 C CNN
+F 0 "U0" H 5450 3450 50  0000 C CNN
 F 1 "ATSAMD10C13A-SS" H 5500 3300 50  0000 C CNN
 F 2 "Package_SO:SOIC-14_3.9x8.7mm_P1.27mm" H 6150 1550 50  0001 C CNN
@@
 P 7100 1550
 AR Path="/616688D6/6193577E" Ref="C?"  Part="1"
-AR Path="/61668514/6193577E" Ref="C?"  Part="1"
-F 0 "C?" H 7192 1596 50  0000 L CNN
+AR Path="/61668514/6193577E" Ref="C5"  Part="1"
+F 0 "C5" H 7192 1596 50  0000 L CNN
 F 1 "4.7u" H 7192 1505 50  0000 L CNN
 F 2 "" H 7100 1550 50  0001 C CNN
@@
 P 7500 1550
 AR Path="/616688D6/61935784" Ref="C?"  Part="1"
-AR Path="/61668514/61935784" Ref="C?"  Part="1"
-F 0 "C?" H 7592 1596 50  0000 L CNN
+AR Path="/61668514/61935784" Ref="C6"  Part="1"
+F 0 "C6" H 7592 1596 50  0000 L CNN
 F 1 "100n" H 7592 1505 50  0000 L CNN
 F 2 "" H 7500 1550 50  0001 C CNN
@@
 P 7500 1800
 AR Path="/616688D6/61935792" Ref="#PWR?"  Part="1"
-AR Path="/61668514/61935792" Ref="#PWR?"  Part="1"
-F 0 "#PWR?" H 7500 1550 50  0001 C CNN
+AR Path="/61668514/61935792" Ref="#PWR0132"  Part="1"
+F 0 "#PWR0132" H 7500 1550 50  0001 C CNN
 F 1 "GND" H 7505 1627 50  0000 C CNN
 F 2 "" H 7500 1800 50  0001 C CNN
@@
 P 7500 1150
 AR Path="/616688D6/619357A2" Ref="#PWR?"  Part="1"
-AR Path="/61668514/619357A2" Ref="#PWR?"  Part="1"
-F 0 "#PWR?" H 7500 1000 50  0001 C CNN
+AR Path="/61668514/619357A2" Ref="#PWR0133"  Part="1"
+F 0 "#PWR0133" H 7500 1000 50  0001 C CNN
 F 1 "+3V3" H 7515 1323 50  0000 C CNN
 F 2 "" H 7500 1150 50  0001 C CNN
@@
 P 6150 3300
 AR Path="/616688D6/61936958" Ref="#PWR?"  Part="1"
-AR Path="/61668514/61936958" Ref="#PWR?"  Part="1"
-F 0 "#PWR?" H 6150 3050 50  0001 C CNN
+AR Path="/61668514/61936958" Ref="#PWR0134"  Part="1"
+F 0 "#PWR0134" H 6150 3050 50  0001 C CNN
 F 1 "GND" H 6155 3127 50  0000 C CNN
 F 2 "" H 6150 3300 50  0001 C CNN
@@
 RESETN
 $Comp
-L Device:R_Small R?
+L Device:R_Small R6
 U 1 1 6193CA84
 P 900 4300
-F 0 "R?" H 959 4346 50  0000 L CNN
+F 0 "R6" H 959 4346 50  0000 L CNN
 F 1 "10k" H 959 4255 50  0000 L CNN
 F 2 "" H 900 4300 50  0001 C CNN
@@
 $EndComp
 $Comp
-L Device:R_Small R?
+L Device:R_Small R7
 U 1 1 6193CA8A
 P 1600 3850
-F 0 "R?" V 1404 3850 50  0000 C CNN
+F 0 "R7" V 1404 3850 50  0000 C CNN
 F 1 "330" V 1495 3850 50  0000 C CNN
 F 2 "" H 1600 3850 50  0001 C CNN
@@
 $EndComp
 $Comp
-L Device:C_Small C?
+L Device:C_Small C4
 U 1 1 6193CA90
 P 1200 4300
-F 0 "C?" H 1292 4346 50  0000 L CNN
+F 0 "C4" H 1292 4346 50  0000 L CNN
 F 1 "100n" H 1292 4255 50  0000 L CNN
 F 2 "" H 1200 4300 50  0001 C CNN
@@
 $EndComp
 $Comp
-L power:+3V3 #PWR?
+L power:+3V3 #PWR0135
 U 1 1 6193CA96
 P 900 4650
-F 0 "#PWR?" H 900 4500 50  0001 C CNN
+F 0 "#PWR0135" H 900 4500 50  0001 C CNN
 F 1 "+3V3" H 915 4823 50  0000 C CNN
 F 2 "" H 900 4650 50  0001 C CNN
@@
 	1200 3850 900  3850
 $Comp
-L power:GND #PWR?
+L power:GND #PWR0136
 U 1 1 6193CAA4
 P 1200 4650
-F 0 "#PWR?" H 1200 4400 50  0001 C CNN
+F 0 "#PWR0136" H 1200 4400 50  0001 C CNN
 F 1 "GND" H 1205 4477 50  0000 C CNN
 F 2 "" H 1200 4650 50  0001 C CNN
@@
 	1200 4650 1200 4550
 $Comp
-L Jumper:SolderJumper_2_Open JP?
+L Jumper:SolderJumper_2_Open JP2
 U 1 1 6193CAAB
 P 1950 4300
-F 0 "JP?" V 1996 4212 50  0000 R CNN
+F 0 "JP2" V 1996 4212 50  0000 R CNN
 F 1 "NRST" V 1905 4212 50  0000 R CNN
 F 2 "" H 1950 4300 50  0001 C CNN
@@
 SWCLK
 $Comp
-L Device:R_Small R?
+L Device:R_Small R8
 U 1 1 6193CAB8
 P 2700 4250
-F 0 "R?" H 2759 4296 50  0000 L CNN
+F 0 "R8" H 2759 4296 50  0000 L CNN
 F 1 "1k" H 2759 4205 50  0000 L CNN
 F 2 "" H 2700 4250 50  0001 C CNN
@@
 $EndComp
 $Comp
-L power:+3V3 #PWR?
+L power:+3V3 #PWR0137
 U 1 1 6193CABE
 P 2700 4650
-F 0 "#PWR?" H 2700 4500 50  0001 C CNN
+F 0 "#PWR0137" H 2700 4500 50  0001 C CNN
 F 1 "+3V3" H 2715 4823 50  0000 C CNN
 F 2 "" H 2700 4650 50  0001 C CNN
@@
 NC
 $Comp
-L Device:R_Small R?
+L Device:R_Small R9
 U 1 1 6193CAC7
 P 3150 4250
-F 0 "R?" H 3209 4296 50  0000 L CNN
+F 0 "R9" H 3209 4296 50  0000 L CNN
 F 1 "100k" H 3209 4205 50  0000 L CNN
 F 2 "" H 3150 4250 50  0001 C CNN
@@
 $EndComp
 $Comp
-L power:GND #PWR?
+L power:GND #PWR0138
 U 1 1 6193CACD
 P 3150 4650
-F 0 "#PWR?" H 3150 4400 50  0001 C CNN
+F 0 "#PWR0138" H 3150 4400 50  0001 C CNN
 F 1 "GND" H 3155 4477 50  0000 C CNN
 F 2 "" H 3150 4650 50  0001 C CNN
@@
 SWO
 $Comp
-L Device:R_Small R?
+L Device:R_Small R10
 U 1 1 6193EA0D
 P 3500 4250
-F 0 "R?" H 3559 4296 50  0000 L CNN
+F 0 "R10" H 3559 4296 50  0000 L CNN
 F 1 "100k" H 3559 4205 50  0000 L CNN
 F 2 "" H 3500 4250 50  0001 C CNN
@@
 $EndComp
 $Comp
-L power:GND #PWR?
+L power:GND #PWR0139
 U 1 1 6193EA13
 P 3500 4650
-F 0 "#PWR?" H 3500 4400 50  0001 C CNN
+F 0 "#PWR0139" H 3500 4400 50  0001 C CNN
 F 1 "GND" H 3505 4477 50  0000 C CNN
 F 2 "" H 3500 4650 50  0001 C CNN

Commit message: added testpoints to daughterboards, updated readme
Parts:
- added TP11: SWDIO, symbol Connector:TestPoint
- added TP12: SWCLK, symbol Connector:TestPoint
- added TP13: SWO, symbol Connector:TestPoint
- added TP14: RESETN, symbol Connector:TestPoint
- added TP15: USART_TX, symbol Connector:TestPoint
- added TP16: USART_RX, symbol Connector:TestPoint
- added TP17: GPIO0, symbol Connector:TestPoint
- added TP18: GPIO1, symbol Connector:TestPoint
- added TP19: GPIO2, symbol Connector:TestPoint
- added TP20: GPIO3, symbol Connector:TestPoint
Connections:
- net GPIO0.0: now also TP17.1
- net GPIO0.1: now also TP18.1
- net GPIO0.2: now also TP19.1
- net GPIO0.3: now also TP20.1
- net RST_0: now also TP14.1
- net TCK|SWDCLK_0: now also TP12.1
- net TDO|SWO_0: now also TP13.1
- net TMS|SWDIO_0: now also TP11.1
- net UART_RxD0: now also TP15.1
- net UART_TxD0: now also TP16.1
Changed lines of the file:
@@
 NoConn ~ 5650 2900
 NoConn ~ 6650 2700
+$Comp
+L Connector:TestPoint TP?
+U 1 1 61917309
+P 2200 1650
+AR Path="/616688D6/61917309" Ref="TP?"  Part="1"
+AR Path="/61668514/61917309" Ref="TP11"  Part="1"
+F 0 "TP11" V 2200 1850 50  0000 L CNN
+F 1 "SWDIO" V 2200 2200 50  0000 L CNN
+F 2 "" H 2400 1650 50  0001 C CNN
+F 3 "~" H 2400 1650 50  0001 C CNN
+	1    2200 1650
+	0    1    1    0
+$EndComp
+$Comp
+L Connector:TestPoint TP?
+U 1 1 6191730F
+P 2200 1750
+AR Path="/616688D6/6191730F" Ref="TP?"  Part="1"
+AR Path="/61668514/6191730F" Ref="TP12"  Part="1"
+F 0 "TP12" V 2200 1950 50  0000 L CNN
+F 1 "SWCLK" V 2200 2300 50  0000 L CNN
+F 2 "" H 2400 1750 50  0001 C CNN
+F 3 "~" H 2400 1750 50  0001 C CNN
+	1    2200 1750
+	0    1    1    0
+$EndComp
+$Comp
+L Connector:TestPoint TP?
+U 1 1 61917315
+P 2200 1850
+AR Path="/616688D6/61917315" Ref="TP?"  Part="1"
+AR Path="/61668514/61917315" Ref="TP13"  Part="1"
+F 0 "TP13" V 2200 2050 50  0000 L CNN
+F 1 "SWO" V 2200 2400 50  0000 L CNN
+F 2 "" H 2400 1850 50  0001 C CNN
+F 3 "~" H 2400 1850 50  0001 C CNN
+	1    2200 1850
+	0    1    1    0
+$EndComp
+$Comp
+L Connector:TestPoint TP?
+U 1 1 6191731B
+P 2200 2050
+AR Path="/616688D6/6191731B" Ref="TP?"  Part="1"
+AR Path="/61668514/6191731B" Ref="TP14"  Part="1"
+F 0 "TP14" V 2200 2250 50  0000 L CNN
+F 1 "RESETN" V 2200 2600 50  0000 L CNN
+F 2 "" H 2400 2050 50  0001 C CNN
+F 3 "~" H 2400 2050 50  0001 C CNN
+	1    2200 2050
+	0    1    1    0
+$EndComp
+$Comp
+L Connector:TestPoint TP?
+U 1 1 61917321
+P 2200 2550
+AR Path="/616688D6/61917321" Ref="TP?"  Part="1"
+AR Path="/61668514/61917321" Ref="TP15"  Part="1"
+F 0 "TP15" V 2200 2750 50  0000 L CNN
+F 1 "USART_TX" V 2200 3100 50  0000 L CNN
+F 2 "" H 2400 2550 50  0001 C CNN
+F 3 "~" H 2400 2550 50  0001 C CNN
+	1    2200 2550
+	0    1    -1   0
+$EndComp
+$Comp
+L Connector:TestPoint TP?
+U 1 1 61917327
+P 2200 2650
+AR Path="/616688D6/61917327" Ref="TP?"  Part="1"
+AR Path="/61668514/61917327" Ref="TP16"  Part="1"
+F 0 "TP16" V 2200 2850 50  0000 L CNN
+F 1 "USART_RX" V 2200 3200 50  0000 L CNN
+F 2 "" H 2400 2650 50  0001 C CNN
+F 3 "~" H 2400 2650 50  0001 C CNN
+	1    2200 2650
+	0    1    -1   0
+$EndComp
+$Comp
+L Connector:TestPoint TP?
+U 1 1 6191732D
+P 2200 2750
+AR Path="/616688D6/6191732D" Ref="TP?"  Part="1"
+AR Path="/61668514/6191732D" Ref="TP17"  Part="1"
+F 0 "TP17" V 2200 2950 50  0000 L CNN
+F 1 "GPIO0" V 2200 3300 50  0000 L CNN
+F 2 "" H 2400 2750 50  0001 C CNN
+F 3 "~" H 2400 2750 50  0001 C CNN
+	1    2200 2750
+	0    1    -1   0
+$EndComp
+$Comp
+L Connector:TestPoint TP?
+U 1 1 61917333
+P 2200 2850
+AR Path="/616688D6/61917333" Ref="TP?"  Part="1"
+AR Path="/61668514/61917333" Ref="TP18"  Part="1"
+F 0 "TP18" V 2200 3050 50  0000 L CNN
+F 1 "GPIO1" V 2200 3400 50  0000 L CNN
+F 2 "" H 2400 2850 50  0001 C CNN
+F 3 "~" H 2400 2850 50  0001 C CNN
+	1    2200 2850
+	0    1    -1   0
+$EndComp
+$Comp
+L Connector:TestPoint TP?
+U 1 1 61917339
+P 2200 2950
+AR Path="/616688D6/61917339" Ref="TP?"  Part="1"
+AR Path="/61668514/61917339" Ref="TP19"  Part="1"
+F 0 "TP19" V 2200 3150 50  0000 L CNN
+F 1 "GPIO2" V 2200 3500 50  0000 L CNN
+F 2 "" H 2400 2950 50  0001 C CNN
+F 3 "~" H 2400 2950 50  0001 C CNN
+	1    2200 2950
+	0    1    -1   0
+$EndComp
+$Comp
+L Connector:TestPoint TP?
+U 1 1 6191733F
+P 2200 3050
+AR Path="/616688D6/6191733F" Ref="TP?"  Part="1"
+AR Path="/61668514/6191733F" Ref="TP20"  Part="1"
+F 0 "TP20" V 2200 3250 50  0000 L CNN
+F 1 "GPIO3" V 2200 3600 50  0000 L CNN
+F 2 "" H 2400 3050 50  0001 C CNN
+F 3 "~" H 2400 3050 50  0001 C CNN
+	1    2200 3050
+	0    1    -1   0
+$EndComp
 $EndSCHEMATC

Commit message: finished ATSAMD daughterboard layout
Parts:
- removed TP13: SWO, symbol Connector:TestPoint
- removed TP14: RESETN, symbol Connector:TestPoint
- removed TP17: GPIO0, symbol Connector:TestPoint
- removed TP18: GPIO1, symbol Connector:TestPoint
- removed TP19: GPIO2, symbol Connector:TestPoint
- removed TP20: GPIO3, symbol Connector:TestPoint
- C4, C5, C6: footprint (none) -> Capacitor_SMD:C_0603_1608Metric_Pad1.05x0.95mm_HandSolder
- JP2: footprint (none) -> Jumper:SolderJumper-2_P1.3mm_Open_TrianglePad1.0x1.5mm
- R10, R6, R7, R8, R9: footprint (none) -> Resistor_SMD:R_0603_1608Metric_Pad1.05x0.95mm_HandSolder
- TP11, TP12, TP15, TP16: footprint (none) -> TestPoint:TestPoint_Pad_1.0x1.0mm
Changed lines of the file:
@@
 F 0 "C5" H 7192 1596 50  0000 L CNN
 F 1 "4.7u" H 7192 1505 50  0000 L CNN
-F 2 "" H 7100 1550 50  0001 C CNN
+F 2 "Capacitor_SMD:C_0603_1608Metric_Pad1.05x0.95mm_HandSolder" H 7100 1550 50  0001 C CNN
 F 3 "~" H 7100 1550 50  0001 C CNN
 	1    7100 1550
@@
 F 0 "C6" H 7592 1596 50  0000 L CNN
 F 1 "100n" H 7592 1505 50  0000 L CNN
-F 2 "" H 7500 1550 50  0001 C CNN
+F 2 "Capacitor_SMD:C_0603_1608Metric_Pad1.05x0.95mm_HandSolder" H 7500 1550 50  0001 C CNN
 F 3 "~" H 7500 1550 50  0001 C CNN
 	1    7500 1550
@@
 F 0 "R6" H 959 4346 50  0000 L CNN
 F 1 "10k" H 959 4255 50  0000 L CNN
-F 2 "" H 900 4300 50  0001 C CNN
+F 2 "Resistor_SMD:R_0603_1608Metric_Pad1.05x0.95mm_HandSolder" H 900 4300 50  0001 C CNN
 F 3 "~" H 900 4300 50  0001 C CNN
 	1    900  4300
@@
 F 0 "R7" V 1404 3850 50  0000 C CNN
 F 1 "330" V 1495 3850 50  0000 C CNN
-F 2 "" H 1600 3850 50  0001 C CNN
+F 2 "Resistor_SMD:R_0603_1608Metric_Pad1.05x0.95mm_HandSolder" H 1600 3850 50  0001 C CNN
 F 3 "~" H 1600 3850 50  0001 C CNN
 	1    1600 3850
@@
 F 0 "C4" H 1292 4346 50  0000 L CNN
 F 1 "100n" H 1292 4255 50  0000 L CNN
-F 2 "" H 1200 4300 50  0001 C CNN
+F 2 "Capacitor_SMD:C_0603_1608Metric_Pad1.05x0.95mm_HandSolder" H 1200 4300 50  0001 C CNN
 F 3 "~" H 1200 4300 50  0001 C CNN
 	1    1200 4300
@@
 F 0 "JP2" V 1996 4212 50  0000 R CNN
 F 1 "NRST" V 1905 4212 50  0000 R CNN
-F 2 "" H 1950 4300 50  0001 C CNN
+F 2 "Jumper:SolderJumper-2_P1.3mm_Open_TrianglePad1.0x1.5mm" H 1950 4300 50  0001 C CNN
 F 3 "~" H 1950 4300 50  0001 C CNN
 	1    1950 4300
@@
 F 0 "R8" H 2759 4296 50  0000 L CNN
 F 1 "1k" H 2759 4205 50  0000 L CNN
-F 2 "" H 2700 4250 50  0001 C CNN
+F 2 "Resistor_SMD:R_0603_1608Metric_Pad1.05x0.95mm_HandSolder" H 2700 4250 50  0001 C CNN
 F 3 "~" H 2700 4250 50  0001 C CNN
 	1    2700 4250
@@
 F 0 "R9" H 3209 4296 50  0000 L CNN
 F 1 "100k" H 3209 4205 50  0000 L CNN
-F 2 "" H 3150 4250 50  0001 C CNN
+F 2 "Resistor_SMD:R_0603_1608Metric_Pad1.05x0.95mm_HandSolder" H 3150 4250 50  0001 C CNN
 F 3 "~" H 3150 4250 50  0001 C CNN
 	1    3150 4250
@@
 F 0 "R10" H 3559 4296 50  0000 L CNN
 F 1 "100k" H 3559 4205 50  0000 L CNN
-F 2 "" H 3500 4250 50  0001 C CNN
+F 2 "Resistor_SMD:R_0603_1608Metric_Pad1.05x0.95mm_HandSolder" H 3500 4250 50  0001 C CNN
 F 3 "~" H 3500 4250 50  0001 C CNN
 	1    3500 4250
@@
 F 0 "TP11" V 2200 1850 50  0000 L CNN
 F 1 "SWDIO" V 2200 2200 50  0000 L CNN
-F 2 "" H 2400 1650 50  0001 C CNN
+F 2 "TestPoint:TestPoint_Pad_1.0x1.0mm" H 2400 1650 50  0001 C CNN
 F 3 "~" H 2400 1650 50  0001 C CNN
 	1    2200 1650
@@
 F 0 "TP12" V 2200 1950 50  0000 L CNN
 F 1 "SWCLK" V 2200 2300 50  0000 L CNN
-F 2 "" H 2400 1750 50  0001 C CNN
+F 2 "TestPoint:TestPoint_Pad_1.0x1.0mm" H 2400 1750 50  0001 C CNN
 F 3 "~" H 2400 1750 50  0001 C CNN
 	1    2200 1750
-	0    1    1    0
-$EndComp
-$Comp
-L Connector:TestPoint TP?
-U 1 1 61917315
-P 2200 1850
-AR Path="/616688D6/61917315" Ref="TP?"  Part="1"
-AR Path="/61668514/61917315" Ref="TP13"  Part="1"
-F 0 "TP13" V 2200 2050 50  0000 L CNN
-F 1 "SWO" V 2200 2400 50  0000 L CNN
-F 2 "" H 2400 1850 50  0001 C CNN
-F 3 "~" H 2400 1850 50  0001 C CNN
-	1    2200 1850
-	0    1    1    0
-$EndComp
-$Comp
-L Connector:TestPoint TP?
-U 1 1 6191731B
-P 2200 2050
-AR Path="/616688D6/6191731B" Ref="TP?"  Part="1"
-AR Path="/61668514/6191731B" Ref="TP14"  Part="1"
-F 0 "TP14" V 2200 2250 50  0000 L CNN
-F 1 "RESETN" V 2200 2600 50  0000 L CNN
-F 2 "" H 2400 2050 50  0001 C CNN
-F 3 "~" H 2400 2050 50  0001 C CNN
-	1    2200 2050
 	0    1    1    0
 $EndComp
@@
 F 0 "TP15" V 2200 2750 50  0000 L CNN
 F 1 "USART_TX" V 2200 3100 50  0000 L CNN
-F 2 "" H 2400 2550 50  0001 C CNN
+F 2 "TestPoint:TestPoint_Pad_1.0x1.0mm" H 2400 2550 50  0001 C CNN
 F 3 "~" H 2400 2550 50  0001 C CNN
 	1    2200 2550
@@
 F 0 "TP16" V 2200 2850 50  0000 L CNN
 F 1 "USART_RX" V 2200 3200 50  0000 L CNN
-F 2 "" H 2400 2650 50  0001 C CNN
+F 2 "TestPoint:TestPoint_Pad_1.0x1.0mm" H 2400 2650 50  0001 C CNN
 F 3 "~" H 2400 2650 50  0001 C CNN
 	1    2200 2650
 	0    1    -1   0
 $EndComp
-$Comp
-L Connector:TestPoint TP?
-U 1 1 6191732D
-P 2200 2750
-AR Path="/616688D6/6191732D" Ref="TP?"  Part="1"
-AR Path="/61668514/6191732D" Ref="TP17"  Part="1"
-F 0 "TP17" V 2200 2950 50  0000 L CNN
-F 1 "GPIO0" V 2200 3300 50  0000 L CNN
-F 2 "" H 2400 2750 50  0001 C CNN
-F 3 "~" H 2400 2750 50  0001 C CNN
-	1    2200 2750
-	0    1    -1   0
-$EndComp
-$Comp
-L Connector:TestPoint TP?
-U 1 1 61917333
-P 2200 2850
-AR Path="/616688D6/61917333" Ref="TP?"  Part="1"
-AR Path="/61668514/61917333" Ref="TP18"  Part="1"
-F 0 "TP18" V 2200 3050 50  0000 L CNN
-F 1 "GPIO1" V 2200 3400 50  0000 L CNN
-F 2 "" H 2400 2850 50  0001 C CNN
-F 3 "~" H 2400 2850 50  0001 C CNN
-	1    2200 2850
-	0    1    -1   0
-$EndComp
-$Comp
-L Connector:TestPoint TP?
-U 1 1 61917339
-P 2200 2950
-AR Path="/616688D6/61917339" Ref="TP?"  Part="1"
-AR Path="/61668514/61917339" Ref="TP19"  Part="1"
-F 0 "TP19" V 2200 3150 50  0000 L CNN
-F 1 "GPIO2" V 2200 3500 50  0000 L CNN
-F 2 "" H 2400 2950 50  0001 C CNN
-F 3 "~" H 2400 2950 50  0001 C CNN
-	1    2200 2950
-	0    1    -1   0
-$EndComp
-$Comp
-L Connector:TestPoint TP?
-U 1 1 6191733F
-P 2200 3050
-AR Path="/616688D6/6191733F" Ref="TP?"  Part="1"
-AR Path="/61668514/6191733F" Ref="TP20"  Part="1"
-F 0 "TP20" V 2200 3250 50  0000 L CNN
-F 1 "GPIO3" V 2200 3600 50  0000 L CNN
-F 2 "" H 2400 3050 50  0001 C CNN
-F 3 "~" H 2400 3050 50  0001 C CNN
-	1    2200 3050
-	0    1    -1   0
-$EndComp
