File: daughterboard/ATSAMD_00/target2.sch (KiCad schematic (older format))
At the start: 14 parts

Commit message: ERC on daughterboards
Parts:
- gave numbers to parts that had none: 14
Changed lines of the file:
@@
 Add your target here and connect it to the provided Debug and GPIO/UART connections.\n\nDebug and GPIO/UART connections are 5V tolerant. Min signal level is 3.3V
 $Comp
-L MCU_Microchip_SAMD:ATSAMD51J18A-A U?
+L MCU_Microchip_SAMD:ATSAMD51J18A-A U2
 U 1 1 618877C3
 P 5700 3550
-F 0 "U?" H 5700 2350 50  0000 C CNN
+F 0 "U2" H 5700 2350 50  0000 C CNN
 F 1 "ATSAMD51J18A-A" H 5700 2500 50  0000 C CNN
 F 2 "Package_QFP:TQFP-64_10x10mm_P0.5mm" H 5700 3550 50  0001 C CIN
@@
 $EndComp
 $Comp
-L Device:C_Small C?
+L Device:C_Small C10
 U 1 1 6188BA83
 P 6600 1450
-F 0 "C?" H 6692 1496 50  0000 L CNN
+F 0 "C10" H 6692 1496 50  0000 L CNN
 F 1 "10u" H 6692 1405 50  0000 L CNN
 F 2 "" H 6600 1450 50  0001 C CNN
@@
 $EndComp
 $Comp
-L Device:C_Small C?
+L Device:C_Small C9
 U 1 1 6188C49F
 P 4800 1450
-F 0 "C?" H 4892 1496 50  0000 L CNN
+F 0 "C9" H 4892 1496 50  0000 L CNN
 F 1 "4.7u" H 4892 1405 50  0000 L CNN
 F 2 "" H 4800 1450 50  0001 C CNN
@@
 $EndComp
 $Comp
-L Device:C_Small C?
+L Device:C_Small C12
 U 1 1 6188CBA3
 P 7350 1450
-F 0 "C?" H 7442 1496 50  0000 L CNN
+F 0 "C12" H 7442 1496 50  0000 L CNN
 F 1 "100n" H 7442 1405 50  0000 L CNN
 F 2 "" H 7350 1450 50  0001 C CNN
@@
 $EndComp
 $Comp
-L Device:C_Small C?
+L Device:C_Small C8
 U 1 1 6188D060
 P 4350 1450
-F 0 "C?" H 4442 1496 50  0000 L CNN
+F 0 "C8" H 4442 1496 50  0000 L CNN
 F 1 "100n" H 4442 1405 50  0000 L CNN
 F 2 "" H 4350 1450 50  0001 C CNN
@@
 $EndComp
 $Comp
-L Device:C_Small C?
+L Device:C_Small C13
 U 1 1 6188D91D
 P 7750 1450
-F 0 "C?" H 7842 1496 50  0000 L CNN
+F 0 "C13" H 7842 1496 50  0000 L CNN
 F 1 "100n" H 7842 1405 50  0000 L CNN
 F 2 "" H 7750 1450 50  0001 C CNN
@@
 $EndComp
 $Comp
-L Device:C_Small C?
+L Device:C_Small C14
 U 1 1 6188DECF
 P 8150 1450
-F 0 "C?" H 8242 1496 50  0000 L CNN
+F 0 "C14" H 8242 1496 50  0000 L CNN
 F 1 "100n" H 8242 1405 50  0000 L CNN
 F 2 "" H 8150 1450 50  0001 C CNN
@@
 	4350 1650 4350 1550
 $Comp
-L Device:C_Small C?
+L Device:C_Small C11
 U 1 1 6188AF65
 P 6950 1450
-F 0 "C?" H 7042 1496 50  0000 L CNN
+F 0 "C11" H 7042 1496 50  0000 L CNN
 F 1 "1u" H 7042 1405 50  0000 L CNN
 F 2 "" H 6950 1450 50  0001 C CNN
@@
 RESETN
 $Comp
-L Device:R_Small R?
+L Device:R_Small R11
 U 1 1 6189EE33
 P 850 4300
-F 0 "R?" H 909 4346 50  0000 L CNN
+F 0 "R11" H 909 4346 50  0000 L CNN
 F 1 "10k" H 909 4255 50  0000 L CNN
 F 2 "" H 850 4300 50  0001 C CNN
@@
 $EndComp
 $Comp
-L Device:R_Small R?
+L Device:R_Small R12
 U 1 1 6189FEAF
 P 1550 3850
-F 0 "R?" V 1354 3850 50  0000 C CNN
+F 0 "R12" V 1354 3850 50  0000 C CNN
 F 1 "330" V 1445 3850 50  0000 C CNN
 F 2 "" H 1550 3850 50  0001 C CNN
@@
 $EndComp
 $Comp
-L Device:C_Small C?
+L Device:C_Small C7
 U 1 1 618A1004
 P 1150 4300
-F 0 "C?" H 1242 4346 50  0000 L CNN
+F 0 "C7" H 1242 4346 50  0000 L CNN
 F 1 "100n" H 1242 4255 50  0000 L CNN
 F 2 "" H 1150 4300 50  0001 C CNN
@@
 	1150 4650 1150 4550
 $Comp
-L Jumper:SolderJumper_2_Open JP?
+L Jumper:SolderJumper_2_Open JP3
 U 1 1 618A7F56
 P 1900 4300
-F 0 "JP?" V 1946 4212 50  0000 R CNN
+F 0 "JP3" V 1946 4212 50  0000 R CNN
 F 1 "NRST" V 1855 4212 50  0000 R CNN
 F 2 "" H 1900 4300 50  0001 C CNN
@@
 SWCLK
 $Comp
-L Device:R_Small R?
+L Device:R_Small R13
 U 1 1 618ADFBE
 P 2650 4250
-F 0 "R?" H 2709 4296 50  0000 L CNN
+F 0 "R13" H 2709 4296 50  0000 L CNN
 F 1 "1k" H 2709 4205 50  0000 L CNN
 F 2 "" H 2650 4250 50  0001 C CNN
@@
 NC
 $Comp
-L Device:R_Small R?
+L Device:R_Small R14
 U 1 1 618B5399
 P 3100 4250
-F 0 "R?" H 3159 4296 50  0000 L CNN
+F 0 "R14" H 3159 4296 50  0000 L CNN
 F 1 "100k" H 3159 4205 50  0000 L CNN
 F 2 "" H 3100 4250 50  0001 C CNN

Commit message: added testpoints to daughterboards, updated readme
Parts:
- added TP21: SWDIO, symbol Connector:TestPoint
- added TP22: SWCLK, symbol Connector:TestPoint
- added TP23: SWO, symbol Connector:TestPoint
- added TP24: RESETN, symbol Connector:TestPoint
- added TP25: USART_TX, symbol Connector:TestPoint
- added TP26: USART_RX, symbol Connector:TestPoint
- added TP27: GPIO0, symbol Connector:TestPoint
- added TP28: GPIO1, symbol Connector:TestPoint
- added TP29: GPIO2, symbol Connector:TestPoint
- added TP30: GPIO3, symbol Connector:TestPoint
Connections:
- net GPIO2.0: now also TP27.1
- net GPIO2.1: now also TP28.1
- net GPIO2.2: now also TP29.1
- net GPIO2.3: now also TP30.1
- net RST_2: now also TP24.1
- net TCK|SWDCLK_2: now also TP22.1
- net TDO|SWO_2: now also TP23.1
- net TMS|SWDIO_2: now also TP21.1
- net UART_RxD2: now also TP25.1
- net UART_TxD2: now also TP26.1
Changed lines of the file:
@@
 NoConn ~ 6400 4150
 NoConn ~ 6400 4350
+$Comp
+L Connector:TestPoint TP21
+U 1 1 61908316
+P 2150 1700
+F 0 "TP21" V 2150 1900 50  0000 L CNN
+F 1 "SWDIO" V 2150 2250 50  0000 L CNN
+F 2 "" H 2350 1700 50  0001 C CNN
+F 3 "~" H 2350 1700 50  0001 C CNN
+	1    2150 1700
+	0    1    1    0
+$EndComp
+$Comp
+L Connector:TestPoint TP22
+U 1 1 6190B4C1
+P 2150 1800
+F 0 "TP22" V 2150 2000 50  0000 L CNN
+F 1 "SWCLK" V 2150 2350 50  0000 L CNN
+F 2 "" H 2350 1800 50  0001 C CNN
+F 3 "~" H 2350 1800 50  0001 C CNN
+	1    2150 1800
+	0    1    1    0
+$EndComp
+$Comp
+L Connector:TestPoint TP23
+U 1 1 6190B74B
+P 2150 1900
+F 0 "TP23" V 2150 2100 50  0000 L CNN
+F 1 "SWO" V 2150 2450 50  0000 L CNN
+F 2 "" H 2350 1900 50  0001 C CNN
+F 3 "~" H 2350 1900 50  0001 C CNN
+	1    2150 1900
+	0    1    1    0
+$EndComp
+$Comp
+L Connector:TestPoint TP24
+U 1 1 6190B914
+P 2150 2100
+F 0 "TP24" V 2150 2300 50  0000 L CNN
+F 1 "RESETN" V 2150 2650 50  0000 L CNN
+F 2 "" H 2350 2100 50  0001 C CNN
+F 3 "~" H 2350 2100 50  0001 C CNN
+	1    2150 2100
+	0    1    1    0
+$EndComp
+$Comp
+L Connector:TestPoint TP25
+U 1 1 6190C327
+P 2150 2600
+F 0 "TP25" V 2150 2800 50  0000 L CNN
+F 1 "USART_TX" V 2150 3150 50  0000 L CNN
+F 2 "" H 2350 2600 50  0001 C CNN
+F 3 "~" H 2350 2600 50  0001 C CNN
+	1    2150 2600
+	0    1    -1   0
+$EndComp
+$Comp
+L Connector:TestPoint TP26
+U 1 1 6190E9FD
+P 2150 2700
+F 0 "TP26" V 2150 2900 50  0000 L CNN
+F 1 "USART_RX" V 2150 3250 50  0000 L CNN
+F 2 "" H 2350 2700 50  0001 C CNN
+F 3 "~" H 2350 2700 50  0001 C CNN
+	1    2150 2700
+	0    1    -1   0
+$EndComp
+$Comp
+L Connector:TestPoint TP27
+U 1 1 6190ECF6
+P 2150 2800
+F 0 "TP27" V 2150 3000 50  0000 L CNN
+F 1 "GPIO0" V 2150 3350 50  0000 L CNN
+F 2 "" H 2350 2800 50  0001 C CNN
+F 3 "~" H 2350 2800 50  0001 C CNN
+	1    2150 2800
+	0    1    -1   0
+$EndComp
+$Comp
+L Connector:TestPoint TP28
+U 1 1 6190EE9D
+P 2150 2900
+F 0 "TP28" V 2150 3100 50  0000 L CNN
+F 1 "GPIO1" V 2150 3450 50  0000 L CNN
+F 2 "" H 2350 2900 50  0001 C CNN
+F 3 "~" H 2350 2900 50  0001 C CNN
+	1    2150 2900
+	0    1    -1   0
+$EndComp
+$Comp
+L Connector:TestPoint TP29
+U 1 1 6190F16D
+P 2150 3000
+F 0 "TP29" V 2150 3200 50  0000 L CNN
+F 1 "GPIO2" V 2150 3550 50  0000 L CNN
+F 2 "" H 2350 3000 50  0001 C CNN
+F 3 "~" H 2350 3000 50  0001 C CNN
+	1    2150 3000
+	0    1    -1   0
+$EndComp
+$Comp
+L Connector:TestPoint TP30
+U 1 1 6190F306
+P 2150 3100
+F 0 "TP30" V 2150 3300 50  0000 L CNN
+F 1 "GPIO3" V 2150 3650 50  0000 L CNN
+F 2 "" H 2350 3100 50  0001 C CNN
+F 3 "~" H 2350 3100 50  0001 C CNN
+	1    2150 3100
+	0    1    -1   0
+$EndComp
 $EndSCHEMATC

Commit message: finished ATSAMD daughterboard layout
Parts:
- removed TP24: RESETN, symbol Connector:TestPoint
- removed TP27: GPIO0, symbol Connector:TestPoint
- removed TP28: GPIO1, symbol Connector:TestPoint
- removed TP29: GPIO2, symbol Connector:TestPoint
- removed TP30: GPIO3, symbol Connector:TestPoint
- added C20: 100n, Capacitor_SMD:C_0603_1608Metric_Pad1.05x0.95mm_HandSolder, symbol Device:C_Small
- C10, C11, C12, C13, C14, C7, C8, C9: footprint (none) -> Capacitor_SMD:C_0603_1608Metric_Pad1.05x0.95mm_HandSolder
- JP3: footprint (none) -> Jumper:SolderJumper-2_P1.3mm_Open_TrianglePad1.0x1.5mm
- R11, R12, R13, R14: footprint (none) -> Resistor_SMD:R_0603_1608Metric_Pad1.05x0.95mm_HandSolder
- TP21, TP22, TP23, TP25, TP26: footprint (none) -> TestPoint:TestPoint_Pad_1.0x1.0mm
Connections:
- net +3V3: now also C20.1
- net GND: now also C20.2
Changed lines of the file:
@@
 F 0 "C10" H 6692 1496 50  0000 L CNN
 F 1 "10u" H 6692 1405 50  0000 L CNN
-F 2 "" H 6600 1450 50  0001 C CNN
+F 2 "Capacitor_SMD:C_0603_1608Metric_Pad1.05x0.95mm_HandSolder" H 6600 1450 50  0001 C CNN
 F 3 "~" H 6600 1450 50  0001 C CNN
 	1    6600 1450
@@
 F 0 "C9" H 4892 1496 50  0000 L CNN
 F 1 "4.7u" H 4892 1405 50  0000 L CNN
-F 2 "" H 4800 1450 50  0001 C CNN
+F 2 "Capacitor_SMD:C_0603_1608Metric_Pad1.05x0.95mm_HandSolder" H 4800 1450 50  0001 C CNN
 F 3 "~" H 4800 1450 50  0001 C CNN
 	1    4800 1450
@@
 F 0 "C12" H 7442 1496 50  0000 L CNN
 F 1 "100n" H 7442 1405 50  0000 L CNN
-F 2 "" H 7350 1450 50  0001 C CNN
+F 2 "Capacitor_SMD:C_0603_1608Metric_Pad1.05x0.95mm_HandSolder" H 7350 1450 50  0001 C CNN
 F 3 "~" H 7350 1450 50  0001 C CNN
 	1    7350 1450
@@
 F 0 "C8" H 4442 1496 50  0000 L CNN
 F 1 "100n" H 4442 1405 50  0000 L CNN
-F 2 "" H 4350 1450 50  0001 C CNN
+F 2 "Capacitor_SMD:C_0603_1608Metric_Pad1.05x0.95mm_HandSolder" H 4350 1450 50  0001 C CNN
 F 3 "~" H 4350 1450 50  0001 C CNN
 	1    4350 1450
@@
 F 0 "C13" H 7842 1496 50  0000 L CNN
 F 1 "100n" H 7842 1405 50  0000 L CNN
-F 2 "" H 7750 1450 50  0001 C CNN
+F 2 "Capacitor_SMD:C_0603_1608Metric_Pad1.05x0.95mm_HandSolder" H 7750 1450 50  0001 C CNN
 F 3 "~" H 7750 1450 50  0001 C CNN
 	1    7750 1450
@@
 F 0 "C14" H 8242 1496 50  0000 L CNN
 F 1 "100n" H 8242 1405 50  0000 L CNN
-F 2 "" H 8150 1450 50  0001 C CNN
+F 2 "Capacitor_SMD:C_0603_1608Metric_Pad1.05x0.95mm_HandSolder" H 8150 1450 50  0001 C CNN
 F 3 "~" H 8150 1450 50  0001 C CNN
 	1    8150 1450
@@
 F 0 "C11" H 7042 1496 50  0000 L CNN
 F 1 "1u" H 7042 1405 50  0000 L CNN
-F 2 "" H 6950 1450 50  0001 C CNN
+F 2 "Capacitor_SMD:C_0603_1608Metric_Pad1.05x0.95mm_HandSolder" H 6950 1450 50  0001 C CNN
 F 3 "~" H 6950 1450 50  0001 C CNN
 	1    6950 1450
@@
 L power:GND #PWR0121
 U 1 1 618934CB
-P 8150 1700
-F 0 "#PWR0121" H 8150 1450 50  0001 C CNN
-F 1 "GND" H 8155 1527 50  0000 C CNN
-F 2 "" H 8150 1700 50  0001 C CNN
-F 3 "" H 8150 1700 50  0001 C CNN
-	1    8150 1700
-	1    0    0    -1
-$EndComp
-Wire Wire Line
-	8150 1700 8150 1650
+P 8550 1700
+F 0 "#PWR0121" H 8550 1450 50  0001 C CNN
+F 1 "GND" H 8555 1527 50  0000 C CNN
+F 2 "" H 8550 1700 50  0001 C CNN
+F 3 "" H 8550 1700 50  0001 C CNN
+	1    8550 1700
+	1    0    0    -1
+$EndComp
 Wire Wire Line
 	6600 1550 6600 1650
 Wire Wire Line
 	6600 1650 6950 1650
-Connection ~ 8150 1650
 Wire Wire Line
 	8150 1650 8150 1550
@@
 L power:+3V3 #PWR0124
 U 1 1 61896848
-P 8150 1050
-F 0 "#PWR0124" H 8150 900 50  0001 C CNN
-F 1 "+3V3" H 8165 1223 50  0000 C CNN
-F 2 "" H 8150 1050 50  0001 C CNN
-F 3 "" H 8150 1050 50  0001 C CNN
-	1    8150 1050
-	1    0    0    -1
-$EndComp
-Wire Wire Line
-	8150 1150 8150 1050
-Connection ~ 8150 1150
+P 8550 1050
+F 0 "#PWR0124" H 8550 900 50  0001 C CNN
+F 1 "+3V3" H 8565 1223 50  0000 C CNN
+F 2 "" H 8550 1050 50  0001 C CNN
+F 3 "" H 8550 1050 50  0001 C CNN
+	1    8550 1050
+	1    0    0    -1
+$EndComp
+Wire Wire Line
+	8550 1150 8550 1050
 $Comp
 L power:GND #PWR0125
@@
 F 0 "R11" H 909 4346 50  0000 L CNN
 F 1 "10k" H 909 4255 50  0000 L CNN
-F 2 "" H 850 4300 50  0001 C CNN
+F 2 "Resistor_SMD:R_0603_1608Metric_Pad1.05x0.95mm_HandSolder" H 850 4300 50  0001 C CNN
 F 3 "~" H 850 4300 50  0001 C CNN
 	1    850  4300
@@
 F 0 "R12" V 1354 3850 50  0000 C CNN
 F 1 "330" V 1445 3850 50  0000 C CNN
-F 2 "" H 1550 3850 50  0001 C CNN
+F 2 "Resistor_SMD:R_0603_1608Metric_Pad1.05x0.95mm_HandSolder" H 1550 3850 50  0001 C CNN
 F 3 "~" H 1550 3850 50  0001 C CNN
 	1    1550 3850
@@
 F 0 "C7" H 1242 4346 50  0000 L CNN
 F 1 "100n" H 1242 4255 50  0000 L CNN
-F 2 "" H 1150 4300 50  0001 C CNN
+F 2 "Capacitor_SMD:C_0603_1608Metric_Pad1.05x0.95mm_HandSolder" H 1150 4300 50  0001 C CNN
 F 3 "~" H 1150 4300 50  0001 C CNN
 	1    1150 4300
@@
 F 0 "JP3" V 1946 4212 50  0000 R CNN
 F 1 "NRST" V 1855 4212 50  0000 R CNN
-F 2 "" H 1900 4300 50  0001 C CNN
+F 2 "Jumper:SolderJumper-2_P1.3mm_Open_TrianglePad1.0x1.5mm" H 1900 4300 50  0001 C CNN
 F 3 "~" H 1900 4300 50  0001 C CNN
 	1    1900 4300
@@
 F 0 "R13" H 2709 4296 50  0000 L CNN
 F 1 "1k" H 2709 4205 50  0000 L CNN
-F 2 "" H 2650 4250 50  0001 C CNN
+F 2 "Resistor_SMD:R_0603_1608Metric_Pad1.05x0.95mm_HandSolder" H 2650 4250 50  0001 C CNN
 F 3 "~" H 2650 4250 50  0001 C CNN
 	1    2650 4250
@@
 F 0 "R14" H 3159 4296 50  0000 L CNN
 F 1 "100k" H 3159 4205 50  0000 L CNN
-F 2 "" H 3100 4250 50  0001 C CNN
+F 2 "Resistor_SMD:R_0603_1608Metric_Pad1.05x0.95mm_HandSolder" H 3100 4250 50  0001 C CNN
 F 3 "~" H 3100 4250 50  0001 C CNN
 	1    3100 4250
@@
 F 0 "TP21" V 2150 1900 50  0000 L CNN
 F 1 "SWDIO" V 2150 2250 50  0000 L CNN
-F 2 "" H 2350 1700 50  0001 C CNN
+F 2 "TestPoint:TestPoint_Pad_1.0x1.0mm" H 2350 1700 50  0001 C CNN
 F 3 "~" H 2350 1700 50  0001 C CNN
 	1    2150 1700
@@
 F 0 "TP22" V 2150 2000 50  0000 L CNN
 F 1 "SWCLK" V 2150 2350 50  0000 L CNN
-F 2 "" H 2350 1800 50  0001 C CNN
+F 2 "TestPoint:TestPoint_Pad_1.0x1.0mm" H 2350 1800 50  0001 C CNN
 F 3 "~" H 2350 1800 50  0001 C CNN
 	1    2150 1800
@@
 F 0 "TP23" V 2150 2100 50  0000 L CNN
 F 1 "SWO" V 2150 2450 50  0000 L CNN
-F 2 "" H 2350 1900 50  0001 C CNN
+F 2 "TestPoint:TestPoint_Pad_1.0x1.0mm" H 2350 1900 50  0001 C CNN
 F 3 "~" H 2350 1900 50  0001 C CNN
 	1    2150 1900
-	0    1    1    0
-$EndComp
-$Comp
-L Connector:TestPoint TP24
-U 1 1 6190B914
-P 2150 2100
-F 0 "TP24" V 2150 2300 50  0000 L CNN
-F 1 "RESETN" V 2150 2650 50  0000 L CNN
-F 2 "" H 2350 2100 50  0001 C CNN
-F 3 "~" H 2350 2100 50  0001 C CNN
-	1    2150 2100
 	0    1    1    0
 $EndComp
@@
 F 0 "TP25" V 2150 2800 50  0000 L CNN
 F 1 "USART_TX" V 2150 3150 50  0000 L CNN
-F 2 "" H 2350 2600 50  0001 C CNN
+F 2 "TestPoint:TestPoint_Pad_1.0x1.0mm" H 2350 2600 50  0001 C CNN
 F 3 "~" H 2350 2600 50  0001 C CNN
 	1    2150 2600
@@
 F 0 "TP26" V 2150 2900 50  0000 L CNN
 F 1 "USART_RX" V 2150 3250 50  0000 L CNN
-F 2 "" H 2350 2700 50  0001 C CNN
+F 2 "TestPoint:TestPoint_Pad_1.0x1.0mm" H 2350 2700 50  0001 C CNN
 F 3 "~" H 2350 2700 50  0001 C CNN
 	1    2150 2700
@@
 $EndComp
 $Comp
-L Connector:TestPoint TP27
-U 1 1 6190ECF6
-P 2150 2800
-F 0 "TP27" V 2150 3000 50  0000 L CNN
-F 1 "GPIO0" V 2150 3350 50  0000 L CNN
-F 2 "" H 2350 2800 50  0001 C CNN
-F 3 "~" H 2350 2800 50  0001 C CNN
-	1    2150 2800
-	0    1    -1   0
-$EndComp
-$Comp
-L Connector:TestPoint TP28
-U 1 1 6190EE9D
-P 2150 2900
-F 0 "TP28" V 2150 3100 50  0000 L CNN
-F 1 "GPIO1" V 2150 3450 50  0000 L CNN
-F 2 "" H 2350 2900 50  0001 C CNN
-F 3 "~" H 2350 2900 50  0001 C CNN
-	1    2150 2900
-	0    1    -1   0
-$EndComp
-$Comp
-L Connector:TestPoint TP29
-U 1 1 6190F16D
-P 2150 3000
-F 0 "TP29" V 2150 3200 50  0000 L CNN
-F 1 "GPIO2" V 2150 3550 50  0000 L CNN
-F 2 "" H 2350 3000 50  0001 C CNN
-F 3 "~" H 2350 3000 50  0001 C CNN
-	1    2150 3000
-	0    1    -1   0
-$EndComp
-$Comp
-L Connector:TestPoint TP30
-U 1 1 6190F306
-P 2150 3100
-F 0 "TP30" V 2150 3300 50  0000 L CNN
-F 1 "GPIO3" V 2150 3650 50  0000 L CNN
-F 2 "" H 2350 3100 50  0001 C CNN
-F 3 "~" H 2350 3100 50  0001 C CNN
-	1    2150 3100
-	0    1    -1   0
-$EndComp
+L Device:C_Small C20
+U 1 1 6192C465
+P 8550 1450
+F 0 "C20" H 8642 1496 50  0000 L CNN
+F 1 "100n" H 8642 1405 50  0000 L CNN
+F 2 "Capacitor_SMD:C_0603_1608Metric_Pad1.05x0.95mm_HandSolder" H 8550 1450 50  0001 C CNN
+F 3 "~" H 8550 1450 50  0001 C CNN
+	1    8550 1450
+	1    0    0    -1
+$EndComp
+Wire Wire Line
+	8150 1150 8550 1150
+Connection ~ 8150 1150
+Wire Wire Line
+	8550 1350 8550 1150
+Connection ~ 8550 1150
+Wire Wire Line
+	8550 1550 8550 1650
+Wire Wire Line
+	8150 1650 8550 1650
+Connection ~ 8150 1650
+Connection ~ 8550 1650
+Wire Wire Line
+	8550 1650 8550 1700
 $EndSCHEMATC
