File: daughterboard/NRF_00/target0.sch (KiCad schematic (older format))
At the start: 8 parts

Commit message: finished NRF daughterboard schematics
Parts:
- gave numbers to parts that had none: 8
Changed lines of the file:
@@
 Add your target here and connect it to the provided Debug and GPIO/UART connections.\n\nDebug and GPIO/UART connections are 5V tolerant. Min signal level is 3.3V
 $Comp
-L hive_daughterboard:BT40E U?
+L hive_daughterboard:BT40E U0
 U 1 1 619125EF
 P 7350 1900
-F 0 "U?" H 6550 2100 50  0000 C CNN
+F 0 "U0" H 6550 2100 50  0000 C CNN
 F 1 "BT40E" H 6650 2000 50  0000 C CNN
 F 2 "hive_daughterboard:BT40E" H 7350 1900 50  0001 C CNN
@@
 $EndComp
 $Comp
-L power:GND #PWR?
+L power:GND #PWR011
 U 1 1 619137F3
 P 7150 3100
-F 0 "#PWR?" H 7150 2850 50  0001 C CNN
+F 0 "#PWR011" H 7150 2850 50  0001 C CNN
 F 1 "GND" H 7155 2927 50  0000 C CNN
 F 2 "" H 7150 3100 50  0001 C CNN
@@
 SWDCLK
 $Comp
-L Device:R_Small R?
+L Device:R_Small R3
 U 1 1 61917F77
 P 950 4000
-F 0 "R?" H 1009 4046 50  0000 L CNN
+F 0 "R3" H 1009 4046 50  0000 L CNN
 F 1 "100k" H 1009 3955 50  0000 L CNN
 F 2 "" H 950 4000 50  0001 C CNN
@@
 NRST
 $Comp
-L power:+3V3 #PWR?
+L power:+3V3 #PWR08
 U 1 1 61919DFF
 P 950 4400
-F 0 "#PWR?" H 950 4250 50  0001 C CNN
+F 0 "#PWR08" H 950 4250 50  0001 C CNN
 F 1 "+3V3" H 965 4573 50  0000 C CNN
 F 2 "" H 950 4400 50  0001 C CNN
@@
 	950  4400 950  4100
 $Comp
-L Device:C_Small C?
+L Device:C_Small C9
 U 1 1 6191B654
 P 1400 4000
-F 0 "C?" H 1492 4046 50  0000 L CNN
+F 0 "C9" H 1492 4046 50  0000 L CNN
 F 1 "100n" H 1492 3955 50  0000 L CNN
 F 2 "" H 1400 4000 50  0001 C CNN
@@
 	950  3750 950  3350
 $Comp
-L power:GND #PWR?
+L power:GND #PWR09
 U 1 1 6191C425
 P 1850 4400
-F 0 "#PWR?" H 1850 4150 50  0001 C CNN
+F 0 "#PWR09" H 1850 4150 50  0001 C CNN
 F 1 "GND" H 1855 4227 50  0000 C CNN
 F 2 "" H 1850 4400 50  0001 C CNN
@@
 $EndComp
 $Comp
-L Jumper:SolderJumper_2_Open JP?
+L Jumper:SolderJumper_2_Open JP2
 U 1 1 6191D1B0
 P 1850 4050
-F 0 "JP?" V 1804 4118 50  0000 L CNN
+F 0 "JP2" V 1804 4118 50  0000 L CNN
 F 1 "NRST" V 1895 4118 50  0000 L CNN
 F 2 "" H 1850 4050 50  0001 C CNN
@@
 	7350 1450 7600 1450
 $Comp
-L Device:C_Small C?
+L Device:C_Small C10
 U 1 1 61922430
 P 7600 1600
-F 0 "C?" H 7692 1646 50  0000 L CNN
+F 0 "C10" H 7692 1646 50  0000 L CNN
 F 1 "100n" H 7692 1555 50  0000 L CNN
 F 2 "" H 7600 1600 50  0001 C CNN
@@
 $EndComp
 $Comp
-L Device:C_Small C?
+L Device:C_Small C11
 U 1 1 619236BB
 P 8000 1600
-F 0 "C?" H 8092 1646 50  0000 L CNN
+F 0 "C11" H 8092 1646 50  0000 L CNN
 F 1 "4.7u" H 8092 1555 50  0000 L CNN
 F 2 "" H 8000 1600 50  0001 C CNN
@@
 $EndComp
 $Comp
-L Device:C_Small C?
+L Device:C_Small C12
 U 1 1 61923D20
 P 8400 1600
-F 0 "C?" H 8492 1646 50  0000 L CNN
+F 0 "C12" H 8492 1646 50  0000 L CNN
 F 1 "10u" H 8492 1555 50  0000 L CNN
 F 2 "" H 8400 1600 50  0001 C CNN
@@
 	7600 1450 8000 1450
 $Comp
-L power:+3V3 #PWR?
+L power:+3V3 #PWR012
 U 1 1 61928507
 P 8400 1350
-F 0 "#PWR?" H 8400 1200 50  0001 C CNN
+F 0 "#PWR012" H 8400 1200 50  0001 C CNN
 F 1 "+3V3" H 8415 1523 50  0000 C CNN
 F 2 "" H 8400 1350 50  0001 C CNN
@@
 Connection ~ 8400 1450
 $Comp
-L power:GND #PWR?
+L power:GND #PWR013
 U 1 1 61929331
 P 8400 1900
-F 0 "#PWR?" H 8400 1650 50  0001 C CNN
+F 0 "#PWR013" H 8400 1650 50  0001 C CNN
 F 1 "GND" H 8405 1727 50  0000 C CNN
 F 2 "" H 8400 1900 50  0001 C CNN
@@
 NC
 $Comp
-L Device:R_Small R?
+L Device:R_Small R4
 U 1 1 61932627
 P 2400 4000
-F 0 "R?" H 2459 4046 50  0000 L CNN
+F 0 "R4" H 2459 4046 50  0000 L CNN
 F 1 "100k" H 2459 3955 50  0000 L CNN
 F 2 "" H 2400 4000 50  0001 C CNN
@@
 $EndComp
 $Comp
-L power:GND #PWR?
+L power:GND #PWR010
 U 1 1 6193262D
 P 2400 4400
-F 0 "#PWR?" H 2400 4150 50  0001 C CNN
+F 0 "#PWR010" H 2400 4150 50  0001 C CNN
 F 1 "GND" H 2405 4227 50  0000 C CNN
 F 2 "" H 2400 4400 50  0001 C CNN

Commit message: added testpoints to daughterboards, updated readme
Parts:
- added TP12: SWDIO, symbol Connector:TestPoint
- added TP13: SWDCLK, symbol Connector:TestPoint
- added TP14: SWO, symbol Connector:TestPoint
- added TP15: NRST, symbol Connector:TestPoint
- added TP16: UART_TX, symbol Connector:TestPoint
- added TP17: UART_RX, symbol Connector:TestPoint
- added TP18: GPIO0, symbol Connector:TestPoint
- added TP19: GPIO1, symbol Connector:TestPoint
- added TP20: GPIO2, symbol Connector:TestPoint
- added TP21: GPIO3, symbol Connector:TestPoint
Connections:
- net GPIO0.0: now also TP18.1
- net GPIO0.1: now also TP19.1
- net GPIO0.2: now also TP20.1
- net GPIO0.3: now also TP21.1
- net RST_0: now also TP15.1
- net TCK|SWDCLK_0: now also TP13.1
- net TDO|SWO_0: now also TP14.1
- net TMS|SWDIO_0: now also TP12.1
- net UART_RxD0: now also TP16.1
- net UART_TxD0: now also TP17.1
Changed lines of the file:
@@
 Wire Wire Line
 	2400 4400 2400 4100
+$Comp
+L Connector:TestPoint TP?
+U 1 1 6190F334
+P 2250 2050
+AR Path="/616688D6/6190F334" Ref="TP?"  Part="1"
+AR Path="/61668514/6190F334" Ref="TP15"  Part="1"
+F 0 "TP15" V 2250 2250 50  0000 L CNN
+F 1 "NRST" V 2250 2600 50  0000 L CNN
+F 2 "" H 2450 2050 50  0001 C CNN
+F 3 "~" H 2450 2050 50  0001 C CNN
+	1    2250 2050
+	0    1    1    0
+$EndComp
+$Comp
+L Connector:TestPoint TP?
+U 1 1 6190F33A
+P 2250 1850
+AR Path="/616688D6/6190F33A" Ref="TP?"  Part="1"
+AR Path="/61668514/6190F33A" Ref="TP14"  Part="1"
+F 0 "TP14" V 2250 2050 50  0000 L CNN
+F 1 "SWO" V 2250 2400 50  0000 L CNN
+F 2 "" H 2450 1850 50  0001 C CNN
+F 3 "~" H 2450 1850 50  0001 C CNN
+	1    2250 1850
+	0    1    1    0
+$EndComp
+$Comp
+L Connector:TestPoint TP?
+U 1 1 6190F340
+P 2250 1750
+AR Path="/616688D6/6190F340" Ref="TP?"  Part="1"
+AR Path="/61668514/6190F340" Ref="TP13"  Part="1"
+F 0 "TP13" V 2250 1950 50  0000 L CNN
+F 1 "SWDCLK" V 2250 2300 50  0000 L CNN
+F 2 "" H 2450 1750 50  0001 C CNN
+F 3 "~" H 2450 1750 50  0001 C CNN
+	1    2250 1750
+	0    1    1    0
+$EndComp
+$Comp
+L Connector:TestPoint TP?
+U 1 1 6190F346
+P 2250 1650
+AR Path="/616688D6/6190F346" Ref="TP?"  Part="1"
+AR Path="/61668514/6190F346" Ref="TP12"  Part="1"
+F 0 "TP12" V 2250 1850 50  0000 L CNN
+F 1 "SWDIO" V 2250 2200 50  0000 L CNN
+F 2 "" H 2450 1650 50  0001 C CNN
+F 3 "~" H 2450 1650 50  0001 C CNN
+	1    2250 1650
+	0    1    1    0
+$EndComp
+$Comp
+L Connector:TestPoint TP?
+U 1 1 6190F34C
+P 2250 2550
+AR Path="/616688D6/6190F34C" Ref="TP?"  Part="1"
+AR Path="/61668514/6190F34C" Ref="TP16"  Part="1"
+F 0 "TP16" V 2250 2750 50  0000 L CNN
+F 1 "UART_TX" V 2250 3100 50  0000 L CNN
+F 2 "" H 2450 2550 50  0001 C CNN
+F 3 "~" H 2450 2550 50  0001 C CNN
+	1    2250 2550
+	0    1    1    0
+$EndComp
+$Comp
+L Connector:TestPoint TP?
+U 1 1 6190F352
+P 2250 2650
+AR Path="/616688D6/6190F352" Ref="TP?"  Part="1"
+AR Path="/61668514/6190F352" Ref="TP17"  Part="1"
+F 0 "TP17" V 2250 2850 50  0000 L CNN
+F 1 "UART_RX" V 2250 3200 50  0000 L CNN
+F 2 "" H 2450 2650 50  0001 C CNN
+F 3 "~" H 2450 2650 50  0001 C CNN
+	1    2250 2650
+	0    1    1    0
+$EndComp
+$Comp
+L Connector:TestPoint TP?
+U 1 1 6190F358
+P 2250 2750
+AR Path="/616688D6/6190F358" Ref="TP?"  Part="1"
+AR Path="/61668514/6190F358" Ref="TP18"  Part="1"
+F 0 "TP18" V 2250 2950 50  0000 L CNN
+F 1 "GPIO0" V 2250 3300 50  0000 L CNN
+F 2 "" H 2450 2750 50  0001 C CNN
+F 3 "~" H 2450 2750 50  0001 C CNN
+	1    2250 2750
+	0    1    1    0
+$EndComp
+$Comp
+L Connector:TestPoint TP?
+U 1 1 6190F35E
+P 2250 2850
+AR Path="/616688D6/6190F35E" Ref="TP?"  Part="1"
+AR Path="/61668514/6190F35E" Ref="TP19"  Part="1"
+F 0 "TP19" V 2250 3050 50  0000 L CNN
+F 1 "GPIO1" V 2250 3400 50  0000 L CNN
+F 2 "" H 2450 2850 50  0001 C CNN
+F 3 "~" H 2450 2850 50  0001 C CNN
+	1    2250 2850
+	0    1    1    0
+$EndComp
+$Comp
+L Connector:TestPoint TP?
+U 1 1 6190F364
+P 2250 2950
+AR Path="/616688D6/6190F364" Ref="TP?"  Part="1"
+AR Path="/61668514/6190F364" Ref="TP20"  Part="1"
+F 0 "TP20" V 2250 3150 50  0000 L CNN
+F 1 "GPIO2" V 2250 3500 50  0000 L CNN
+F 2 "" H 2450 2950 50  0001 C CNN
+F 3 "~" H 2450 2950 50  0001 C CNN
+	1    2250 2950
+	0    1    1    0
+$EndComp
+$Comp
+L Connector:TestPoint TP?
+U 1 1 6190F36A
+P 2250 3050
+AR Path="/616688D6/6190F36A" Ref="TP?"  Part="1"
+AR Path="/61668514/6190F36A" Ref="TP21"  Part="1"
+F 0 "TP21" V 2250 3250 50  0000 L CNN
+F 1 "GPIO3" V 2250 3600 50  0000 L CNN
+F 2 "" H 2450 3050 50  0001 C CNN
+F 3 "~" H 2450 3050 50  0001 C CNN
+	1    2250 3050
+	0    1    1    0
+$EndComp
 $EndSCHEMATC

Commit message: finished NRF daughterboard layout
Parts:
- removed TP15: NRST, symbol Connector:TestPoint
- removed TP18: GPIO0, symbol Connector:TestPoint
- removed TP19: GPIO1, symbol Connector:TestPoint
- removed TP20: GPIO2, symbol Connector:TestPoint
- removed TP21: GPIO3, symbol Connector:TestPoint
- C10, C11, C12, C9: footprint (none) -> Capacitor_SMD:C_0603_1608Metric_Pad1.05x0.95mm_HandSolder
- JP2: footprint (none) -> Jumper:SolderJumper-2_P1.3mm_Open_TrianglePad1.0x1.5mm
- R3, R4: footprint (none) -> Resistor_SMD:R_0603_1608Metric_Pad1.05x0.95mm_HandSolder
- TP12, TP13, TP14, TP16, TP17: footprint (none) -> TestPoint:TestPoint_Pad_1.0x1.0mm
Changed lines of the file:
@@
 F 0 "R3" H 1009 4046 50  0000 L CNN
 F 1 "100k" H 1009 3955 50  0000 L CNN
-F 2 "" H 950 4000 50  0001 C CNN
+F 2 "Resistor_SMD:R_0603_1608Metric_Pad1.05x0.95mm_HandSolder" H 950 4000 50  0001 C CNN
 F 3 "~" H 950 4000 50  0001 C CNN
 	1    950  4000
@@
 F 0 "C9" H 1492 4046 50  0000 L CNN
 F 1 "100n" H 1492 3955 50  0000 L CNN
-F 2 "" H 1400 4000 50  0001 C CNN
+F 2 "Capacitor_SMD:C_0603_1608Metric_Pad1.05x0.95mm_HandSolder" H 1400 4000 50  0001 C CNN
 F 3 "~" H 1400 4000 50  0001 C CNN
 	1    1400 4000
@@
 F 0 "JP2" V 1804 4118 50  0000 L CNN
 F 1 "NRST" V 1895 4118 50  0000 L CNN
-F 2 "" H 1850 4050 50  0001 C CNN
+F 2 "Jumper:SolderJumper-2_P1.3mm_Open_TrianglePad1.0x1.5mm" H 1850 4050 50  0001 C CNN
 F 3 "~" H 1850 4050 50  0001 C CNN
 	1    1850 4050
@@
 F 0 "C10" H 7692 1646 50  0000 L CNN
 F 1 "100n" H 7692 1555 50  0000 L CNN
-F 2 "" H 7600 1600 50  0001 C CNN
+F 2 "Capacitor_SMD:C_0603_1608Metric_Pad1.05x0.95mm_HandSolder" H 7600 1600 50  0001 C CNN
 F 3 "~" H 7600 1600 50  0001 C CNN
 	1    7600 1600
@@
 F 0 "C11" H 8092 1646 50  0000 L CNN
 F 1 "4.7u" H 8092 1555 50  0000 L CNN
-F 2 "" H 8000 1600 50  0001 C CNN
+F 2 "Capacitor_SMD:C_0603_1608Metric_Pad1.05x0.95mm_HandSolder" H 8000 1600 50  0001 C CNN
 F 3 "~" H 8000 1600 50  0001 C CNN
 	1    8000 1600
@@
 F 0 "C12" H 8492 1646 50  0000 L CNN
 F 1 "10u" H 8492 1555 50  0000 L CNN
-F 2 "" H 8400 1600 50  0001 C CNN
+F 2 "Capacitor_SMD:C_0603_1608Metric_Pad1.05x0.95mm_HandSolder" H 8400 1600 50  0001 C CNN
 F 3 "~" H 8400 1600 50  0001 C CNN
 	1    8400 1600
@@
 F 0 "R4" H 2459 4046 50  0000 L CNN
 F 1 "100k" H 2459 3955 50  0000 L CNN
-F 2 "" H 2400 4000 50  0001 C CNN
+F 2 "Resistor_SMD:R_0603_1608Metric_Pad1.05x0.95mm_HandSolder" H 2400 4000 50  0001 C CNN
 F 3 "~" H 2400 4000 50  0001 C CNN
 	1    2400 4000
@@
 $Comp
 L Connector:TestPoint TP?
-U 1 1 6190F334
-P 2250 2050
-AR Path="/616688D6/6190F334" Ref="TP?"  Part="1"
-AR Path="/61668514/6190F334" Ref="TP15"  Part="1"
-F 0 "TP15" V 2250 2250 50  0000 L CNN
-F 1 "NRST" V 2250 2600 50  0000 L CNN
-F 2 "" H 2450 2050 50  0001 C CNN
-F 3 "~" H 2450 2050 50  0001 C CNN
-	1    2250 2050
-	0    1    1    0
-$EndComp
-$Comp
-L Connector:TestPoint TP?
 U 1 1 6190F33A
 P 2250 1850
@@
 F 0 "TP14" V 2250 2050 50  0000 L CNN
 F 1 "SWO" V 2250 2400 50  0000 L CNN
-F 2 "" H 2450 1850 50  0001 C CNN
+F 2 "TestPoint:TestPoint_Pad_1.0x1.0mm" H 2450 1850 50  0001 C CNN
 F 3 "~" H 2450 1850 50  0001 C CNN
 	1    2250 1850
@@
 F 0 "TP13" V 2250 1950 50  0000 L CNN
 F 1 "SWDCLK" V 2250 2300 50  0000 L CNN
-F 2 "" H 2450 1750 50  0001 C CNN
+F 2 "TestPoint:TestPoint_Pad_1.0x1.0mm" H 2450 1750 50  0001 C CNN
 F 3 "~" H 2450 1750 50  0001 C CNN
 	1    2250 1750
@@
 F 0 "TP12" V 2250 1850 50  0000 L CNN
 F 1 "SWDIO" V 2250 2200 50  0000 L CNN
-F 2 "" H 2450 1650 50  0001 C CNN
+F 2 "TestPoint:TestPoint_Pad_1.0x1.0mm" H 2450 1650 50  0001 C CNN
 F 3 "~" H 2450 1650 50  0001 C CNN
 	1    2250 1650
@@
 F 0 "TP16" V 2250 2750 50  0000 L CNN
 F 1 "UART_TX" V 2250 3100 50  0000 L CNN
-F 2 "" H 2450 2550 50  0001 C CNN
+F 2 "TestPoint:TestPoint_Pad_1.0x1.0mm" H 2450 2550 50  0001 C CNN
 F 3 "~" H 2450 2550 50  0001 C CNN
 	1    2250 2550
@@
 F 0 "TP17" V 2250 2850 50  0000 L CNN
 F 1 "UART_RX" V 2250 3200 50  0000 L CNN
-F 2 "" H 2450 2650 50  0001 C CNN
+F 2 "TestPoint:TestPoint_Pad_1.0x1.0mm" H 2450 2650 50  0001 C CNN
 F 3 "~" H 2450 2650 50  0001 C CNN
 	1    2250 2650
 	0    1    1    0
 $EndComp
-$Comp
-L Connector:TestPoint TP?
-U 1 1 6190F358
-P 2250 2750
-AR Path="/616688D6/6190F358" Ref="TP?"  Part="1"
-AR Path="/61668514/6190F358" Ref="TP18"  Part="1"
-F 0 "TP18" V 2250 2950 50  0000 L CNN
-F 1 "GPIO0" V 2250 3300 50  0000 L CNN
-F 2 "" H 2450 2750 50  0001 C CNN
-F 3 "~" H 2450 2750 50  0001 C CNN
-	1    2250 2750
-	0    1    1    0
-$EndComp
-$Comp
-L Connector:TestPoint TP?
-U 1 1 6190F35E
-P 2250 2850
-AR Path="/616688D6/6190F35E" Ref="TP?"  Part="1"
-AR Path="/61668514/6190F35E" Ref="TP19"  Part="1"
-F 0 "TP19" V 2250 3050 50  0000 L CNN
-F 1 "GPIO1" V 2250 3400 50  0000 L CNN
-F 2 "" H 2450 2850 50  0001 C CNN
-F 3 "~" H 2450 2850 50  0001 C CNN
-	1    2250 2850
-	0    1    1    0
-$EndComp
-$Comp
-L Connector:TestPoint TP?
-U 1 1 6190F364
-P 2250 2950
-AR Path="/616688D6/6190F364" Ref="TP?"  Part="1"
-AR Path="/61668514/6190F364" Ref="TP20"  Part="1"
-F 0 "TP20" V 2250 3150 50  0000 L CNN
-F 1 "GPIO2" V 2250 3500 50  0000 L CNN
-F 2 "" H 2450 2950 50  0001 C CNN
-F 3 "~" H 2450 2950 50  0001 C CNN
-	1    2250 2950
-	0    1    1    0
-$EndComp
-$Comp
-L Connector:TestPoint TP?
-U 1 1 6190F36A
-P 2250 3050
-AR Path="/616688D6/6190F36A" Ref="TP?"  Part="1"
-AR Path="/61668514/6190F36A" Ref="TP21"  Part="1"
-F 0 "TP21" V 2250 3250 50  0000 L CNN
-F 1 "GPIO3" V 2250 3600 50  0000 L CNN
-F 2 "" H 2450 3050 50  0001 C CNN
-F 3 "~" H 2450 3050 50  0001 C CNN
-	1    2250 3050
-	0    1    1    0
-$EndComp
