File: daughterboard/NRF_00/NRF_00.kicad_pcb (KiCad board)
At the start: 4 copper layers, 67 x 50 mm, 56 parts, among them J1 m2_keyA_67pin_daughterboard, U0 BT40E, U1 nRF52832-QFAB-T, U2 NRF52840-USB-DONGLE, U3 NRF51822-QFAC-R7

Commit message: fixed NRF51822 footprint soldermask, fixed SilÃkscreen of ESP32_SIFIVE daughterboard
Parts:
- U3: value NRF51822-QFAC-R7 -> QFN40P600X600X90-49N
Changed lines of the file:
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@@
       (effects (font (size 1.00089 1.00089) (thickness 0.15)) (justify mirror))
     )
-    (fp_text value NRF51822-QFAC-R7 (at 8.92542 -4.578065 90) (layer B.Fab)
+    (fp_text value QFN40P600X600X90-49N (at 8.92542 -4.578065 90) (layer B.Fab)
       (effects (font (size 1.002858 1.002858) (thickness 0.15)) (justify mirror))
     )
@@
     (fp_circle (center -2.2 2.2) (end -1.976394 2.2) (layer B.Fab) (width 0.127))
     (fp_poly (pts (xy -1.45345 1.45) (xy 1.45 1.45) (xy 1.45 -1.45345) (xy -1.45345 -1.45345)) (layer B.Paste) (width 0.01))
-    (fp_poly (pts (xy 1.77879 3.175) (xy 2.625 3.175) (xy 2.625 2.83103) (xy 1.77879 2.83103)) (layer B.Mask) (width 0.01))
-    (fp_poly (pts (xy 1.37745 3.175) (xy 2.225 3.175) (xy 2.225 2.83004) (xy 1.37745 2.83004)) (layer B.Mask) (width 0.01))
-    (fp_poly (pts (xy 0.978074 3.175) (xy 1.825 3.175) (xy 1.825 2.83391) (xy 0.978074 2.83391)) (layer B.Mask) (width 0.01))
-    (fp_poly (pts (xy 0.576567 3.175) (xy 1.425 3.175) (xy 1.425 2.8327) (xy 0.576567 2.8327)) (layer B.Mask) (width 0.01))
-    (fp_poly (pts (xy 0.175592 3.175) (xy 1.025 3.175) (xy 1.025 2.83456) (xy 0.175592 2.83456)) (layer B.Mask) (width 0.01))
-    (fp_poly (pts (xy -0.225054 3.175) (xy 0.625 3.175) (xy 0.625 2.82567) (xy -0.225054 2.82567)) (layer B.Mask) (width 0.01))
-    (fp_poly (pts (xy -0.626353 3.175) (xy 0.225 3.175) (xy 0.225 2.83111) (xy -0.626353 2.83111)) (layer B.Mask) (width 0.01))
-    (fp_poly (pts (xy -1.02675 3.175) (xy -0.175 3.175) (xy -0.175 2.82982) (xy -1.02675 2.82982)) (layer B.Mask) (width 0.01))
-    (fp_poly (pts (xy -1.42857 3.175) (xy -0.575 3.175) (xy -0.575 2.83207) (xy -1.42857 2.83207)) (layer B.Mask) (width 0.01))
-    (fp_poly (pts (xy -1.82885 3.175) (xy -0.975 3.175) (xy -0.975 2.83097) (xy -1.82885 2.83097)) (layer B.Mask) (width 0.01))
-    (fp_poly (pts (xy -2.22964 3.175) (xy -1.375 3.175) (xy -1.375 2.8309) (xy -2.22964 2.8309)) (layer B.Mask) (width 0.01))
-    (fp_poly (pts (xy -2.62769 3.175) (xy -1.775 3.175) (xy -1.775 2.8279) (xy -2.62769 2.8279)) (layer B.Mask) (width 0.01))
+    (fp_poly (pts (xy 2.02879 2.575) (xy 2.02879 3.42121) (xy 2.37276 3.42121) (xy 2.37276 2.575)) (layer B.Mask) (width 0.01))
+    (fp_poly (pts (xy 1.62745 2.575) (xy 1.62745 3.42255) (xy 1.97241 3.42255) (xy 1.97241 2.575)) (layer B.Mask) (width 0.01))
+    (fp_poly (pts (xy 1.228074 2.575) (xy 1.228074 3.421926) (xy 1.569164 3.421926) (xy 1.569164 2.575)) (layer B.Mask) (width 0.01))
+    (fp_poly (pts (xy 0.826567 2.575) (xy 0.826567 3.423433) (xy 1.168867 3.423433) (xy 1.168867 2.575)) (layer B.Mask) (width 0.01))
+    (fp_poly (pts (xy 0.425592 2.575) (xy 0.425592 3.424408) (xy 0.766032 3.424408) (xy 0.766032 2.575)) (layer B.Mask) (width 0.01))
+    (fp_poly (pts (xy 0.024946 2.575) (xy 0.024946 3.425054) (xy 0.374276 3.425054) (xy 0.374276 2.575)) (layer B.Mask) (width 0.01))
+    (fp_poly (pts (xy -0.376353 2.575) (xy -0.376353 3.426353) (xy -0.032463 3.426353) (xy -0.032463 2.575)) (layer B.Mask) (width 0.01))
+    (fp_poly (pts (xy -0.77675 2.575) (xy -0.77675 3.42675) (xy -0.43157 3.42675) (xy -0.43157 2.575)) (layer B.Mask) (width 0.01))
+    (fp_poly (pts (xy -1.17857 2.575) (xy -1.17857 3.42857) (xy -0.83564 3.42857) (xy -0.83564 2.575)) (layer B.Mask) (width 0.01))
+    (fp_poly (pts (xy -1.57885 2.575) (xy -1.57885 3.42885) (xy -1.23482 3.42885) (xy -1.23482 2.575)) (layer B.Mask) (width 0.01))
+    (fp_poly (pts (xy -1.97964 2.575) (xy -1.97964 3.42964) (xy -1.63554 3.42964) (xy -1.63554 2.575)) (layer B.Mask) (width 0.01))
+    (fp_poly (pts (xy -2.37769 2.575) (xy -2.37769 3.42769) (xy -2.03059 3.42769) (xy -2.03059 2.575)) (layer B.Mask) (width 0.01))
     (fp_poly (pts (xy 2.57967 -2.025) (xy 3.425 -2.025) (xy 3.425 -2.37931) (xy 2.57967 -2.37931)) (layer B.Mask) (width 0.01))
     (fp_poly (pts (xy 2.57935 -1.625) (xy 3.425 -1.625) (xy 3.425 -1.97834) (xy 2.57935 -1.97834)) (layer B.Mask) (width 0.01))
@@
     (fp_poly (pts (xy 2.57837 1.975) (xy 3.425 1.975) (xy 3.425 1.62713) (xy 2.57837 1.62713)) (layer B.Mask) (width 0.01))
     (fp_poly (pts (xy 2.58395 2.375) (xy 3.425 2.375) (xy 3.425 2.03204) (xy 2.58395 2.03204)) (layer B.Mask) (width 0.01))
-    (fp_poly (pts (xy 1.77924 -2.825) (xy 2.625 -2.825) (xy 2.625 -3.18258) (xy 1.77924 -3.18258)) (layer B.Mask) (width 0.01))
-    (fp_poly (pts (xy 1.37887 -2.825) (xy 2.225 -2.825) (xy 2.225 -3.18395) (xy 1.37887 -3.18395)) (layer B.Mask) (width 0.01))
-    (fp_poly (pts (xy 0.977083 -2.825) (xy 1.825 -2.825) (xy 1.825 -3.18178) (xy 0.977083 -3.18178)) (layer B.Mask) (width 0.01))
-    (fp_poly (pts (xy 0.577004 -2.825) (xy 1.425 -2.825) (xy 1.425 -3.18606) (xy 0.577004 -3.18606)) (layer B.Mask) (width 0.01))
-    (fp_poly (pts (xy 0.175613 -2.825) (xy 1.025 -2.825) (xy 1.025 -3.18612) (xy 0.175613 -3.18612)) (layer B.Mask) (width 0.01))
-    (fp_poly (pts (xy -0.225615 -2.825) (xy 0.625 -2.825) (xy 0.625 -3.18366) (xy -0.225615 -3.18366)) (layer B.Mask) (width 0.01))
-    (fp_poly (pts (xy -0.626336 -2.825) (xy 0.225 -2.825) (xy 0.225 -3.18179) (xy -0.626336 -3.18179)) (layer B.Mask) (width 0.01))
-    (fp_poly (pts (xy -1.02662 -2.825) (xy -0.175 -2.825) (xy -0.175 -3.18003) (xy -1.02662 -3.18003)) (layer B.Mask) (width 0.01))
-    (fp_poly (pts (xy -1.42755 -2.825) (xy -0.575 -2.825) (xy -0.575 -3.18067) (xy -1.42755 -3.18067)) (layer B.Mask) (width 0.01))
-    (fp_poly (pts (xy -1.83067 -2.825) (xy -0.975 -2.825) (xy -0.975 -3.18487) (xy -1.83067 -3.18487)) (layer B.Mask) (width 0.01))
-    (fp_poly (pts (xy -2.22621 -2.825) (xy -1.375 -2.825) (xy -1.375 -3.17672) (xy -2.22621 -3.17672)) (layer B.Mask) (width 0.01))
-    (fp_poly (pts (xy -2.63077 -2.825) (xy -1.775 -2.825) (xy -1.775 -3.18198) (xy -2.63077 -3.18198)) (layer B.Mask) (width 0.01))
+    (fp_poly (pts (xy 2.02924 -3.435) (xy 2.02924 -2.58924) (xy 2.38682 -2.58924) (xy 2.38682 -3.435)) (layer B.Mask) (width 0.01))
+    (fp_poly (pts (xy 1.62887 -3.435) (xy 1.62887 -2.58887) (xy 1.98782 -2.58887) (xy 1.98782 -3.435)) (layer B.Mask) (width 0.01))
+    (fp_poly (pts (xy 1.227083 -3.435) (xy 1.227083 -2.587083) (xy 1.583863 -2.587083) (xy 1.583863 -3.435)) (layer B.Mask) (width 0.01))
+    (fp_poly (pts (xy 0.827004 -3.435) (xy 0.827004 -2.587004) (xy 1.188064 -2.587004) (xy 1.188064 -3.435)) (layer B.Mask) (width 0.01))
+    (fp_poly (pts (xy 0.425613 -3.435) (xy 0.425613 -2.585613) (xy 0.786733 -2.585613) (xy 0.786733 -3.435)) (layer B.Mask) (width 0.01))
+    (fp_poly (pts (xy 0.024385 -3.435) (xy 0.024385 -2.584385) (xy 0.383045 -2.584385) (xy 0.383045 -3.435)) (layer B.Mask) (width 0.01))
+    (fp_poly (pts (xy -0.376336 -3.435) (xy -0.376336 -2.583664) (xy -0.019546 -2.583664) (xy -0.019546 -3.435)) (layer B.Mask) (width 0.01))
+    (fp_poly (pts (xy -0.77662 -3.435) (xy -0.77662 -2.58338) (xy -0.42159 -2.58338) (xy -0.42159 -3.435)) (layer B.Mask) (width 0.01))
+    (fp_poly (pts (xy -1.17755 -3.435) (xy -1.17755 -2.58245) (xy -0.82188 -2.58245) (xy -0.82188 -3.435)) (layer B.Mask) (width 0.01))
+    (fp_poly (pts (xy -1.58067 -3.435) (xy -1.58067 -2.57933) (xy -1.2208 -2.57933) (xy -1.2208 -3.435)) (layer B.Mask) (width 0.01))
+    (fp_poly (pts (xy -1.97621 -3.435) (xy -1.97621 -2.58379) (xy -1.62449 -2.58379) (xy -1.62449 -3.435)) (layer B.Mask) (width 0.01))
+    (fp_poly (pts (xy -2.38077 -3.435) (xy -2.38077 -2.57923) (xy -2.02379 -2.57923) (xy -2.02379 -3.435)) (layer B.Mask) (width 0.01))
     (fp_poly (pts (xy -3.4302 -2.025) (xy -2.575 -2.025) (xy -2.575 -2.37861) (xy -3.4302 -2.37861)) (layer B.Mask) (width 0.01))
     (fp_poly (pts (xy -3.4362 -1.625) (xy -2.575 -1.625) (xy -2.575 -1.98146) (xy -3.4362 -1.98146)) (layer B.Mask) (width 0.01))
