File: shields/probe_shield/probe_shield.sch (KiCad schematic (older format))
At the start: 17 parts, among them IC1 NCP1117DT33T5G, J1 Probe Channel 0, J2 Probe Channel 1, J3 Probe Channel 2, J4 Probe Channel 3, J5 GPIO shield connector 40pin, J6 probe shield connector 26pin

Commit message: probe shield 3d model update
Parts:
- J5: footprint Connector_PinHeader_2.54mm:PinHeader_2x20_P2.54mm_Vertical -> hive:PinHeader_2x20_P2.54mm_Vertical_gpio_shield
- J6: footprint Connector_PinHeader_2.54mm:PinHeader_2x13_P2.54mm_Vertical -> hive:PinHeader_2x13_P2.54mm_Vertical_probe_shield_male
- LED1: footprint LEDC1608X80N -> hive:LEDC1608X80N
Changed lines of the file:
@@
 F 0 "J5" H 8700 3517 50  0000 C CNN
 F 1 "GPIO shield connector 40pin" H 8700 3426 50  0000 C CNN
-F 2 "Connector_PinHeader_2.54mm:PinHeader_2x20_P2.54mm_Vertical" H 8650 2400 50  0001 C CNN
+F 2 "hive:PinHeader_2x20_P2.54mm_Vertical_gpio_shield" H 8650 2400 50  0001 C CNN
 F 3 "~" H 8650 2400 50  0001 C CNN
 	1    8650 2400
@@
 F 0 "J6" H 8700 6050 50  0000 C CNN
 F 1 "probe shield connector 26pin" H 8700 5950 50  0000 C CNN
-F 2 "Connector_PinHeader_2.54mm:PinHeader_2x13_P2.54mm_Vertical" H 8650 5200 50  0001 C CNN
+F 2 "hive:PinHeader_2x13_P2.54mm_Vertical_probe_shield_male" H 8650 5200 50  0001 C CNN
 F 3 "~" H 8650 5200 50  0001 C CNN
 	1    8650 5200
@@
 F 0 "LED1" V 5846 2120 50  0000 R CNN
 F 1 "3.3V OK (green)" V 5755 2120 50  0000 R CNN
-F 2 "LEDC1608X80N" H 6000 2400 50  0001 L BNN
+F 2 "hive:LEDC1608X80N" H 6000 2400 50  0001 L BNN
 F 3 "https://componentsearchengine.com/Datasheets/2/150060VS75000.pdf" H 6000 2300 50  0001 L BNN
 F 4 "2.4 V Green LED 1608 (0603) SMD, Wurth Elektronik WL-SMCW 150060VS75000" H 6000 2200 50  0001 L BNN "Description"
@@
 	650  1950 900  1950
 $Comp
-L power:GND #PWR?
+L power:GND #PWR0105
 U 1 1 615DDDAF
 P 900 1950
-F 0 "#PWR?" H 900 1700 50  0001 C CNN
+F 0 "#PWR0105" H 900 1700 50  0001 C CNN
 F 1 "GND" V 905 1822 50  0000 R CNN
 F 2 "" H 900 1950 50  0001 C CNN
@@
 $EndComp
 $Comp
-L power:GND #PWR?
+L power:GND #PWR0106
 U 1 1 6158CD45
 P 7750 4600
-F 0 "#PWR?" H 7750 4350 50  0001 C CNN
+F 0 "#PWR0106" H 7750 4350 50  0001 C CNN
 F 1 "GND" V 7750 4400 50  0000 C CNN
 F 2 "" H 7750 4600 50  0001 C CNN
@@
 	8450 4600 7750 4600
 $Comp
-L power:GND #PWR?
+L power:GND #PWR0107
 U 1 1 61593F46
 P 7750 5200
-F 0 "#PWR?" H 7750 4950 50  0001 C CNN
+F 0 "#PWR0107" H 7750 4950 50  0001 C CNN
 F 1 "GND" V 7750 5000 50  0000 C CNN
 F 2 "" H 7750 5200 50  0001 C CNN
@@
 	8450 5200 7750 5200
 $Comp
-L power:GND #PWR?
+L power:GND #PWR0108
 U 1 1 61598641
 P 7750 5800
-F 0 "#PWR?" H 7750 5550 50  0001 C CNN
+F 0 "#PWR0108" H 7750 5550 50  0001 C CNN
 F 1 "GND" V 7750 5600 50  0000 C CNN
 F 2 "" H 7750 5800 50  0001 C CNN
@@
 	8450 5800 7750 5800
 $Comp
-L power:GND #PWR?
+L power:GND #PWR0109
 U 1 1 6159D4B7
 P 9650 5800
-F 0 "#PWR?" H 9650 5550 50  0001 C CNN
+F 0 "#PWR0109" H 9650 5550 50  0001 C CNN
 F 1 "GND" V 9650 5600 50  0000 C CNN
 F 2 "" H 9650 5800 50  0001 C CNN
@@
 	8950 5800 9650 5800
 $Comp
-L power:GND #PWR?
+L power:GND #PWR0110
 U 1 1 615A1DEC
 P 9650 5200
-F 0 "#PWR?" H 9650 4950 50  0001 C CNN
+F 0 "#PWR0110" H 9650 4950 50  0001 C CNN
 F 1 "GND" V 9650 5000 50  0000 C CNN
 F 2 "" H 9650 5200 50  0001 C CNN
@@
 	8950 5200 9650 5200
 $Comp
-L power:GND #PWR?
+L power:GND #PWR0111
 U 1 1 615A63BC
 P 9650 4600
-F 0 "#PWR?" H 9650 4350 50  0001 C CNN
+F 0 "#PWR0111" H 9650 4350 50  0001 C CNN
 F 1 "GND" V 9650 4400 50  0000 C CNN
 F 2 "" H 9650 4600 50  0001 C CNN

Commit message: added partlist and prices
Parts:
- C1, C2: Digikey Price (CHF) (none) -> 0.15; Mouser Price (CHF) (none) -> 0.13
- H1, H2, H3, H4, H5, H6, R1: Digikey Price (CHF) (none) -> -; Mouser Price (CHF) (none) -> -
- IC1: Digikey Price (CHF) (none) -> 0.62; Mouser Price (CHF) (none) -> 0.64
- J1, J2, J3, J4: Digikey Price (CHF) (none) -> 3.56; Manufacturer_Part_Number (none) -> FTSH-105-01-F-DV-007-K; Mouser Price (CHF) (none) -> 3.61
- J5: Digikey Price (CHF) (none) -> 2.74; Manufacturer_Part_Number (none) -> Adafruit 1979; Mouser Price (CHF) (none) -> 2.77
- J6: Digikey Price (CHF) (none) -> 2.01; Manufacturer_Part_Number (none) -> TSW-113-07-L-D; Mouser Price (CHF) (none) -> 2.02
- LED1: Digikey Price (CHF) (none) -> 0.14; Mouser Price (CHF) (none) -> 0.13
Changed lines of the file:
@@
 F 2 "MountingHole:MountingHole_2.7mm_M2.5_DIN965_Pad" H 850 700 50  0001 C CNN
 F 3 "~" H 850 700 50  0001 C CNN
+F 4 "-" H 850 700 50  0001 C CNN "Digikey Price (CHF)"
+F 5 "-" H 850 700 50  0001 C CNN "Mouser Price (CHF)"
 	1    850  700
 	0    1    1    0
@@
 F 5 "Manufacturer Recommendations" H 1900 3050 50  0001 L BNN "STANDARD"
 F 6 "Samtec" H 1850 3050 50  0001 L BNN "MANUFACTURER"
+F 7 "3.56" H 1850 3050 50  0001 C CNN "Digikey Price (CHF)"
+F 8 "FTSH-105-01-F-DV-007-K" H 1850 3050 50  0001 C CNN "Manufacturer_Part_Number"
+F 9 "3.61" H 1850 3050 50  0001 C CNN "Mouser Price (CHF)"
 	1    1850 3050
 	1    0    0    -1
@@
 F 7 "ON Semiconductor" H 4500 700 50  0001 L CNN "Manufacturer_Name"
 F 8 "NCP1117DT33T5G" H 4500 600 50  0001 L CNN "Manufacturer_Part_Number"
+F 9 "0.62" H 3150 1200 50  0001 C CNN "Digikey Price (CHF)"
+F 10 "0.64" H 3150 1200 50  0001 C CNN "Mouser Price (CHF)"
 	1    3150 1200
 	1    0    0    -1
@@
 F 2 "Capacitor_SMD:C_0805_2012Metric_Pad1.15x1.40mm_HandSolder" H 2800 1300 50  0001 C CNN
 F 3 "~" H 2800 1300 50  0001 C CNN
+F 4 "0.15" H 2800 1300 50  0001 C CNN "Digikey Price (CHF)"
+F 5 "0.13" H 2800 1300 50  0001 C CNN "Mouser Price (CHF)"
 	1    2800 1300
 	1    0    0    -1
@@
 F 2 "Capacitor_SMD:C_0805_2012Metric_Pad1.15x1.40mm_HandSolder" H 4900 1300 50  0001 C CNN
 F 3 "~" H 4900 1300 50  0001 C CNN
+F 4 "0.15" H 4900 1300 50  0001 C CNN "Digikey Price (CHF)"
+F 5 "0.13" H 4900 1300 50  0001 C CNN "Mouser Price (CHF)"
 	1    4900 1300
 	1    0    0    -1
@@
 F 5 "Manufacturer Recommendations" H 1900 4000 50  0001 L BNN "STANDARD"
 F 6 "Samtec" H 1850 4000 50  0001 L BNN "MANUFACTURER"
+F 7 "3.56" H 1850 4000 50  0001 C CNN "Digikey Price (CHF)"
+F 8 "FTSH-105-01-F-DV-007-K" H 1850 4000 50  0001 C CNN "Manufacturer_Part_Number"
+F 9 "3.61" H 1850 4000 50  0001 C CNN "Mouser Price (CHF)"
 	1    1850 4000
 	1    0    0    -1
@@
 F 5 "Manufacturer Recommendations" H 1900 4950 50  0001 L BNN "STANDARD"
 F 6 "Samtec" H 1850 4950 50  0001 L BNN "MANUFACTURER"
+F 7 "3.56" H 1850 4950 50  0001 C CNN "Digikey Price (CHF)"
+F 8 "FTSH-105-01-F-DV-007-K" H 1850 4950 50  0001 C CNN "Manufacturer_Part_Number"
+F 9 "3.61" H 1850 4950 50  0001 C CNN "Mouser Price (CHF)"
 	1    1850 4950
 	1    0    0    -1
@@
 F 5 "Manufacturer Recommendations" H 1900 5900 50  0001 L BNN "STANDARD"
 F 6 "Samtec" H 1850 5900 50  0001 L BNN "MANUFACTURER"
+F 7 "3.56" H 1850 5900 50  0001 C CNN "Digikey Price (CHF)"
+F 8 "FTSH-105-01-F-DV-007-K" H 1850 5900 50  0001 C CNN "Manufacturer_Part_Number"
+F 9 "3.61" H 1850 5900 50  0001 C CNN "Mouser Price (CHF)"
 	1    1850 5900
 	1    0    0    -1
@@
 F 2 "hive:PinHeader_2x20_P2.54mm_Vertical_gpio_shield" H 8650 2400 50  0001 C CNN
 F 3 "~" H 8650 2400 50  0001 C CNN
+F 4 "2.74" H 8650 2400 50  0001 C CNN "Digikey Price (CHF)"
+F 5 "Adafruit 1979" H 8650 2400 50  0001 C CNN "Manufacturer_Part_Number"
+F 6 "2.77" H 8650 2400 50  0001 C CNN "Mouser Price (CHF)"
 	1    8650 2400
 	1    0    0    -1
@@
 F 2 "hive:PinHeader_2x13_P2.54mm_Vertical_probe_shield_male" H 8650 5200 50  0001 C CNN
 F 3 "~" H 8650 5200 50  0001 C CNN
+F 4 "TSW-113-07-L-D" H 8650 5200 50  0001 C CNN "Manufacturer_Part_Number"
+F 5 "2.01" H 8650 5200 50  0001 C CNN "Digikey Price (CHF)"
+F 6 "2.02" H 8650 5200 50  0001 C CNN "Mouser Price (CHF)"
 	1    8650 5200
 	1    0    0    -1
@@
 F 2 "Resistor_SMD:R_0805_2012Metric_Pad1.15x1.40mm_HandSolder" H 5500 1400 50  0001 C CNN
 F 3 "~" H 5500 1400 50  0001 C CNN
+F 4 "-" H 5500 1400 50  0001 C CNN "Digikey Price (CHF)"
+F 5 "-" H 5500 1400 50  0001 C CNN "Mouser Price (CHF)"
 	1    5500 1400
 	1    0    0    -1
@@
 F 8 "Wurth Elektronik" H 6000 1800 50  0001 L BNN "Manufacturer_Name"
 F 9 "150060VS75000" H 6000 1700 50  0001 L BNN "Manufacturer_Part_Number"
+F 10 "0.14" H 5500 2250 50  0001 C CNN "Digikey Price (CHF)"
+F 11 "0.13" H 5500 2250 50  0001 C CNN "Mouser Price (CHF)"
 	1    5500 2250
 	0    -1   -1   0
@@
 F 2 "MountingHole:MountingHole_2.7mm_M2.5_DIN965_Pad" H 850 900 50  0001 C CNN
 F 3 "~" H 850 900 50  0001 C CNN
+F 4 "-" H 850 900 50  0001 C CNN "Digikey Price (CHF)"
+F 5 "-" H 850 900 50  0001 C CNN "Mouser Price (CHF)"
 	1    850  900
 	0    1    1    0
@@
 F 2 "MountingHole:MountingHole_2.7mm_M2.5_DIN965_Pad" H 850 1100 50  0001 C CNN
 F 3 "~" H 850 1100 50  0001 C CNN
+F 4 "-" H 850 1100 50  0001 C CNN "Digikey Price (CHF)"
+F 5 "-" H 850 1100 50  0001 C CNN "Mouser Price (CHF)"
 	1    850  1100
 	0    1    1    0
@@
 F 2 "MountingHole:MountingHole_2.7mm_M2.5_DIN965_Pad" H 850 1300 50  0001 C CNN
 F 3 "~" H 850 1300 50  0001 C CNN
+F 4 "-" H 850 1300 50  0001 C CNN "Digikey Price (CHF)"
+F 5 "-" H 850 1300 50  0001 C CNN "Mouser Price (CHF)"
 	1    850  1300
 	0    1    1    0
@@
 F 2 "MountingHole:MountingHole_2.7mm_M2.5_DIN965_Pad" H 850 1500 50  0001 C CNN
 F 3 "~" H 850 1500 50  0001 C CNN
+F 4 "-" H 850 1500 50  0001 C CNN "Digikey Price (CHF)"
+F 5 "-" H 850 1500 50  0001 C CNN "Mouser Price (CHF)"
 	1    850  1500
 	0    1    1    0
@@
 F 2 "MountingHole:MountingHole_2.7mm_M2.5_DIN965_Pad" H 850 1700 50  0001 C CNN
 F 3 "~" H 850 1700 50  0001 C CNN
+F 4 "-" H 850 1700 50  0001 C CNN "Digikey Price (CHF)"
+F 5 "-" H 850 1700 50  0001 C CNN "Mouser Price (CHF)"
 	1    850  1700
 	0    1    1    0

Commit message: updated LED resistor values, updated partlists, minor change to daughterboard template
Parts:
- R1: value 195 -> 560
Changed lines of the file:
@@
 P 5500 1400
 F 0 "R1" H 5559 1446 50  0000 L CNN
-F 1 "195" H 5559 1355 50  0000 L CNN
+F 1 "560" H 5559 1355 50  0000 L CNN
 F 2 "Resistor_SMD:R_0805_2012Metric_Pad1.15x1.40mm_HandSolder" H 5500 1400 50  0001 C CNN
 F 3 "~" H 5500 1400 50  0001 C CNN
