File: shields/probe_shield/probe_shield.kicad_pcb (KiCad board)
At the start: 4 copper layers, 85 x 56 mm, 18 parts, among them IC1 NCP1117DT33T5G, J1 Probe Channel 0, J2 Probe Channel 1, J3 Probe Channel 2, J4 Probe Channel 3, J5 GPIO shield connector 40pin, J6 probe shield connector 26pin

Commit message: slight layout adjustments for manufacturing
Routing:
- net (no net): track 1.52 -> 0.00 mm
Changed lines of the file:
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@@
     (thickness 1.6)
     (drawings 58)
-    (tracks 551)
+    (tracks 549)
     (zones 0)
     (modules 18)
@@
     (pcbplotparams
       (layerselection 0x010fc_ffffffff)
-      (usegerberextensions false)
+      (usegerberextensions true)
       (usegerberattributes false)
       (usegerberadvancedattributes false)
@@
       (psa4output false)
       (plotreference true)
-      (plotvalue true)
+      (plotvalue false)
       (plotinvisibletext false)
       (padsonsilk false)
-      (subtractmaskfromsilk false)
+      (subtractmaskfromsilk true)
       (outputformat 1)
       (mirror false)
-      (drillshape 1)
+      (drillshape 0)
       (scaleselection 1)
-      (outputdirectory ""))
+      (outputdirectory "gerbers/"))
   )
   (net 0 "")
@@
   (gr_arc (start 192 57) (end 195 57) (angle -90) (layer Edge.Cuts) (width 0.05))
   (gr_arc (start 113 57) (end 113 54) (angle -90) (layer Edge.Cuts) (width 0.05))
-  (segment (start 119.652 58.438) (end 119.652 59.2) (width 0.18) (layer PWR_SIG.Cu) (net 0))
-  (segment (start 122.192 58.438) (end 122.192 59.2) (width 0.18) (layer PWR_SIG.Cu) (net 0))
   (segment (start 115 73.6) (end 115 76.961) (width 0.386) (layer B.Cu) (net 1))
   (via (at 118.89 77.996) (size 1) (drill 0.5) (layers F.Cu B.Cu) (net 1))
@@
   (zone (net 2) (net_name +5V) (layer PWR_SIG.Cu) (hatch edge 0.508)
     (connect_pads (clearance 0.3))
-    (min_thickness 0.254)
+    (min_thickness 0.2)
     (fill yes (arc_segments 32) (thermal_gap 0.508) (thermal_bridge_width 0.508))
     (polygon

Commit message: enhanced mechanical PCB drawings of stack shields and daughterboard template
Parts:
- R1: value 195 -> 560
Other:
- board text added: "All mounting holes: M2.5 pass-through"
- board text added: "All rounded edges: 3mm radius"
- board text added: "Back view"
- board text added: "Front view"
Changed lines of the file:
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@@
   (general
     (thickness 1.6)
-    (drawings 58)
+    (drawings 63)
     (tracks 549)
     (zones 0)
@@
     (visible_elements 7FFFFFFF)
     (pcbplotparams
-      (layerselection 0x010fc_ffffffff)
+      (layerselection 0x10000_7ffffff8)
       (usegerberextensions true)
       (usegerberattributes false)
@@
       (excludeedgelayer true)
       (linewidth 0.100000)
-      (plotframeref false)
+      (plotframeref true)
       (viasonmask false)
       (mode 1)
@@
       (psa4output false)
       (plotreference true)
-      (plotvalue false)
+      (plotvalue true)
       (plotinvisibletext false)
       (padsonsilk false)
       (subtractmaskfromsilk true)
-      (outputformat 1)
-      (mirror false)
+      (outputformat 4)
+      (mirror true)
       (drillshape 0)
       (scaleselection 1)
@@
       (effects (font (size 1 1) (thickness 0.15)))
     )
-    (fp_text user %R (at 1.27 15.24 90) (layer F.Fab)
+    (fp_text user %R (at 1.27 13.74 90) (layer F.Fab)
       (effects (font (size 1 1) (thickness 0.15)))
     )
@@
     (fp_line (start 4.35 50.05) (end 4.35 -1.8) (layer F.CrtYd) (width 0.05))
     (fp_line (start 4.35 -1.8) (end -1.8 -1.8) (layer F.CrtYd) (width 0.05))
-    (fp_text user %R (at 1.27 24.13 180) (layer F.Fab)
+    (fp_text user %R (at 1.27 22.63 180) (layer F.Fab)
       (effects (font (size 1 1) (thickness 0.15)))
     )
@@
       (effects (font (size 1 1) (thickness 0.15)))
     )
-    (fp_text value 195 (at 0 1.65 90) (layer F.Fab)
+    (fp_text value 560 (at 0 1.65 90) (layer F.Fab)
       (effects (font (size 1 1) (thickness 0.15)))
     )
@@
     )
   )
+  (gr_text "Back view" (at 201 37) (layer B.Fab)
+    (effects (font (size 2 2) (thickness 0.15)) (justify mirror))
+  )
+  (gr_text "Front view" (at 103 37) (layer F.Fab)
+    (effects (font (size 2 2) (thickness 0.15)))
+  )
+  (gr_text "All rounded edges: 3mm radius" (at 125 125) (layer F.Fab)
+    (effects (font (size 2 2) (thickness 0.15)))
+  )
+  (gr_text "All mounting holes: M2.5 pass-through" (at 126 121) (layer F.Fab)
+    (effects (font (size 2 2) (thickness 0.15)))
+  )
+  (dimension 23.5 (width 0.15) (layer F.Fab)
+    (gr_text "23.500 mm" (at 183.25 114.8) (layer F.Fab)
+      (effects (font (size 1 1) (thickness 0.15)))
+    )
+    (feature1 (pts (xy 195 106.5) (xy 195 114.086421)))
+    (feature2 (pts (xy 171.5 106.5) (xy 171.5 114.086421)))
+    (crossbar (pts (xy 171.5 113.5) (xy 195 113.5)))
+    (arrow1a (pts (xy 195 113.5) (xy 193.873496 114.086421)))
+    (arrow1b (pts (xy 195 113.5) (xy 193.873496 112.913579)))
+    (arrow2a (pts (xy 171.5 113.5) (xy 172.626504 114.086421)))
+    (arrow2b (pts (xy 171.5 113.5) (xy 172.626504 112.913579)))
+  )
   (dimension 24 (width 0.15) (layer F.Fab)
-    (gr_text "24.000 mm" (at 199.8 98 270) (layer F.Fab)
-      (effects (font (size 1 1) (thickness 0.15)))
-    )
+    (gr_text "24.000 mm" (at 199.8 98 90) (layer F.Fab)
+      (effects (font (size 1 1) (thickness 0.15)))
+    )
