File: daughterboard/daughterboard_template/daughterboard_template.kicad_pcb (KiCad board)
At the start: 4 copper layers, 67 x 50 mm, 2 parts, among them J1 m2_keyA_67pin_daughterboard

Commit message: enhanced mechanical PCB drawings of stack shields and daughterboard template
Other:
- board text added: "All rounded corners: 2mm radius"
- board text added: "Front view"
- board text added: "M.2 PCIE connector measurements according to specification"
- board text added: "hole: M2.5 pass-through"
Changed lines of the file:
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@@
   (general
     (thickness 0.8)
-    (drawings 38)
+    (drawings 49)
     (tracks 65)
     (zones 0)
@@
     (visible_elements 7FFFFFFF)
     (pcbplotparams
-      (layerselection 0x010fc_ffffffff)
+      (layerselection 0x20000_7ffffff8)
       (usegerberextensions false)
       (usegerberattributes false)
@@
       (excludeedgelayer true)
       (linewidth 0.100000)
-      (plotframeref false)
+      (plotframeref true)
       (viasonmask false)
       (mode 1)
@@
       (padsonsilk false)
       (subtractmaskfromsilk false)
-      (outputformat 1)
+      (outputformat 4)
       (mirror false)
-      (drillshape 1)
+      (drillshape 0)
       (scaleselection 1)
-      (outputdirectory ""))
+      (outputdirectory "gerbers/"))
   )
   (net 0 "")
@@
     (fp_circle (center 0 0) (end 2.95 0) (layer F.CrtYd) (width 0.05))
     (fp_circle (center 0 0) (end 2.7 0) (layer Cmts.User) (width 0.15))
-    (fp_text user %R (at 0.3 0) (layer F.Fab)
+    (fp_text user %R (at 0.3 0) (layer F.Fab) hide
       (effects (font (size 1 1) (thickness 0.15)))
     )
@@
       (net 44 +5V) (solder_mask_margin 0.1016))
   )
+  (gr_text "hole: M2.5 pass-through" (at 139.5 153) (layer F.Fab)
+    (effects (font (size 2 2) (thickness 0.15)))
+  )
+  (dimension 15.5 (width 0.15) (layer F.Fab)
+    (gr_text "15.500 mm" (at 144.2 84.75 90) (layer F.Fab)
+      (effects (font (size 1 1) (thickness 0.15)))
+    )
+    (feature1 (pts (xy 148.5 77) (xy 144.913579 77)))
+    (feature2 (pts (xy 148.5 92.5) (xy 144.913579 92.5)))
+    (crossbar (pts (xy 145.5 92.5) (xy 145.5 77)))
+    (arrow1a (pts (xy 145.5 77) (xy 146.086421 78.126504)))
+    (arrow1b (pts (xy 145.5 77) (xy 144.913579 78.126504)))
+    (arrow2a (pts (xy 145.5 92.5) (xy 146.086421 91.373496)))
+    (arrow2b (pts (xy 145.5 92.5) (xy 144.913579 91.373496)))
+  )
+  (gr_text "M.2 PCIE connector measurements according to specification" (at 139.5 148.5) (layer F.Fab)
+    (effects (font (size 2 2) (thickness 0.15)))
+  )
+  (dimension 4.35 (width 0.15) (layer F.Fab)
+    (gr_text "4.350 mm" (at 156.275 124.2) (layer F.Fab)
+      (effects (font (size 1 1) (thickness 0.15)))
+    )
+    (feature1 (pts (xy 154.1 127.5) (xy 154.1 124.913579)))
+    (feature2 (pts (xy 158.45 127.5) (xy 158.45 124.913579)))
+    (crossbar (pts (xy 158.45 125.5) (xy 154.1 125.5)))
+    (arrow1a (pts (xy 154.1 125.5) (xy 155.226504 124.913579)))
+    (arrow1b (pts (xy 154.1 125.5) (xy 155.226504 126.086421)))
+    (arrow2a (pts (xy 158.45 125.5) (xy 157.323496 124.913579)))
+    (arrow2b (pts (xy 158.45 125.5) (xy 157.323496 126.086421)))
+  )
+  (dimension 19.9 (width 0.15) (layer F.Fab)
+    (gr_text "19.900 mm" (at 148.5 133.799999) (layer F.Fab)
+      (effects (font (size 1 1) (thickness 0.15)))
+    )
+    (feature1 (pts (xy 158.45 130.8) (xy 158.45 133.08642)))
+    (feature2 (pts (xy 138.55 130.8) (xy 138.55 133.08642)))
+    (crossbar (pts (xy 138.55 132.499999) (xy 158.45 132.499999)))
+    (arrow1a (pts (xy 158.45 132.499999) (xy 157.323496 133.08642)))
+    (arrow1b (pts (xy 158.45 132.499999) (xy 157.323496 131.913578)))
+    (arrow2a (pts (xy 138.55 132.499999) (xy 139.676504 133.08642)))
+    (arrow2b (pts (xy 138.55 132.499999) (xy 139.676504 131.913578)))
+  )
+  (gr_text "Front view" (at 112 64.5) (layer F.Fab)
+    (effects (font (size 2 2) (thickness 0.15)))
+  )
+  (gr_text "All rounded corners: 2mm radius\n" (at 139.5 144) (layer F.Fab)
+    (effects (font (size 2 2) (thickness 0.15)))
+  )
+  (dimension 4 (width 0.15) (layer F.Fab)
+    (gr_text "4.000 mm" (at 134.2 135 90) (layer F.Fab)
+      (effects (font (size 1 1) (thickness 0.15)))
+    )
+    (feature1 (pts (xy 138.5 127) (xy 134.913579 127)))
+    (feature2 (pts (xy 138.5 131) (xy 134.913579 131)))
+    (crossbar (pts (xy 135.5 131) (xy 135.5 127)))
+    (arrow1a (pts (xy 135.5 127) (xy 136.086421 128.126504)))
+    (arrow1b (pts (xy 135.5 127) (xy 134.913579 128.126504)))
+    (arrow2a (pts (xy 135.5 131) (xy 136.086421 129.873496)))
+    (arrow2b (pts (xy 135.5 131) (xy 134.913579 129.873496)))
+  )
+  (gr_circle (center 148.5 92.5) (end 150.081139 92.5) (layer F.Fab) (width 0.15))
+  (gr_line (start 159.3 127) (end 180 127) (layer F.Fab) (width 0.1))
+  (gr_line (start 117 127) (end 137.7 127) (layer F.Fab) (width 0.1))
   (gr_text "Do not place any components inside the filled zone!\nZone will be obscured by magnet" (at 149 86) (layer Cmts.User)
     (effects (font (size 1 1) (thickness 0.15)))
